File: serial/serial.kicad_pcb (KiCad board)
At the start: 2 copper layers, 24 x 12 mm, 8 parts, among them J2 Conn_02x03_Odd_Even, Q1 BSS138, Q2 BSS138, U1 CH340K

Commit message: -
Parts:
- 0u1 x3: renamed from C2
- BSS138 x2: renamed from Q2
- renumbered C1 to 0u1, C3 to 0u1, U1 to CH340K
Other:
- board text added: "0E5 TRG"
- board text added: "CH340K*1 BSS138*2 0.1uF*3"
- board text removed: "5V G EN RX 0 TX"
- board text removed: "@McbeEringi"

Commit message: -
Other:
- board size 24 x 12 mm -> 24.2 x 12.2 mm

Commit message: -
Parts:
- turned 0u1 to 0 degrees
Routing:
- net Net-(J2-Pin_6): track 14.5 -> 17.7 mm
- net Net-(J2-Pin_2): track 17.8 -> 19.3 mm
- net Net-(J2-Pin_5): track 15.6 -> 14.6 mm
- net Net-(Q1-G): track 5.84 -> 6.66 mm
- net Net-(J2-Pin_1): track 5.26 -> 5.10 mm, vias 8 -> 10
Other:
- board text added: "JLCJLCJLCJLC"

Commit message: -
Other:
- board text added: "USB-Serial ESP32"
- board text removed: "CH340K ~5v UART ESP32 AUTO PGM"
- board text removed: "CH340K*1 BSS138*2 0.1uF*3"

Commit message: -
Routing:
- net Net-(J2-Pin_1): track 5.10 -> 10.6 mm
Changed lines of the file:
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@@
     (pad "4" smd rect (at 4.945 3.5) (size 7.41 1) (layers "F.Cu" "F.Paste" "F.Mask")
       (net 1 "Net-(J2-Pin_2)") (pinfunction "VBUS") (pintype "power_in") (thermal_bridge_angle 45))
-    (pad "5" smd rect (at 5.16 -2.75) (size 2 2.5) (layers "B.Cu" "B.Paste" "B.Mask")
+    (pad "5" smd rect (at 4.16 -2.75) (size 2 2.5) (layers "B.Cu" "B.Paste" "B.Mask")
       (net 2 "Net-(J2-Pin_1)") (pinfunction "SHIELD") (pintype "power_in") (thermal_bridge_angle 45))
-    (pad "6" smd rect (at 5.16 2.75) (size 2 2.5) (layers "B.Cu" "B.Paste" "B.Mask")
+    (pad "6" smd rect (at 4.16 2.75) (size 2 2.5) (layers "B.Cu" "B.Paste" "B.Mask")
       (net 2 "Net-(J2-Pin_1)") (pinfunction "SHIELD") (pintype "power_in") (thermal_bridge_angle 45))
   )
@@
   (via (at 110.9 105.3) (size 0.8) (drill 0.4) (layers "F.Cu" "B.Cu") (free) (net 2))
   (via (at 114.15 98.3) (size 0.8) (drill 0.4) (layers "F.Cu" "B.Cu") (free) (net 2))
+  (segment (start 104.16 97.25) (end 104.16 102.75) (width 0.5) (layer "B.Cu") (net 2))
   (segment (start 112.6 98.3) (end 112.6 99.95) (width 0.25) (layer "F.Cu") (net 3))
   (segment (start 115.113299 102.275) (end 118.633299 102.275) (width 0.25) (layer "F.Cu") (net 4))
@@
     (polygon
       (pts
-        (xy 99.9 93.9)
+        (xy 110.2 93.8)
         (xy 124.1 93.9)
         (xy 124.1 106.1)
-        (xy 99.9 106.1)
+        (xy 110.2 106)
       )
     )
