File: t85/t85.kicad_sch (KiCad schematic)
At the start: 14 parts, among them J1 USB, J2 Conn_02x04_Counter_Clockwise, SW1 SW_Push, U1 ATtiny85-20S

Commit message: -
Parts:
- J1: footprint Library:USB -> Library:USB-micro-b
Changed lines of the file:
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@@
   (junction (at 119.38 93.98) (diameter 0) (color 0 0 0 0)
   )
-  (junction (at 101.6 101.6) (diameter 0) (color 0 0 0 0)
+  (junction (at 101.6 100.33) (diameter 0) (color 0 0 0 0)
   )
   (junction (at 147.32 111.76) (diameter 0) (color 0 0 0 0)
@@
   (junction (at 113.03 93.98) (diameter 0) (color 0 0 0 0)
   )
-  (wire (pts (xy 99.06 101.6) (xy 99.06 100.33))
-    (stroke (width 0) (type default))
-  )
   (wire (pts (xy 147.32 111.76) (xy 110.49 111.76))
     (stroke (width 0) (type default))
@@
     (stroke (width 0) (type default))
   )
+  (wire (pts (xy 123.19 81.28) (xy 147.32 81.28))
+    (stroke (width 0) (type default))
+  )
+  (wire (pts (xy 110.49 81.28) (xy 123.19 81.28))
+    (stroke (width 0) (type default))
+  )
+  (wire (pts (xy 99.06 100.33) (xy 101.6 100.33))
+    (stroke (width 0) (type default))
+  )
+  (wire (pts (xy 123.19 81.28) (xy 123.19 83.82))
+    (stroke (width 0) (type default))
+  )
+  (wire (pts (xy 113.03 93.98) (xy 119.38 93.98))
+    (stroke (width 0) (type default))
+  )
+  (wire (pts (xy 101.6 101.6) (xy 110.49 101.6))
+    (stroke (width 0) (type default))
+  )
+  (wire (pts (xy 119.38 101.6) (xy 123.19 101.6))
+    (stroke (width 0) (type default))
+  )
+  (wire (pts (xy 184.15 111.76) (xy 147.32 111.76))
+    (stroke (width 0) (type default))
+  )
+  (wire (pts (xy 119.38 93.98) (xy 125.73 93.98))
+    (stroke (width 0) (type default))
+  )
   (wire (pts (xy 110.49 96.52) (xy 110.49 101.6))
     (stroke (width 0) (type default))
   )
-  (wire (pts (xy 123.19 81.28) (xy 147.32 81.28))
-    (stroke (width 0) (type default))
-  )
-  (wire (pts (xy 110.49 81.28) (xy 123.19 81.28))
-    (stroke (width 0) (type default))
-  )
-  (wire (pts (xy 101.6 101.6) (xy 110.49 101.6))
-    (stroke (width 0) (type default))
-  )
-  (wire (pts (xy 123.19 81.28) (xy 123.19 83.82))
-    (stroke (width 0) (type default))
-  )
-  (wire (pts (xy 113.03 93.98) (xy 119.38 93.98))
-    (stroke (width 0) (type default))
-  )
-  (wire (pts (xy 119.38 101.6) (xy 123.19 101.6))
-    (stroke (width 0) (type default))
-  )
-  (wire (pts (xy 184.15 111.76) (xy 147.32 111.76))
-    (stroke (width 0) (type default))
-  )
-  (wire (pts (xy 119.38 93.98) (xy 125.73 93.98))
-    (stroke (width 0) (type default))
-  )
   (wire (pts (xy 113.03 91.44) (xy 123.19 91.44))
     (stroke (width 0) (type default))
@@
     (stroke (width 0) (type default))
   )
+  (wire (pts (xy 101.6 101.6) (xy 101.6 100.33))
+    (stroke (width 0) (type default))
+  )
   (wire (pts (xy 110.49 81.28) (xy 110.49 88.9))
     (stroke (width 0) (type default))
   )
   (wire (pts (xy 110.49 91.44) (xy 113.03 91.44))
-    (stroke (width 0) (type default))
-  )
-  (wire (pts (xy 101.6 101.6) (xy 101.6 100.33))
-    (stroke (width 0) (type default))
-  )
-  (wire (pts (xy 99.06 101.6) (xy 101.6 101.6))
     (stroke (width 0) (type default))
   )
@@
     )
   )
-  (symbol (lib_id "Device:LED") (at 209.55 118.11 90) (unit 1)
-    (in_bom yes) (on_board yes) (dnp no) (fields_autoplaced)
-    (property "Reference" "D1" (at 213.36 118.4275 90)
-      (effects (font (size 1.27 1.27)) (justify right))
-    )
-    (property "Value" "LED" (at 213.36 120.9675 90)
-      (effects (font (size 1.27 1.27)) (justify right))
-    )
-    (property "Footprint" "LED_SMD:LED_0603_1608Metric" (at 209.55 118.11 0)
-      (effects (font (size 1.27 1.27)) hide)
-    )
-    (property "Datasheet" "~" (at 209.55 118.11 0)
-      (effects (font (size 1.27 1.27)) hide)
-    )
-    (pin "1")
-    (pin "2")
-    (instances
-      (project "t85"
-        (path "/d25b5218-2adb-4dad-ba1c-be3909cba342"
-          (reference "D1") (unit 1)
-        )
-      )
-    )
-  )
   (symbol (lib_id "Library:USB") (at 102.87 92.71 0) (unit 1)
     (in_bom yes) (on_board yes) (dnp no) (fields_autoplaced)
@@
       (effects (font (size 1.27 1.27)))
     )
-    (property "Footprint" "Library:USB" (at 110.49 92.71 0)
+    (property "Footprint" "Library:USB-micro-b" (at 110.49 92.71 0)
       (effects (font (size 1.27 1.27)) hide)
     )
@@
         )
       )
+    )
+  )
+  (symbol (lib_id "Device:LED") (at 209.55 118.11 90) (unit 1)
+    (in_bom yes) (on_board yes) (dnp no) (fields_autoplaced)
+    (property "Reference" "D1" (at 213.36 118.4275 90)
+      (effects (font (size 1.27 1.27)) (justify right))
+    )
+    (property "Value" "LED" (at 213.36 120.9675 90)
+      (effects (font (size 1.27 1.27)) (justify right))
+    )
+    (property "Footprint" "LED_SMD:LED_0603_1608Metric" (at 209.55 118.11 0)
+      (effects (font (size 1.27 1.27)) hide)
+    )
+    (property "Datasheet" "~" (at 209.55 118.11 0)
+      (effects (font (size 1.27 1.27)) hide)
+    )
+    (pin "1")
+    (pin "2")
+    (instances
+      (project "t85"
+        (path "/d25b5218-2adb-4dad-ba1c-be3909cba342"
+          (reference "D1") (unit 1)
+        )
+      )
