File: t85/t85.kicad_pcb (KiCad board)
At the start: 2 copper layers, 20.3 x 7.6 mm, 15 parts, among them J1 USB, J2 Conn_02x04_Counter_Clockwise, SW1 SW_Push, U1 ATtiny85-20S

Commit message: -
Parts:
- removed REF**: smd_3x4, Library:smd_3x4
- removed TP1, TP2: TestPoint, TestPoint:TestPoint_Pad_D1.0mm
- added C2: 1F5, Library:edlc, F.Cu at (112.7, 100.0)
- added R5: 5k1, Resistor_SMD:R_0603_1608Metric, B.Cu at (100.6, 98.4)
- added R6: 5k1, Resistor_SMD:R_0603_1608Metric, B.Cu at (100.6, 101.7)
- added SW2: SW_SPDT, Library:sw, F.Cu at (115.2, 100.0)
- J1: value USB -> USB-C; footprint Library:USB-micro-b -> Library:USB-C
- J2: value Conn_02x04_Counter_Clockwise -> OUT
- moved J1 12.0 mm to (100.0, 100.0)
- moved R4 11.2 mm to (110.2, 98.4)
- moved SW1 10.8 mm to (102.7, 100.0)
- moved R2 10.7 mm to (107.6, 98.4), turned to -90 degrees
- moved R3 10.7 mm to (105.1, 98.4)
- moved D2 10.7 mm to (106.3, 98.2)
- moved D3 10.7 mm to (108.9, 98.2)
- moved J2 10.7 mm to (110.2, 96.2)
- moved U1 10.7 mm to (106.3, 100.0)
- moved C1 9.47 mm to (110.2, 101.7)
- moved R1 9.47 mm to (108.9, 101.7)
- moved D1 9.47 mm to (107.6, 101.7)
Connections:
- net RESET# renamed EN
- C1 pad 1: +5V -> VCC
- J1 pad 4: +5V -> VCC
- J2 pad 8: +5V -> VCC
- R2 pad 1: D- -> PB3
- R2 pad 2: PB3 -> D-
- R4 pad 1: D- -> VCC
- R4 pad 2: +5V -> D-
- U1 pad 8: +5V -> VCC
Routing:
- net GND: track 2.57 -> 19.8 mm, vias 5 -> 7
- net VCC: track 0.00 -> 16.4 mm, vias 0 -> 6
- net PB3: track 12.4 -> 5.40 mm
- net D+: track 11.4 -> 7.92 mm
- net +5V: track 2.57 -> 0.00 mm, vias 3 -> 0
- net /Vedlc: track 0.00 -> 2.54 mm
- net PB4: track 11.3 -> 8.83 mm
- net PB1: track 7.69 -> 8.76 mm
- net D-: track 13.0 -> 12.4 mm
- added copper zone on B.Cu, net VCC
- added copper zone on F.Cu, net VCC
- removed copper zone on B.Cu, net +5V
- removed copper zone on F.Cu, net +5V
Other:
- board size 20.3 x 7.6 mm -> 21.6 x 7.6 mm

Commit message: -
Parts:
- moved C2 3.81 mm to (116.5, 100.0)
- moved SW2 3.81 mm to (119.0, 100.0)
Routing:
- net D+: track 7.92 -> 14.4 mm, vias 0 -> 1
- net GND: track 19.8 -> 23.8 mm
- net VCC: track 16.4 -> 20.2 mm
- net D-: track 12.4 -> 16.1 mm, vias 0 -> 1
- net Net-(J1-CC2): track 0.00 -> 3.55 mm
- net Net-(J1-CC1): track 0.00 -> 3.55 mm, vias 0 -> 1
Other:
- board text added: "ATtiny85 USB-C"
- board text removed: "ATtiny85 Micronucleus"

Commit message: -
Routing:
- net PB0: track 1.64 -> 3.38 mm, vias 1 -> 0
Changed lines of the file:
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@@
   )
   (footprint "Library:sw_push_smd" (layer "F.Cu")
-    (at 102.7 100 90)
+    (at 102.72 100 90)
     (property "Sheetfile" "t85.kicad_sch")
     (property "Sheetname" "")
@@
   (segment (start 103.875 101.44538) (end 103.875 102.48) (width 0.25) (layer "B.Cu") (net 2))
   (segment (start 102.7 100.635) (end 103.32 101.255) (width 0.25) (layer "B.Cu") (net 2))
+  (segment (start 103.32 101.255) (end 103.68462 101.255) (width 0.25) (layer "B.Cu") (net 2))
   (segment (start 103.875 102.48) (end 105.08 103.685) (width 0.25) (layer "B.Cu") (net 2))
-  (segment (start 103.32 101.255) (end 103.68462 101.255) (width 0.25) (layer "B.Cu") (net 2))
   (segment (start 103.68462 101.255) (end 103.875 101.44538) (width 0.25) (layer "B.Cu") (net 2))
   (segment (start 104.46358 99.174) (end 104.164579 98.875) (width 0.2) (layer "F.Cu") (net 3))
@@
   (segment (start 99.25 100.5) (end 98.5 99.75) (width 0.2) (layer "B.Cu") (net 4))
   (segment (start 98.5 99.75) (end 97.465 99.75) (width 0.2) (layer "B.Cu") (net 4))
-  (via (at 102.7 102.225) (size 0.8) (drill 0.4) (layers "F.Cu" "B.Cu") (net 5))
-  (segment (start 102.54 102.385) (end 102.54 103.685) (width 0.25) (layer "B.Cu") (net 5))
-  (segment (start 102.7 102.225) (end 102.54 102.385) (width 0.25) (layer "B.Cu") (net 5))
-  (segment (start 102.7 102.225) (end 102.62 102.145) (width 0.25) (layer "B.Cu") (net 5))
+  (segment (start 102.54 102.405) (end 102.54 103.685) (width 0.25) (layer "F.Cu") (net 5))
+  (segment (start 102.72 102.225) (end 102.54 102.405) (width 0.25) (layer "F.Cu") (net 5))
+  (segment (start 102.7 101.905) (end 102.54 102.065) (width 0.25) (layer "B.Cu") (net 5))
+  (segment (start 102.54 102.065) (end 102.54 103.685) (width 0.25) (layer "B.Cu") (net 5))
   (segment (start 106.538878 103.685) (end 107.62 103.685) (width 0.25) (layer "B.Cu") (net 6))
-  (segment (start 103.91066 99.25) (end 104.35 99.68934) (width 0.25) (layer "B.Cu") (net 6))
-  (segment (start 104.35 102.318604) (end 104.716396 102.685) (width 0.25) (layer "B.Cu") (net 6))
-  (segment (start 104.35 99.68934) (end 104.35 102.318604) (width 0.25) (layer "B.Cu") (net 6))
+  (segment (start 104.37 99.68934) (end 104.37 102.338604) (width 0.25) (layer "B.Cu") (net 6))
+  (segment (start 104.716396 102.685) (end 105.538878 102.685) (width 0.25) (layer "B.Cu") (net 6))
   (segment (start 105.538878 102.685) (end 106.538878 103.685) (width 0.25) (layer "B.Cu") (net 6))
-  (segment (start 102.815 99.25) (end 103.91066 99.25) (width 0.25) (layer "B.Cu") (net 6))
+  (segment (start 102.815 99.25) (end 103.93066 99.25) (width 0.25) (layer "B.Cu") (net 6))
+  (segment (start 103.93066 99.25) (end 104.37 99.68934) (width 0.25) (layer "B.Cu") (net 6))
+  (segment (start 104.37 102.338604) (end 104.716396 102.685) (width 0.25) (layer "B.Cu") (net 6))
   (segment (start 102.7 99.365) (end 102.815 99.25) (width 0.25) (layer "B.Cu") (net 6))
-  (segment (start 104.716396 102.685) (end 105.538878 102.685) (width 0.25) (layer "B.Cu") (net 6))
   (segment (start 107.62 102.4385) (end 107.6575 102.476) (width 0.25) (layer "F.Cu") (net 7))
   (segment (start 107.6575 102.476) (end 108.89 102.476) (width 0.25) (layer "F.Cu") (net 7))
   (segment (start 105.08 97.463) (end 105.08 96.315) (width 0.25) (layer "F.Cu") (net 8))
+  (segment (start 109.38 100.015) (end 110 100.635) (width 0.25) (layer "B.Cu") (net 8))
+  (segment (start 108.825 99.82462) (end 109.01538 100.015) (width 0.25) (layer "B.Cu") (net 8))
+  (segment (start 108.375 97.706396) (end 108.375 98.741016) (width 0.25) (layer "B.Cu") (net 8))
+  (segment (start 105.08 96.315) (end 106.161122 96.315) (width 0.25) (layer "B.Cu") (net 8))
+  (segment (start 108.375 98.741016) (end 108.825 99.191016) (width 0.25) (layer "B.Cu") (net 8))
+  (segment (start 107.17 97.323878) (end 107.992482 97.323878) (width 0.25) (layer "B.Cu") (net 8))
+  (segment (start 109.01538 100.015) (end 109.38 100.015) (width 0.25) (layer "B.Cu") (net 8))
   (segment (start 107.992482 97.323878) (end 108.375 97.706396) (width 0.25) (layer "B.Cu") (net 8))
-  (segment (start 108.375 97.706396) (end 108.375 98.741016) (width 0.25) (layer "B.Cu") (net 8))
-  (segment (start 109.38 100.015) (end 110 100.635) (width 0.25) (layer "B.Cu") (net 8))
   (segment (start 106.161122 96.315) (end 107.17 97.323878) (width 0.25) (layer "B.Cu") (net 8))
   (segment (start 108.825 99.191016) (end 108.825 99.82462) (width 0.25) (layer "B.Cu") (net 8))
-  (segment (start 109.01538 100.015) (end 109.38 100.015) (width 0.25) (layer "B.Cu") (net 8))
-  (segment (start 105.08 96.315) (end 106.161122 96.315) (width 0.25) (layer "B.Cu") (net 8))
-  (segment (start 107.17 97.323878) (end 107.992482 97.323878) (width 0.25) (layer "B.Cu") (net 8))
-  (segment (start 108.825 99.82462) (end 109.01538 100.015) (width 0.25) (layer "B.Cu") (net 8))
-  (segment (start 108.375 98.741016) (end 108.825 99.191016) (width 0.25) (layer "B.Cu") (net 8))
   (segment (start 107.62 97.463) (end 107.62 96.315) (width 0.25) (layer "F.Cu") (net 9))
   (segment (start 110 99.365) (end 109.38 98.745) (width 0.25) (layer "B.Cu") (net 9))

Commit message: -
Other:
- board text added: "t85 Micronucleus"
- board text removed: "ATtiny85 USB-C"
Changed lines of the file:
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@@
     (effects (font (size 0.9 0.9) (thickness 0.18) bold) (justify mirror))
   )
-  (gr_text "ATtiny85 USB-C" (at 100.635 100 90) (layer "F.Mask")
+  (gr_text "t85 Micronucleus" (at 100.635 100 90) (layer "F.Mask")
     (effects (font (size 0.5 0.5) (thickness 0.1) bold))
   )

Commit message: -
Parts:
- added G***: LOGO, LOGO, F.Cu at (105.5, 101.4)
- added G***: LOGO, LOGO, F.Cu at (113.3, 100.0)
