File: t202/t202.kicad_pcb (KiCad board)
At the start: 2 copper layers, 23 x 12.2 mm, 7 parts, among them J1 Conn_02x04_Counter_Clockwise, SW1 SW_Push, U1 ATtiny202-SS

Commit message: -
Parts:
- removed U2: ~, Library:PCB_USB_Conn
- added C2: 0u1, Capacitor_SMD:C_0603_1608Metric_Pad1.08x0.95mm_HandSolder, B.Cu at (120.3, 102.9)
- added C3: 1.5F, Library:ELDC_v, B.Cu at (123.7, 100.0)
- added J2: ~, Library:PCB_USB_Conn, F.Cu at (100.0, 100.0)
- added JP1: SolderJumper_2_Open, Library:sop_jumper, F.Cu at (116.2, 102.4)
- added SW2: SW_SPDT, Library:3pad_2.5_h, F.Cu at (119.8, 93.9)
- added U3: CH340K, Package_SO:SSOP-10_3.9x4.9mm_P1.00mm, B.Cu at (115.2, 101.1)
- C1: value C -> 0u1
- SW1: footprint Library:THAF01-NC-R -> Library:TVAF06-A020B-R; moved to F.Cu
- moved SW1 9.92 mm to (120.6, 106.0), turned to 90 degrees
- moved D1 7.09 mm to (113.6, 95.0), turned to 180 degrees
- moved U1 4.98 mm to (115.6, 101.1)
- moved J1 4.98 mm to (113.5, 104.9)
- moved R1 4.93 mm to (113.6, 95.0), turned to 180 degrees
- moved C1 4.46 mm to (118.5, 95.6)
Routing:
- net +5V: track 15.3 -> 27.6 mm
- net Net-(SW2-C): track 0.00 -> 9.65 mm
- net Net-(J2-D+): track 0.00 -> 9.20 mm, vias 0 -> 1
- net GND: track 9.82 -> 4.46 mm, vias 7 -> 6
- net Net-(J2-D-): track 0.00 -> 5.06 mm, vias 0 -> 1
- net Net-(J1-Pin_3): track 11.1 -> 6.72 mm, vias 1 -> 0
- net Net-(J1-Pin_7): track 4.51 -> 7.18 mm, vias 1 -> 0
- net Net-(D1-A): track 2.42 -> 0.00 mm
- net Net-(U3-V3): track 0.00 -> 1.72 mm
- net Net-(J1-Pin_5): track 8.52 -> 9.57 mm, vias 0 -> 1
- net Net-(J1-Pin_6): track 5.62 -> 5.94 mm, vias 0 -> 2
Other:
- board size 23 x 12.2 mm -> 24.2 x 12.2 mm
- board text added: "ATTiny~02 w/ serialupdi"
- board text added: "VG 63 70 12"
- board text added: "VG NN NT NR"
- board text added: "Vbat"
- board text removed: "0"
- board text removed: "1"
- board text removed: "2"
- board text removed: "3"
- board text removed: "6"
- board text removed: "7"
- board text removed: "V"

Commit message: -
Routing:
- net GND: vias 6 -> 7

Commit message: -
Other:
- board text added: "8p tinyAVR w/ serialupdi"
- board text removed: "ATTiny~02 w/ serialupdi"

Commit message: -
Other:
- board text added: "tinyAVR serialupdi"
- board text removed: "8p tinyAVR w/ serialupdi"

Commit message: -
Parts:
- moved C2 0.70 mm to (121.0, 102.9)
- moved SW1 0.22 mm to (120.4, 106.1)
- moved JP1 0.21 mm to (116.4, 102.3)
Connections:
- net Net-(J1-Pin_2) renamed PA6
- net Net-(J1-Pin_3) renamed PA7
- net Net-(J1-Pin_4) renamed PA1
- net Net-(J1-Pin_5) renamed PA2
- net Net-(J1-Pin_7) renamed PA3
- net Net-(J2-D+) renamed D+
- net Net-(J2-D-) renamed D-
- J1 pad 6: Net-(J1-Pin_6) -> PA0
- JP1 pad 2: Net-(J1-Pin_6) -> Net-(JP1-B)
- U1 pad 6: Net-(J1-Pin_6) -> PA0
- U3 pad 8: Net-(J1-Pin_6) -> Net-(JP1-B)
- U3 pad 9: Net-(J1-Pin_6) -> PA0
Routing:
- net D-: track 5.06 -> 12.5 mm
- net Net-(J1-Pin_6): track 5.94 -> 0.00 mm, vias 2 -> 0
- net GND: track 4.46 -> 9.96 mm, vias 7 -> 8
- net PA0: track 0.00 -> 5.50 mm, vias 0 -> 1
- net PA2: track 9.57 -> 7.65 mm
- net Net-(JP1-B): track 0.00 -> 1.69 mm, vias 0 -> 1
- net Net-(U3-V3): track 1.72 -> 2.42 mm
Other:
- board text added: "2T"
- board text added: "TR"
- board text removed: "VG NN NT NR"

Commit message: -
Parts:
- removed JP1: SolderJumper_2_Open, Library:sop_jumper
- removed U3: CH340K, Package_SO:SSOP-10_3.9x4.9mm_P1.00mm
- added R5: 5k1, Resistor_SMD:R_0603_1608Metric, B.Cu at (100.6, 98.3)
- added R6: 5k1, Resistor_SMD:R_0603_1608Metric, B.Cu at (100.6, 101.7)
- added U2: CH340K, Package_SO:SSOP-10_3.9x4.9mm_P1.00mm, F.Cu at (107.6, 100.0)
- C1: value 0u1 -> 4u7; footprint Capacitor_SMD:C_0603_1608Metric_Pad1.08x0.95mm_HandSolder -> Capacitor_SMD:C_0603_1608Metric
- C2: value 0u1 -> 1F5; footprint Capacitor_SMD:C_0603_1608Metric_Pad1.08x0.95mm_HandSolder -> Library:edlc; moved to F.Cu
- C3: value 1.5F -> 0u1; footprint Library:ELDC_v -> Capacitor_SMD:C_0603_1608Metric
- D1: footprint LED_SMD:LED_0603_1608Metric_Pad1.05x0.95mm_HandSolder -> LED_SMD:LED_0603_1608Metric; moved to B.Cu
- J1: value Conn_02x04_Counter_Clockwise -> USB-C; footprint Package_DIP:DIP-8_W7.62mm -> Library:USB-C
- J2: value ~ -> OUT; footprint Library:PCB_USB_Conn -> Package_DIP:DIP-8_W7.62mm_Socket
- R1: footprint Resistor_SMD:R_0603_1608Metric_Pad0.98x0.95mm_HandSolder -> Resistor_SMD:R_0603_1608Metric
- SW1: footprint Library:TVAF06-A020B-R -> Library:sw_push_smd
- SW2: footprint Library:3pad_2.5_h -> Library:sw
- U1: moved to B.Cu
- moved SW1 18.7 mm to (102.7, 100.0), turned to -90 degrees
- moved J1 14.3 mm to (100.0, 100.0), turned to 180 degrees
- moved C3 13.6 mm to (110.2, 98.1), turned to 180 degrees
- moved J2 10.9 mm to (110.2, 96.2), turned to -90 degrees
- moved U1 10.6 mm to (105.1, 100.0)
- moved C1 9.76 mm to (110.8, 101.6), turned to -90 degrees
- moved R1 7.75 mm to (109.5, 101.6), turned to -90 degrees
- moved SW2 6.15 mm to (119.0, 100.0), turned to 0 degrees
- moved D1 5.56 mm to (110.2, 99.4)
- moved C2 5.35 mm to (116.5, 100.0), turned to 180 degrees
Connections:
- C1 pad 1: +5V -> VCC
- C2 pad 1: Net-(U3-V3) -> /Vedlc
- C3 pad 1: Net-(SW2-C) -> Net-(U2-V3)
- D1 pad 1: GND -> Net-(D1-K)
- D1 pad 2: Net-(D1-A) -> PA3
- J1 pad 1: +5V -> GND
- J1 pad 2: PA6 -> D+
- J1 pad 3: PA7 -> D-
- J1 pad 4: PA1 -> VCC
- J1 pad 5: PA2 -> Net-(J1-CC1)
- J1 pad 6: PA0 -> Net-(J1-CC2)
- J2 pad 1: GND -> VCC
- J2 pad 2: D+ -> PA6
- J2 pad 3: D- -> PA7
- J2 pad 4: +5V -> PA1
- J2 pad 5: GND -> PA2
- J2 pad 6: GND -> UPDI
- R1 pad 1: PA3 -> Net-(D1-K)
- R1 pad 2: Net-(D1-A) -> GND
- SW1 pad 1: PA7 -> GND
- SW1 pad 2: GND -> PA7
- SW2 pad 1: +5V -> VCC
- SW2 pad 2: +5V -> VCC
- SW2 pad 3: Net-(SW2-C) -> /Vedlc
- U1 pad 1: +5V -> VCC
- U1 pad 6: PA0 -> UPDI
Routing:
- net +5V: track 27.6 -> 0.00 mm, vias 1 -> 0
- net VCC: track 0.00 -> 23.5 mm, vias 0 -> 6
- net GND: track 9.96 -> 23.8 mm, vias 8 -> 6
- net Net-(SW2-C): track 9.65 -> 0.00 mm
- net UPDI: track 0.00 -> 9.41 mm, vias 0 -> 1
- net PA1: track 8.73 -> 1.81 mm, vias 1 -> 0
- net PA0: track 5.50 -> 0.00 mm, vias 1 -> 0
- net D+: track 8.95 -> 13.2 mm
- net Net-(J1-CC2): track 0.00 -> 3.55 mm
- net Net-(J1-CC1): track 0.00 -> 3.55 mm, vias 0 -> 1
- net /Vedlc: track 0.00 -> 2.54 mm
- net Net-(U3-V3): track 2.42 -> 0.00 mm
- net D-: track 12.5 -> 10.4 mm
- net Net-(D1-K): track 0.00 -> 2.08 mm
- net Net-(JP1-B): track 1.69 -> 0.00 mm, vias 1 -> 0
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- added copper zone on B.Cu, net VCC
- added copper zone on F.Cu, net VCC
Other:
- board size 24.2 x 12.2 mm -> 21.6 x 7.6 mm
- board text added: "ATtiny202 USB-C"
- board text removed: "2T"
- board text removed: "G"
- board text removed: "TR"
- board text removed: "VG 63 70 12"
- board text removed: "Vbat"
- board text removed: "tinyAVR serialupdi"

Commit message: -
Routing:
- net VCC: vias 6 -> 7
- net GND: vias 6 -> 7
Changed lines of the file:
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@@
   (segment (start 100.635 102.476) (end 101.206 102.476) (width 0.375) (layer "F.Cu") (net 1))
   (segment (start 101.206 102.476) (end 101.27 102.54) (width 0.375) (layer "F.Cu") (net 1))
+  (via (at 110.795 103.175) (size 0.8) (drill 0.4) (layers "F.Cu" "B.Cu") (free) (net 1))
   (via (at 109.1705 98.095) (size 0.5) (drill 0.3) (layers "F.Cu" "B.Cu") (net 1))
   (via (at 100.635 102.476) (size 0.8) (drill 0.4) (layers "F.Cu" "B.Cu") (net 1))
@@
   (via (at 96.5 98.5) (size 0.5) (drill 0.3) (layers "F.Cu" "B.Cu") (net 13))
   (via (at 98.25 98.5) (size 0.5) (drill 0.3) (layers "F.Cu" "B.Cu") (net 13))
+  (via (at 110.795 96.825) (size 0.8) (drill 0.4) (layers "F.Cu" "B.Cu") (net 13))
   (segment (start 116.51 102.5) (end 119.05 102.5) (width 0.375) (layer "F.Cu") (net 14))
   (segment (start 108.255 99) (end 110.17 99) (width 0.25) (layer "F.Cu") (net 15))

Commit message: -
Other:
- board text added: "t202 SerialUPDI"
- board text removed: "ATtiny202 USB-C"
Changed lines of the file:
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@@
     (effects (font (size 0.9 0.9) (thickness 0.18) bold) (justify mirror))
   )
-  (gr_text "ATtiny202 USB-C" (at 100.635 100 90) (layer "F.Mask")
+  (gr_text "t202 SerialUPDI" (at 100.635 100 90) (layer "F.Mask")
     (effects (font (size 0.5 0.5) (thickness 0.1) bold))
   )
