File: esp32c3-mini-1/esp32c3-mini-1.kicad_pcb (KiCad board)
At the start: 2 copper layers, 12.2 x 10.2 mm, 7 parts, among them J1 USB-C, U1 ESP32C3, U2 LM1117MP-3.3, U3 WS2812C

Commit message: -
Parts:
- added G***: LOGO, LOGO, B.Cu at (103.0, 85.5)
- added G***: LOGO, LOGO, B.Cu at (97.0, 85.5)
- R1, R2, R3, U2, U3: moved to B.Cu
- moved U3 75.8 mm to (96.5, 96.8)
- moved R1 71.8 mm to (96.5, 94.8), turned to 180 degrees
- moved J1 69.1 mm to (100.0, 100.0), turned to -90 degrees
- moved R3 68.4 mm to (99.8, 96.5)
- moved R2 65.6 mm to (102.8, 96.5), turned to 180 degrees
- moved U1 53.8 mm to (100.0, 93.9)
- moved U2 49.2 mm to (100.8, 92.0), turned to 180 degrees
Routing:
- net +5V: track 0.00 -> 19.3 mm, vias 0 -> 5
- net D+: track 0.00 -> 16.8 mm, vias 0 -> 1
- net D-: track 0.00 -> 11.8 mm, vias 0 -> 1
- net Net-(J1-CC2): track 0.00 -> 11.0 mm, vias 0 -> 2
- net GND: track 0.00 -> 6.78 mm, vias 0 -> 7
- net Net-(J1-CC1): track 0.00 -> 6.37 mm, vias 0 -> 1
- net Net-(R1-Pad2): track 0.00 -> 1.86 mm
- net NPDI: track 0.00 -> 1.61 mm
- added copper zone on B.Cu, net +3.3V
- added copper zone on B.Cu, net GND
- added copper zone on F.Cu, net GND
Other:
- board size 12.2 x 10.2 mm -> 14 x 17.5 mm

Commit message: -
Parts:
- removed G*** (x2): LOGO, LOGO
- added J2: Conn_02x08_Counter_Clockwise, Package_DIP:DIP-16_W7.62mm, F.Cu at (96.2, 101.3)
- R1, R2, R3, U2, U3: moved to F.Cu
- U1: footprint Library:ESP32C3-MINI-1_THT -> Library:ESP32C3-MINI-1
- moved U3 37.4 mm to (125.9, 73.6)
- moved R1 33.4 mm to (122.2, 73.3), turned to 0 degrees
- moved R3 28.8 mm to (122.2, 78.3)
- moved R2 28.4 mm to (122.2, 75.8), turned to 0 degrees
- moved J1 20.8 mm to (100.0, 120.8)
- moved U2 19.9 mm to (120.3, 88.6), turned to 0 degrees
- moved U1 0.24 mm to (100.0, 94.1)
Connections:
- net NPDI renamed IO0
- U1 pad 1: unconnected-(U1-IO1-Pad1) -> IO1
- U1 pad 10: unconnected-(U1-IO10-Pad10) -> IO10
- U1 pad 2: unconnected-(U1-IO2-Pad2) -> IO2
- U1 pad 20: unconnected-(U1-RXD-Pad20) -> RXD
- U1 pad 21: unconnected-(U1-TXD-Pad21) -> TXD
- U1 pad 3: unconnected-(U1-IO3-Pad3) -> IO3
- U1 pad 4: unconnected-(U1-IO4-Pad4) -> IO4
- U1 pad 5: unconnected-(U1-IO5-Pad5) -> IO5
- U1 pad 6: unconnected-(U1-IO6-Pad6) -> IO6
- U1 pad 7: unconnected-(U1-IO7-Pad7) -> IO7
- U1 pad 8: unconnected-(U1-IO8-Pad8) -> IO8
- U1 pad 9: unconnected-(U1-IO9-Pad9) -> IO9
Routing:
- net +5V: track 19.3 -> 0.00 mm, vias 5 -> 0
- net D+: track 16.8 -> 0.00 mm, vias 1 -> 0
- net D-: track 11.8 -> 0.00 mm, vias 1 -> 0
- net Net-(J1-CC2): track 11.0 -> 0.00 mm, vias 2 -> 0
- net GND: track 6.78 -> 0.00 mm, vias 7 -> 0
- net Net-(J1-CC1): track 6.37 -> 0.00 mm, vias 1 -> 0
- net Net-(R1-Pad2): track 1.86 -> 0.00 mm
- net IO0: track 1.61 -> 0.00 mm
- removed copper zone on B.Cu, net +3.3V
- removed copper zone on B.Cu, net GND
- removed copper zone on F.Cu, net GND
Other:
- board size 14 x 17.5 mm -> 6.7 x 4.5 mm

Commit message: -
Parts:
- added ?: , clipboard:0cc91ec2-0069-494b-bf66-8693916d34c6, F.Cu at (100.0, 89.8)
- J2: footprint Package_DIP:DIP-16_W7.62mm -> Package_DIP:DIP-16_W10.16mm
- moved R3 30.2 mm to (98.7, 97.5), turned to 90 degrees
- moved R2 30.1 mm to (101.3, 97.5), turned to 90 degrees
- moved U3 26.9 mm to (100.0, 81.0)
- moved R1 25.8 mm to (97.5, 81.0), turned to 90 degrees
- moved J1 20.8 mm to (100.0, 100.0)
- moved J2 20.4 mm to (94.9, 81.0)
- moved U2 20.4 mm to (100.0, 87.3), turned to 90 degrees
- moved U1 20.3 mm to (100.0, 73.8)
Other:
- board size 6.7 x 4.5 mm -> 14 x 37.5 mm
- board text added: "G T R 9 8 7 6 5"
- board text added: "V E 2 3 0 1 a 4"

Commit message: -
Parts:
- added G***: LOGO, LOGO, B.Cu at (97.5, 70.8)
- added G***: LOGO, LOGO, B.Cu at (102.5, 70.8)
- added J3: Conn_01x01_Pin, Connector_PinHeader_2.54mm:PinHeader_1x01_P2.54mm_Vertical, F.Cu at (100.0, 96.2)
- moved U3 1.91 mm to (101.9, 81.0)
- moved R2 1.27 mm to (102.5, 97.5)
- moved R3 1.27 mm to (97.5, 97.5)
- moved R1 0.90 mm to (98.1, 81.6), turned to 180 degrees
- moved U2 0.63 mm to (100.0, 86.7)
- moved U1 0.18 mm to (100.0, 73.6)
Connections:
- R1 pad 2: Net-(R1-Pad2) -> EN
- U1 pad EN: Net-(R1-Pad2) -> EN
Routing:
- net D+: track 0.00 -> 38.4 mm, vias 0 -> 2
- net D-: track 0.00 -> 34.7 mm, vias 0 -> 2
- net +5V: track 0.00 -> 28.6 mm, vias 0 -> 5
- net IO0: track 0.00 -> 25.5 mm, vias 0 -> 1
- net IO4: track 0.00 -> 25.2 mm, vias 0 -> 1
- net IO5: track 0.00 -> 24.6 mm, vias 0 -> 1
- net IO6: track 0.00 -> 20.7 mm, vias 0 -> 1
- net IO10: track 0.00 -> 20.7 mm, vias 0 -> 1
- net IO1: track 0.00 -> 20.4 mm, vias 0 -> 1
- net IO7: track 0.00 -> 19.0 mm, vias 0 -> 1
- net IO3: track 0.00 -> 18.1 mm, vias 0 -> 1
- net IO8: track 0.00 -> 17.4 mm, vias 0 -> 1
- net IO9: track 0.00 -> 15.9 mm, vias 0 -> 1
- net RXD: track 0.00 -> 15.1 mm, vias 0 -> 1
- net IO2: track 0.00 -> 15.1 mm, vias 0 -> 1
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- added copper zone on B.Cu, net +3.3V
- added copper zone on F.Cu, net +3.3V
- added copper zone on B.Cu, net GND
- added copper zone on F.Cu, net GND
Other:
- board size 14 x 37.5 mm -> 12.7 x 31.8 mm
- board text added: "Vin"
