File: c3-mini/c3-mini.kicad_sch (KiCad schematic)
At the start: 9 parts, among them J1 USB-C, J2 Conn_02x08_Counter_Clockwise, J3 Conn_01x01_Pin, U2 LM1117MP-3.3, U3 WS2812C, U4 ESP32-C3-MINI-1

Commit message: -
Parts:
- removed J2: Conn_02x08_Counter_Clockwise, Package_DIP:DIP-16_W10.16mm, symbol Connector_Generic:Conn_02x08_Counter_Clockwise
- added J2, J4: Conn_01x08_Pin, Connector_PinHeader_2.54mm:PinHeader_1x08_P2.54mm_Vertical, symbol Connector:Conn_01x08_Pin
Connections:
- net +3.3V: now also J2.1 (Pin_1)
- net EN: now also J2.2 (Pin_2)
- net GND: now also J4.1 (Pin_1)
- net IO0: now also J2.5 (Pin_5); no longer U3.3 (DI)
- net IO1: now also J2.6 (Pin_6)
- net IO10: now also J2.7 (Pin_7)
- net IO2: now also J2.3 (Pin_3)
- net IO3: now also J2.4 (Pin_4)
- net IO4: now also J2.8 (Pin_8)
- net IO5: now also J4.8 (Pin_8)
- net IO6: now also J4.7 (Pin_7)
- net IO7: now also J4.6 (Pin_6)
- net IO8: now also U3.3 (DI), J4.5 (Pin_5)
- net IO9: now also J4.4 (Pin_4)
- net RXD: now also J4.3 (Pin_3)
- net TXD: now also J4.2 (Pin_2)
