File: c3-mini/c3-mini.kicad_pcb (KiCad board)
At the start: 2 copper layers, 12.7 x 31.8 mm, 12 parts, among them J1 USB-C, J2 Conn_02x08_Counter_Clockwise, J3 Conn_01x01_Pin, U2 LM1117MP-3.3, U3 WS2812C, U4 ESP32-C3-MINI-1

Commit message: -
Parts:
- added J4: Conn_01x08_Pin, Connector_PinHeader_2.54mm:PinHeader_1x08_P2.54mm_Vertical, F.Cu at (105.1, 81.0)
- J2: value Conn_02x08_Counter_Clockwise -> Conn_01x08_Pin; footprint Package_DIP:DIP-16_W10.16mm -> Connector_PinHeader_2.54mm:PinHeader_1x08_P2.54mm_Vertical
Connections:
- U3 pad 3: IO0 -> IO8
Routing:
- net IO0: track 25.5 -> 18.7 mm
- net IO8: track 17.4 -> 21.0 mm

Commit message: -
Routing:
- net GND: vias 31 -> 32
Other:
- board text added: "JLCJLCJLCJLC"
Changed lines of the file:
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@@
     (effects (font (size 0.79 0.79) (thickness 0.158) bold) (justify bottom))
+  )
+  (gr_text "JLCJLCJLCJLC" (at 100 70.79) (layer "F.SilkS")
+    (effects (font (size 1 1) (thickness 0.2) bold) (justify bottom))
   )
   (segment (start 97.25 99.75) (end 97.25 102.81) (width 0.25) (layer "F.Cu") (net 1))
@@
   (via (at 101.975 73.6) (size 0.8) (drill 0.4) (layers "F.Cu" "B.Cu") (net 1))
   (via (at 98.4 68.7) (size 0.5) (drill 0.3) (layers "F.Cu" "B.Cu") (net 1))
+  (via (at 99.37 93.65) (size 0.5) (drill 0.3) (layers "F.Cu" "B.Cu") (net 1))
   (via (at 94 99.75) (size 0.5) (drill 0.3) (layers "F.Cu" "B.Cu") (net 1))
   (via (at 100 97.640003) (size 0.8) (drill 0.4) (layers "F.Cu" "B.Cu") (free) (net 1))
@@
   (via (at 100 71.625) (size 0.8) (drill 0.4) (layers "F.Cu" "B.Cu") (net 1))
   (via (at 99.83 80) (size 0.5) (drill 0.3) (layers "F.Cu" "B.Cu") (net 1))
-  (via (at 99.68 87.5) (size 0.8) (drill 0.4) (layers "F.Cu" "B.Cu") (free) (net 1))
+  (via (at 99.68 87.3) (size 0.8) (drill 0.4) (layers "F.Cu" "B.Cu") (free) (net 1))
   (via (at 101.6 68.7) (size 0.5) (drill 0.3) (layers "F.Cu" "B.Cu") (net 1))
   (via (at 96.82 87.481782) (size 0.5) (drill 0.3) (layers "F.Cu" "B.Cu") (net 1))

Commit message: -
Routing:
- net IO5: track 25.0 -> 23.9 mm
- net IO8: track 21.0 -> 20.3 mm
- net IO7: track 19.2 -> 18.6 mm
- net IO4: track 25.2 -> 24.6 mm
- net IO6: track 20.8 -> 20.2 mm
- net IO10: track 20.7 -> 20.1 mm
- net GND: vias 32 -> 30

Commit message: -
Changed lines of the file:
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@@
   (via (at 99.5 100.75) (size 0.5) (drill 0.3) (layers "F.Cu" "B.Cu") (net 2))
   (via (at 104.25 75.25) (size 0.5) (drill 0.3) (layers "F.Cu" "B.Cu") (net 2))
-  (segment (start 100.25 103.464386) (end 99.964386 103.75) (width 0.2) (layer "B.Cu") (net 2))
   (segment (start 100.7 99.55) (end 100.7 97.116346) (width 0.2) (layer "B.Cu") (net 2))
-  (segment (start 99.325 100.925) (end 99.5 100.75) (width 0.2) (layer "B.Cu") (net 2))
-  (segment (start 100.25 102.535) (end 100.25 103.464386) (width 0.2) (layer "B.Cu") (net 2))
   (segment (start 100.856496 76.3) (end 101.856496 76.3) (width 0.2) (layer "B.Cu") (net 2))
-  (segment (start 99.5 103.75) (end 99.325 103.575) (width 0.2) (layer "B.Cu") (net 2))
   (segment (start 99.5 100.75) (end 100.7 99.55) (width 0.2) (layer "B.Cu") (net 2))
   (segment (start 100.3 76.856497) (end 100.856496 76.3) (width 0.2) (layer "B.Cu") (net 2))
-  (segment (start 99.964386 103.75) (end 99.5 103.75) (width 0.2) (layer "B.Cu") (net 2))
-  (segment (start 99.325 103.575) (end 99.325 100.925) (width 0.2) (layer "B.Cu") (net 2))
   (segment (start 100.7 97.116346) (end 101.15 96.666346) (width 0.2) (layer "B.Cu") (net 2))
   (segment (start 100.3 78.279899) (end 100.3 76.856497) (width 0.2) (layer "B.Cu") (net 2))
   (segment (start 100.38 78.359899) (end 100.3 78.279899) (width 0.2) (layer "B.Cu") (net 2))
+  (segment (start 100.25 102.535) (end 100.25 103.3) (width 0.2) (layer "B.Cu") (net 2))
   (segment (start 101.856496 76.3) (end 102.956496 75.2) (width 0.2) (layer "B.Cu") (net 2))
+  (segment (start 99.25 103.3) (end 99.25 101) (width 0.2) (layer "B.Cu") (net 2))
   (segment (start 101.15 96.666346) (end 101.15 95.713654) (width 0.2) (layer "B.Cu") (net 2))
   (segment (start 104.2 75.2) (end 104.25 75.25) (width 0.2) (layer "B.Cu") (net 2))
   (segment (start 101.15 95.713654) (end 100.38 94.943654) (width 0.2) (layer "B.Cu") (net 2))
+  (segment (start 99.75 103.8) (end 99.75 103.8) (width 0.2) (layer "B.Cu") (net 2))
+  (segment (start 99.25 101) (end 99.5 100.75) (width 0.2) (layer "B.Cu") (net 2))
   (segment (start 100.38 94.943654) (end 100.38 78.359899) (width 0.2) (layer "B.Cu") (net 2))
   (segment (start 102.956496 75.2) (end 104.2 75.2) (width 0.2) (layer "B.Cu") (net 2))
+  (arc (start 99.75 103.8) (mid 99.396447 103.653553) (end 99.25 103.3) (width 0.2) (layer "B.Cu") (net 2))
+  (arc (start 99.75 103.8) (mid 100.103553 103.653553) (end 100.25 103.3) (width 0.2) (layer "B.Cu") (net 2))
   (segment (start 105.9 76.8) (end 104.8 76.8) (width 0.2) (layer "F.Cu") (net 3))
   (segment (start 104.8 76.8) (end 103.75 75.75) (width 0.2) (layer "F.Cu") (net 3))

Commit message: -
Routing:
- net D+: track 38.4 -> 3.39 mm, vias 2 -> 1
- net D-: track 34.7 -> 3.87 mm, vias 2 -> 1
- net IO9: track 15.6 -> 17.4 mm
- net IO8: track 20.3 -> 21.9 mm
- net IO7: track 18.6 -> 19.9 mm
- net IO4: track 24.6 -> 25.8 mm
- net IO5: track 23.9 -> 25.1 mm
- net IO0: track 18.3 -> 19.3 mm
- net IO10: track 20.1 -> 21.0 mm
- net IO6: track 20.2 -> 20.9 mm
- net IO3: track 17.8 -> 17.1 mm
- net RXD: track 14.9 -> 15.5 mm
- net GND: vias 30 -> 23

Commit message: -
Parts:
- moved R2 1.73 mm to (101.8, 99.0), turned to 0 degrees
- moved R3 1.73 mm to (98.2, 99.0), turned to 180 degrees
- moved U3 0.08 mm to (101.9, 81.0)
Routing:
- net D+: track 3.39 -> 39.2 mm, vias 1 -> 2
- net D-: track 3.87 -> 35.6 mm, vias 1 -> 2
- net +5V: track 28.6 -> 30.5 mm, vias 5 -> 4
- net Net-(J1-CC2): track 4.99 -> 3.75 mm
- net Net-(J1-CC1): track 4.99 -> 3.75 mm
- net +3.3V: track 7.77 -> 7.27 mm
- net GND: vias 23 -> 20

Commit message: -
Parts:
- moved U3 0.08 mm to (101.9, 81.0)
Routing:
- net +5V: track 30.5 -> 31.2 mm
- net GND: vias 20 -> 30
