File: c3-wroom/c3-wroom.kicad_pcb (KiCad board)
At the start: 2 copper layers, 20.3 x 34.3 mm, 13 parts, among them J1 USB-C, J2 Conn_01x08_Pin, J3 Conn_01x01_Pin, J4 Conn_01x08_Pin, U1 ESP32-C3-WROOM-02, U2 LM1117MP-3.3, U3 WS2812C

Commit message: -
Parts:
- moved R2 0.25 mm to (101.8, 94.5)
- moved R3 0.25 mm to (98.2, 94.5)
Routing:
- net D+: track 3.68 -> 35.6 mm, vias 1 -> 2
- net D-: track 3.68 -> 34.3 mm, vias 1 -> 2
- net +5V: track 11.0 -> 30.7 mm
- net GND: track 0.00 -> 11.2 mm, vias 8 -> 15
- net Net-(J1-CC1): track 0.00 -> 3.92 mm
- net Net-(J1-CC2): track 0.00 -> 3.92 mm, vias 0 -> 1

Commit message: -
Routing:
- net +5V: track 30.7 -> 29.4 mm
- net D+: track 35.6 -> 34.4 mm
- net D-: track 34.3 -> 33.2 mm
- net GND: track 11.2 -> 12.2 mm, vias 15 -> 23
Other:
- board text added: "G 0 1 2 3 R T a"
- board text added: "V E 4 5 6 7 8 9"
- board text removed: "G T R 9 8 7 6 5"
- board text removed: "V E 2 3 0 1 a 4"

Commit message: -
Parts:
- moved G*** 2.54 mm to (97.5, 68.2)
- moved G*** 2.54 mm to (102.5, 68.2)
Routing:
- net GND: vias 23 -> 27
Changed lines of the file:
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@@
   )
   (footprint "LOGO" (layer "B.Cu")
-    (at 97.46 70.79 180)
+    (at 97.46 68.25 180)
     (attr board_only exclude_from_pos_files exclude_from_bom)
     (fp_text reference "G***" (at 0 0) (layer "B.SilkS") hide
@@
   )
   (footprint "LOGO" (layer "B.Cu")
-    (at 102.54 70.79 180)
+    (at 102.54 68.25 180)
     (attr board_only exclude_from_pos_files exclude_from_bom)
     (fp_text reference "G***" (at 0 0) (layer "B.SilkS") hide
@@
   (via (at 109.75 99.75) (size 0.5) (drill 0.3) (layers "F.Cu" "B.Cu") (net 1))
   (via (at 106.720648 91.753297) (size 0.5) (drill 0.3) (layers "F.Cu" "B.Cu") (net 1))
+  (via (at 100.91 71.26) (size 0.8) (drill 0.4) (layers "F.Cu" "B.Cu") (net 1))
+  (via (at 102.06 72.36) (size 0.8) (drill 0.4) (layers "F.Cu" "B.Cu") (net 1))
   (via (at 106.412484 93.855451) (size 0.5) (drill 0.3) (layers "F.Cu" "B.Cu") (net 1))
   (via (at 100 80.95) (size 0.8) (drill 0.4) (layers "F.Cu" "B.Cu") (free) (net 1))
@@
   (via (at 104.75 99.5) (size 0.5) (drill 0.3) (layers "F.Cu" "B.Cu") (net 1))
   (via (at 92.974757 89.628585) (size 0.5) (drill 0.3) (layers "F.Cu" "B.Cu") (net 1))
+  (via (at 99.86 72.36) (size 0.8) (drill 0.4) (layers "F.Cu" "B.Cu") (net 1))
   (via (at 93.286388 91.727766) (size 0.5) (drill 0.3) (layers "F.Cu" "B.Cu") (net 1))
   (via (at 95.25 99.5) (size 0.5) (drill 0.3) (layers "F.Cu" "B.Cu") (net 1))
+  (via (at 100.91 73.46) (size 0.8) (drill 0.4) (layers "F.Cu" "B.Cu") (net 1))
   (via (at 97.5 99.25) (size 0.5) (drill 0.3) (layers "F.Cu" "B.Cu") (net 1))
   (via (at 102.5 97.25) (size 0.5) (drill 0.3) (layers "F.Cu" "B.Cu") (net 1))
