File: card-c3/card-c3.kicad_pcb (KiCad board)
At the start: 2 copper layers, 34.7 x 54.9 mm, 36 parts, among them J1 USB-C, J2 Conn_01x08_Pin, J3 Conn_01x01_Pin, J4 Conn_01x08_Pin, U1 ESP32-C3-WROOM-02, U2 LM1117MP-3.3, U3 WS2812C, U4 ESP32-C3-MINI-1

Commit message: -
Parts:
- added G***: LOGO, LOGO, B.Cu at (157.3, 112.7)
- added G***: LOGO, LOGO, B.Cu at (145.5, 110.2)
- added G***: LOGO, LOGO, B.Cu at (157.3, 125.0)
- added G***: LOGO, LOGO, B.Cu at (157.3, 107.7)
- added G***: LOGO, LOGO, B.Cu at (157.3, 142.3)
- added G***: LOGO, LOGO, B.Cu at (157.3, 147.3)
- added G***: LOGO, LOGO, B.Cu at (145.5, 148.0)
- added G***: LOGO, LOGO, B.Cu at (157.3, 130.0)
- added J1: USB-C, Library:USB-C, F.Cu at (186.5, 127.5)
- added J1: USB-C, Library:USB-C, F.Cu at (184.5, 110.2)
- added J1: USB-C, Library:USB-C, F.Cu at (184.5, 144.8)
- added J2: Conn_01x08_Pin, Connector_PinHeader_2.54mm:PinHeader_1x08_P2.54mm_Vertical, F.Cu at (167.4, 132.6)
- added J2: Conn_01x08_Pin, Connector_PinHeader_2.54mm:PinHeader_1x08_P2.54mm_Vertical, F.Cu at (170.0, 153.7)
- added J2: Conn_01x08_Pin, Connector_PinHeader_2.54mm:PinHeader_1x08_P2.54mm_Vertical, F.Cu at (170.0, 119.1)
- added J3: Conn_01x01_Pin, Connector_PinHeader_2.54mm:PinHeader_1x01_P2.54mm_Vertical, F.Cu at (180.1, 141.0)
- added J3: Conn_01x01_Pin, Connector_PinHeader_2.54mm:PinHeader_1x01_P2.54mm_Vertical, F.Cu at (182.7, 127.5)
- added J3: Conn_01x01_Pin, Connector_PinHeader_2.54mm:PinHeader_1x01_P2.54mm_Vertical, F.Cu at (180.2, 106.4)
- added J4: Conn_01x08_Pin, Connector_PinHeader_2.54mm:PinHeader_1x08_P2.54mm_Vertical, F.Cu at (167.4, 122.4)
- added J4: Conn_01x08_Pin, Connector_PinHeader_2.54mm:PinHeader_1x08_P2.54mm_Vertical, F.Cu at (170.0, 135.9)
- added J4: Conn_01x08_Pin, Connector_PinHeader_2.54mm:PinHeader_1x08_P2.54mm_Vertical, F.Cu at (170.0, 101.3)
- added R1: 10k, Resistor_SMD:R_0603_1608Metric, F.Cu at (170.0, 114.0)
- added R1: 10k, Resistor_SMD:R_0603_1608Metric, F.Cu at (170.0, 148.6)
- added R1: 10k, Resistor_SMD:R_0603_1608Metric, F.Cu at (168.1, 129.4)
- added R2: 5.1k, Resistor_SMD:R_0603_1608Metric, F.Cu at (185.5, 125.8)
- added R2: 5.1k, Resistor_SMD:R_0603_1608Metric, F.Cu at (183.5, 143.1)
- added R2: 5.1k, Resistor_SMD:R_0603_1608Metric, F.Cu at (183.5, 108.4)
- added R3: 5.1k, Resistor_SMD:R_0603_1608Metric, F.Cu at (185.5, 129.2)
- added R3: 5.1k, Resistor_SMD:R_0603_1608Metric, F.Cu at (183.5, 146.6)
- added R3: 5.1k, Resistor_SMD:R_0603_1608Metric, F.Cu at (183.5, 111.9)
- added U1: ESP32-C3-WROOM-02, PCM_Espressif:ESP32-C3-WROOM-02, F.Cu at (161.1, 144.8)
- added U1: ESP32-C3-WROOM-02, PCM_Espressif:ESP32-C3-WROOM-02, F.Cu at (161.1, 110.2)
- added U2: LM1117MP-3.3, Package_TO_SOT_SMD:SOT-223-3_TabPin2, F.Cu at (175.1, 144.8)
- added U2: LM1117MP-3.3, Package_TO_SOT_SMD:SOT-223-3_TabPin2, F.Cu at (175.1, 110.2)
- added U2: LM1117MP-3.3, Package_TO_SOT_SMD:SOT-223-3_TabPin2, F.Cu at (173.2, 127.5)
- added U3: WS2812C, Library:WS2812C-2020, F.Cu at (170.0, 107.7)
- added U3: WS2812C, Library:WS2812C-2020, F.Cu at (170.0, 142.3)
- added U3: WS2812C, Library:WS2812C-2020, F.Cu at (167.4, 125.6)
- added U4: ESP32-C3-MINI-1, PCM_Espressif:ESP32-C3-MINI-1, F.Cu at (157.4, 127.5)
Routing:
- net (no net): track 1291.9 -> 2583.8 mm, vias 156 -> 312
Other:
- board size 34.7 x 54.9 mm -> 87.1 x 54.9 mm
- board text added: "ESP32-C3-WROOM-02 *4 ESP32-C3-MINI-1 *2"
- board text added: "エリンギ @McbeEringi"
