File: tx04/tx04.kicad_pcb (KiCad board)
At the start: 2 copper layers, 25.4 x 10.2 mm, 17 parts, among them J1 USB_C_Receptacle_USB2.0_16P, J2 Conn_02x07_Counter_Clockwise, SW1 SW_Push, SW2 SW_SPDT, U1 ATtiny1604-SS, U2 CH340E, U3 TS5A23159DGS

Commit message: -
Parts:
- moved C3 3.81 mm to (108.3, 102.5), turned to 0 degrees
Connections:
- C3 pad 2: VCC -> GND
Routing:
- net Net-(U2-V3): track 1.57 -> 2.83 mm
Changed lines of the file:
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@@
 		(property ki_fp_filters "Connector*:*_2x??_*")
 		(sheetname "ルート")
-		(sheetfile "t1604.kicad_sch")
+		(sheetfile "tx04.kicad_sch")
 		(attr through_hole)
 		(fp_line
@@
 		(property ki_fp_filters "USB*C*Receptacle*")
 		(sheetname "ルート")
-		(sheetfile "t1604.kicad_sch")
+		(sheetfile "tx04.kicad_sch")
 		(attr smd)
 		(fp_line
@@
 		)
 		(sheetname "ルート")
-		(sheetfile "t1604.kicad_sch")
+		(sheetfile "tx04.kicad_sch")
 		(attr smd)
 		(fp_rect
@@
 		(property ki_fp_filters "SOIC*3.9x8.7mm*P1.27mm*")
 		(sheetname "ルート")
-		(sheetfile "t1604.kicad_sch")
+		(sheetfile "tx04.kicad_sch")
 		(attr smd)
 		(fp_line
@@
 		(property ki_fp_filters "LED* LED_SMD:* LED_THT:*")
 		(sheetname "ルート")
-		(sheetfile "t1604.kicad_sch")
+		(sheetfile "tx04.kicad_sch")
 		(attr smd)
 		(fp_line
@@
 		(property ki_fp_filters "C_*")
 		(sheetname "ルート")
-		(sheetfile "t1604.kicad_sch")
+		(sheetfile "tx04.kicad_sch")
 		(attr through_hole)
 		(fp_circle
@@
 		)
 		(sheetname "ルート")
-		(sheetfile "t1604.kicad_sch")
+		(sheetfile "tx04.kicad_sch")
 		(attr smd)
 		(fp_text user "${REFERENCE}"
@@
 		(property ki_fp_filters "R_*")
 		(sheetname "ルート")
-		(sheetfile "t1604.kicad_sch")
+		(sheetfile "tx04.kicad_sch")
 		(attr smd)
 		(fp_line
@@
 		(property ki_fp_filters "R_*")
 		(sheetname "ルート")
-		(sheetfile "t1604.kicad_sch")
+		(sheetfile "tx04.kicad_sch")
 		(attr smd)
 		(fp_line
@@
 		(tags "resistor")
 		(property "Reference" "R3"
-			(at 0 1.43 360)
+			(at 0 1.43 0)
 			(layer "B.SilkS")
 			(hide yes)
@@
 		)
 		(property "Value" "4.7k"
-			(at 0 -1.43 360)
+			(at 0 -1.43 0)
 			(layer "B.Fab")
 			(hide yes)
@@
 		(property ki_fp_filters "R_*")
 		(sheetname "ルート")
-		(sheetfile "t1604.kicad_sch")
+		(sheetfile "tx04.kicad_sch")
 		(attr smd)
 		(fp_line
@@
 		)
 		(fp_text user "${REFERENCE}"
-			(at 0 0 360)
+			(at 0 0 0)
 			(layer "B.Fab")
 			(effects
@@
 	(footprint "Capacitor_SMD:C_0603_1608Metric"
 		(layer "B.Cu")
-		(at 104.445 102.54 180)
+		(at 108.255 102.54)
 		(descr "Capacitor SMD 0603 (1608 Metric), square (rectangular) end terminal, IPC_7351 nominal, (Body size source: IPC-SM-782 page 76, https://www.pcb-3d.com/wordpress/wp-content/uploads/ipc-sm-782a_amendment_1_and_2.pdf), generated with kicad-footprint-generator")
 		(tags "capacitor")
 		(property "Reference" "C3"
-			(at 0 1.43 0)
+			(at 0 1.43 360)
 			(layer "B.SilkS")
 			(hide yes)
@@
 		)
 		(property "Value" "0u1"
-			(at 0 -1.43 0)
+			(at 0 -1.43 360)
 			(layer "B.Fab")
 			(hide yes)
@@
 		)
 		(property "Footprint" "Capacitor_SMD:C_0603_1608Metric"
-			(at 0 0 0)
+			(at 0 0 180)
 			(unlocked yes)
 			(layer "B.Fab")
@@
 		)
 		(property "Datasheet" ""
-			(at 0 0 0)
+			(at 0 0 180)
 			(unlocked yes)
 			(layer "B.Fab")
@@
 		)
 		(property "Description" ""
-			(at 0 0 0)
+			(at 0 0 180)
 			(unlocked yes)
 			(layer "B.Fab")
@@
 		(property ki_fp_filters "C_*")
 		(sheetname "ルート")
-		(sheetfile "t1604.kicad_sch")
+		(sheetfile "tx04.kicad_sch")
 		(attr smd)
 		(fp_line
-			(start 0.14058 0.51)
-			(end -0.14058 0.51)
+			(start 0.14058 -0.51)
+			(end -0.14058 -0.51)
 			(stroke
 				(width 0.12)
@@
 		)
 		(fp_line
-			(start 0.14058 -0.51)
-			(end -0.14058 -0.51)
+			(start 0.14058 0.51)
+			(end -0.14058 0.51)
 			(stroke
 				(width 0.12)
@@
 		)
 		(fp_line
-			(start 1.48 0.73)
-			(end -1.48 0.73)
+			(start -1.48 -0.73)
+			(end 1.48 -0.73)
 			(stroke
 				(width 0.05)
@@
 		)
 		(fp_line
-			(start 1.48 -0.73)
-			(end 1.48 0.73)
+			(start -1.48 0.73)
+			(end -1.48 -0.73)
 			(stroke
 				(width 0.05)
@@
 		)
 		(fp_line
-			(start -1.48 0.73)
-			(end -1.48 -0.73)
+			(start 1.48 -0.73)
+			(end 1.48 0.73)
 			(stroke
 				(width 0.05)
@@
 		)
 		(fp_line
-			(start -1.48 -0.73)
-			(end 1.48 -0.73)
+			(start 1.48 0.73)
+			(end -1.48 0.73)
 			(stroke
 				(width 0.05)
@@
 		)
 		(fp_line
-			(start 0.8 0.4)
-			(end -0.8 0.4)
+			(start -0.8 -0.4)
+			(end 0.8 -0.4)
 			(stroke
 				(width 0.1)
@@
 		)
 		(fp_line
-			(start 0.8 -0.4)
-			(end 0.8 0.4)
+			(start -0.8 0.4)
+			(end -0.8 -0.4)
 			(stroke
 				(width 0.1)
@@
 		)
 		(fp_line
-			(start -0.8 0.4)
-			(end -0.8 -0.4)
+			(start 0.8 -0.4)
+			(end 0.8 0.4)
 			(stroke
 				(width 0.1)
@@
 		)
 		(fp_line
-			(start -0.8 -0.4)
-			(end 0.8 -0.4)
+			(start 0.8 0.4)
+			(end -0.8 0.4)
 			(stroke
 				(width 0.1)
@@
 		)
 		(fp_text user "${REFERENCE}"
-			(at 0 0 0)
+			(at 0 0 360)
 			(layer "B.Fab")
 			(effects
@@
 		)
 		(pad "1" smd roundrect
-			(at -0.775 0 180)
+			(at -0.775 0)
 			(size 0.9 0.95)
 			(layers "B.Cu" "B.Paste" "B.Mask")
@@
 		)
 		(pad "2" smd roundrect
-			(at 0.775 0 180)
+			(at 0.775 0)
 			(size 0.9 0.95)
 			(layers "B.Cu" "B.Paste" "B.Mask")
 			(roundrect_rratio 0.25)
-			(net 13 "VCC")
+			(net 1 "GND")
 			(pintype "passive")
 		)
@@
 		(property ki_fp_filters "R_*")
 		(sheetname "ルート")
-		(sheetfile "t1604.kicad_sch")
+		(sheetfile "tx04.kicad_sch")
 		(attr smd)
 		(fp_line
@@
 		(tags "capacitor")
 		(property "Reference" "C1"
-			(at 0 1.43 360)
+			(at 0 1.43 0)
 			(layer "B.SilkS")
 			(hide yes)
@@
 		)
 		(property "Value" "4u7"
-			(at 0 -1.43 360)
+			(at 0 -1.43 0)
 			(layer "B.Fab")
 			(hide yes)
@@
 		(property ki_fp_filters "C_*")
 		(sheetname "ルート")
-		(sheetfile "t1604.kicad_sch")
+		(sheetfile "tx04.kicad_sch")
 		(attr smd)
 		(fp_line
@@
 		)
 		(fp_text user "${REFERENCE}"
-			(at 0 0 360)
+			(at 0 0 0)
 			(layer "B.Fab")
 			(effects
@@
 		(tags "resistor")
 		(property "Reference" "R2"
-			(at 0 1.43 360)
+			(at 0 1.43 0)
 			(layer "B.SilkS")
 			(hide yes)
@@
 		)
 		(property "Value" "4.7k"
-			(at 0 -1.43 360)
+			(at 0 -1.43 0)
 			(layer "B.Fab")
 			(hide yes)
@@
 		(property ki_fp_filters "R_*")
 		(sheetname "ルート")
-		(sheetfile "t1604.kicad_sch")
+		(sheetfile "tx04.kicad_sch")
 		(attr smd)
 		(fp_line
@@
 		)
 		(fp_text user "${REFERENCE}"
-			(at 0 0 360)
+			(at 0 0 0)
 			(layer "B.Fab")
 			(effects
@@
 		(tags "VSSOP SO")
 		(property "Reference" "U3"
-			(at 0 2.45 360)
+			(at 0 2.45 0)
 			(layer "B.SilkS")
 			(hide yes)
@@
 		)
 		(property "Value" "TS5A23159DGS"
-			(at 0 -2.45 360)
+			(at 0 -2.45 0)
 			(layer "B.Fab")
 			(hide yes)
@@
 		(property ki_fp_filters "VSSOP*3x3mm*P0.5mm*")
 		(sheetname "ルート")
-		(sheetfile "t1604.kicad_sch")
+		(sheetfile "tx04.kicad_sch")
 		(attr smd)
 		(fp_line
@@
 		)
 		(fp_text user "${REFERENCE}"
-			(at 0 0 360)
+			(at 0 0 0)
 			(layer "B.Fab")
 			(effects
@@
 		(tags "resistor")
 		(property "Reference" "R4"
-			(at 0 1.43 360)
+			(at 0 1.43 0)
 			(layer "B.SilkS")
 			(hide yes)
@@
 		)
 		(property "Value" "4.7k"
-			(at 0 -1.43 360)
+			(at 0 -1.43 0)
 			(layer "B.Fab")
 			(hide yes)
@@
 		(property ki_fp_filters "R_*")
 		(sheetname "ルート")
-		(sheetfile "t1604.kicad_sch")
+		(sheetfile "tx04.kicad_sch")
 		(attr smd)
 		(fp_line
@@
 		)
 		(fp_text user "${REFERENCE}"
-			(at 0 0 360)
+			(at 0 0 0)
 			(layer "B.Fab")
 			(effects
@@
 		(property ki_fp_filters "MSOP*3x3mm*P0.5mm*")
 		(sheetname "ルート")
-		(sheetfile "t1604.kicad_sch")
+		(sheetfile "tx04.kicad_sch")
 		(attr smd)
 		(fp_line
@@
 	)
 	(segment
-		(start 105.2875 102.4725)
-		(end 105.2875 101)
+		(start 107.48 102.54)
+		(end 106.8275 102.54)
 		(width 0.25)
 		(layer "B.Cu")
@@
 	)
 	(segment
-		(start 105.22 102.54)
-		(end 105.2875 102.4725)
+		(start 106.8275 102.54)
+		(end 105.2875 101)
 		(width 0.25)
 		(layer "B.Cu")

Commit message: -
Parts:
- added G***: LOGO, LOGO, B.Cu at (94.9, 100.0)
Other:
- board text added: "tinyAVR X04"
