File: pd-fix/pd-fix.kicad_pcb (KiCad board)
At the start: 2 copper layers, 9 x 10 mm, 9 parts, among them J1 USB_C_Receptacle_PowerOnly_6P, J2 Conn_01x02_Pin, U1 CH221K

Commit message: -
Parts:
- moved J2 0.50 mm to (105.8, 101.3)
Routing:
- net VBUS: track 3.56 -> 1.28 mm
Other:
- board size 9 x 10 mm -> 10 x 10 mm
Changed lines of the file:
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@@
 	(footprint "Connector_PinHeader_2.54mm:PinHeader_1x02_P2.54mm_Vertical"
 		(layer "F.Cu")
-		(at 105.25 101.275 180)
+		(at 105.75 101.275 180)
 		(descr "Through hole straight pin header, 1x02, 2.54mm pitch, single row")
 		(tags "Through hole pin header THT 1x02 2.54mm single row")
 		(property "Reference" "J2"
-			(at 0 -2.33 360)
+			(at 0 -2.33 0)
 			(layer "F.SilkS")
 			(hide yes)
@@
 		)
 		(property "Value" "Conn_01x02_Pin"
-			(at 0 4.87 360)
+			(at 0 4.87 0)
 			(layer "F.Fab")
 			(hide yes)
@@
 		(tags "resistor")
 		(property "Reference" "R2"
-			(at 0 1.43 360)
+			(at 0 1.43 0)
 			(layer "B.SilkS")
 			(hide yes)
@@
 		)
 		(property "Value" "4.7k"
-			(at 0 -1.43 360)
+			(at 0 -1.43 0)
 			(layer "B.Fab")
 			(hide yes)
@@
 		)
 	)
-	(gr_rect
+	(gr_line
 		(start 97.5 95)
-		(end 106.5 105)
+		(end 97.5 105)
 		(stroke
 			(width 0.05)
 			(type default)
 		)
-		(fill none)
+		(layer "Edge.Cuts")
+	)
+	(gr_line
+		(start 107.5 105)
+		(end 107.5 95)
+		(stroke
+			(width 0.05)
+			(type default)
+		)
+		(layer "Edge.Cuts")
+	)
+	(gr_line
+		(start 97.5 95)
+		(end 107.5 95)
+		(stroke
+			(width 0.05)
+			(type default)
+		)
+		(layer "Edge.Cuts")
+	)
+	(gr_line
+		(start 97.5 105)
+		(end 107.5 105)
+		(stroke
+			(width 0.05)
+			(type default)
+		)
 		(layer "Edge.Cuts")
 	)
@@
 		(net 2)
 	)
-	(segment
-		(start 104.995 98.48)
-		(end 105.25 98.735)
-		(width 0.5)
-		(layer "F.Cu")
-		(net 3)
-	)
-	(segment
-		(start 103.08 98.48)
-		(end 104.995 98.48)
-		(width 0.5)
-		(layer "F.Cu")
-		(net 3)
-	)
 	(via
 		(at 100.5 98.25)
@@
 		(polygon
 			(pts
-				(xy 100 98) (xy 103 98) (xy 103 102) (xy 100 102)
-			)
-		)
+				(xy 100 97.75) (xy 104.25 97.75) (xy 104.75 97.25) (xy 107.5 97.25) (xy 107.5 99.5) (xy 105 102)
+				(xy 100 102)
+			)
+		)
