File: avr/mx09_48/mx09_48.kicad_pcb (KiCad board)
At the start: 2 copper layers, 61 x 17.8 mm, 19 parts, among them J1 USB_C_Receptacle_USB2.0_16P, J2 Conn_02x24_Counter_Clockwise, SW1 SW_Push, U1 ATmega4809-A, U2 CH340E, U3 TS5A23159DGS

Commit message: -
Parts:
- removed the G*** at (124.8, 86.5)
- added ?: , Library:PCB.MCBEERINGI.DEV, B.Cu at (122.5, 100.0)
- moved SW1 6.98 mm to (86.2, 100.0), turned to 180 degrees
- moved D1 5.00 mm to (93.0, 100.0)
- moved R1 5.00 mm to (91.2, 100.0)
- moved D2 3.25 mm to (79.5, 100.0), turned to -90 degrees
- moved R7 3.25 mm to (81.2, 100.0), turned to -90 degrees
Routing:
- net VCC: track 66.1 -> 53.6 mm
- net PA7: track 47.6 -> 37.6 mm
- net PA3: track 34.3 -> 29.5 mm
- net TNOW: track 5.56 -> 1.82 mm
- net PA0: track 33.8 -> 33.3 mm
Other:
- board text added: "05 06 07 08 09 10 11 12 13 14 15 16 17 V G 18 19 20 21 22 23 24 25 26"
- board text added: "27 28 29 V G 30 31 32 33 34 35 36 37 38 39 40 U V G 00 01 02 03 04"
- board text added: "A3"
- board text added: "A5 A6 A7 A8 A9 Aa Ab T2 R2 Ac Ad Ae Af T0 R0 DA CL"
- board text added: "T1 R1"
- board text added: "T3 R3 b3 a0 a0 a0 a0 a0 a0 A0 A1 A2 A3 A4"
- board text added: "b0 b1"
- board text added: "pcb.mcbeeringi.dev"
