File: avr/tx04/tx04.kicad_pcb (KiCad board)
At the start: 2 copper layers, 25.4 x 10.2 mm, 18 parts, among them J1 USB_C_Receptacle_USB2.0_16P, J2 Conn_02x07_Counter_Clockwise, SW1 SW_Push, SW2 SW_SPDT, U1 ATtiny1604-SS, U2 CH340E, U3 TS5A23159DGS

Commit message: -
Parts:
- removed the G*** at (94.9, 100.0)
- added G***: LOGO, LOGO, F.Cu at (115.2, 100.0)
- added G***: LOGO, LOGO, B.Cu at (95.8, 100.0)
- moved C2 13.5 mm to (126.2, 100.0)
- moved SW2 5.62 mm to (121.2, 97.5), turned to 90 degrees
- moved R5 0.57 mm to (95.2, 97.0)
- moved R6 0.57 mm to (95.2, 103.0)
Routing:
- net VCC: track 29.3 -> 23.1 mm
- net /Vedlc: track 0.00 -> 2.50 mm
- net GND: vias 2 -> 18
- added copper zone on F.Cu, net VCC
Other:
- board size 25.4 x 10.2 mm -> 35.6 x 12.7 mm
- board text added: "B1 B0 U A1 A2 A3 G"
- board text added: "V A4 A5 A6 A7 B3 B2"

Commit message: -
Parts:
- moved G*** 0.50 mm to (95.2, 100.0)

Commit message: tx04_updi_fix
Parts:
- G***: moved to B.Cu
- moved C1 5.94 mm to (101.8, 102.8)
- moved SW2 5.00 mm to (121.2, 102.5)
- moved C3 3.51 mm to (104.8, 102.8), turned to 180 degrees
- moved R2 3.51 mm to (104.8, 97.2), turned to 180 degrees
- moved U3 1.91 mm to (108.2, 100.0), turned to -90 degrees
- moved R3 1.24 mm to (110.8, 98.5), turned to 90 degrees
- moved R4 1.24 mm to (110.8, 101.5), turned to -90 degrees
- moved R1 0.52 mm to (101.8, 97.2)
- moved G*** 0.50 mm to (114.8, 100.0), turned to -90 degrees
- moved U2 0.08 mm to (103.2, 100.0)
- turned C2 to 180 degrees
Connections:
- U3 pad 2: Net-(R3-Pad1) -> Net-(R2-Pad1)
- U3 pad 4: Net-(R4-Pad1) -> UPDI
- U3 pad 7: UPDI -> Net-(R4-Pad1)
- U3 pad 9: Net-(R2-Pad1) -> Net-(R3-Pad1)
Routing:
- net RTS#: track 16.1 -> 11.0 mm, vias 2 -> 3
- net TXD: track 7.97 -> 3.65 mm
- net RXD: track 2.88 -> 7.10 mm
- net PB3: track 14.6 -> 11.0 mm
- net VCC: track 23.1 -> 19.8 mm
- net Net-(R3-Pad1): track 3.23 -> 5.09 mm
- net UPDI: track 8.78 -> 10.5 mm
- net Net-(U2-V3): track 2.83 -> 1.82 mm
- net GND: vias 18 -> 16

Commit message: -
Other:
- board text added: "6~ 7~ b 8 9^ a~ G"
- board text added: "V 0~ 1~ 2^ 3 4 5~"

Commit message: -
Parts:
- removed C2: 1F5, Library:edlc
- removed SW2: SW_SPDT, Library:sw
- moved D1 0.29 mm to (101.5, 97.0)
- moved SW1 0.26 mm to (101.5, 100.8)
- moved G*** 0.25 mm to (114.5, 100.0)
- moved U1 0.13 mm to (107.8, 100.0)
Routing:
- net /Vedlc: track 2.50 -> 0.00 mm
- net PB3: track 11.0 -> 10.4 mm
- net GND: vias 16 -> 22
Other:
- board size 35.6 x 12.7 mm -> 25.4 x 12.7 mm

Commit message: -
Parts:
- removed the G*** at (114.5, 100.0)
- added ?: , Library:PCB.MCBEERINGI.DEV_small, B.Cu at (114.5, 100.0)
Routing:
- net D-: track 4.52 -> 5.08 mm
