File: 7seg/7seg.kicad_sch (KiCad schematic)
At the start: 22 parts, among them J1 Conn_01x05_Pin, U1 D168K, U10 D168K, U2 74HC595, U3 74HC595, U4 D168K, U5 D168K, U6 D168K, U7 D168K, U8 D168K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

Commit message: 7seg
Parts:
- removed U1, U10, U4, U5, U6, U7, U8, U9: D168K, Display_7Segment:D1X8K, symbol Display_Character:D168K
- removed U3: 74HC595, Package_SO:SOP-16_4.55x10.3mm_P1.27mm, symbol 74xx:74HC595
- added U1: 74HC595, Package_SO:SOP-16_4.55x10.3mm_P1.27mm, symbol 74xx:74HC595
- added U10, U3, U4, U5, U6, U7, U8, U9: ~, Library:LA-501DD, symbol Library:LA-501DD
Connections:
- net A: now also U10.7 (A), U3.7 (A), U4.7 (A), U5.7 (A), U6.7 (A), U7.7 (A), U8.7 (A), U9.7 (A)
- net B: now also U10.6 (B), U3.6 (B), U4.6 (B), U5.6 (B), U6.6 (B), U7.6 (B), U8.6 (B), U9.6 (B)
- net C: now also U10.4 (C), U3.4 (C), U4.4 (C), U5.4 (C), U6.4 (C), U7.4 (C), U8.4 (C), U9.4 (C)
- net C0: now also U2.15 (QA), U3.3 (COM), U3.8 (COM)
- net C1: now also U2.1 (QB), U4.3 (COM), U4.8 (COM)
- net C2: now also U2.2 (QC), U5.3 (COM), U5.8 (COM)
- net C3: now also U2.3 (QD), U6.3 (COM), U6.8 (COM)
- net C4: now also U2.4 (QE), U7.3 (COM), U7.8 (COM)
- net C5: now also U2.5 (QF), U8.3 (COM), U8.8 (COM)
- net C6: now also U2.6 (QG), U9.3 (COM), U9.8 (COM)
- net C7: now also U2.7 (QH), U10.3 (COM), U10.8 (COM)
- net D: now also U10.2 (D), U3.2 (D), U4.2 (D), U5.2 (D), U6.2 (D), U7.2 (D), U8.2 (D), U9.2 (D)
- net DP: now also U10.5 (DP), U3.5 (DP), U4.5 (DP), U5.5 (DP), U6.5 (DP), U7.5 (DP), U8.5 (DP), U9.5 (DP)
- net E: now also U10.1 (E), U3.1 (E), U4.1 (E), U5.1 (E), U6.1 (E), U7.1 (E), U8.1 (E), U9.1 (E)
- net F: now also U10.9 (F), U3.9 (F), U4.9 (F), U5.9 (F), U6.9 (F), U7.9 (F), U8.9 (F), U9.9 (F)
- net G: now also U10.10 (G), U3.10 (G), U4.10 (G), U5.10 (G), U6.10 (G), U7.10 (G), U8.10 (G), U9.10 (G)
- net GND: now also U1.8 (GND)
- net OE#: now also U1.13 (~{OE})
- net RCLK: now also U1.12 (RCLK)
- net SER: now also U1.14 (SER); no longer U2.14 (SER)
- net SRCLK: now also U1.11 (SRCLK)
- net VCC: now also U1.10 (~{SRCLR}), U1.16 (VCC)
- net at R1.1: now also U1.15 (QA); no longer U2.15 (QA)
- net at R7.1: now also U1.6 (QG); no longer U2.6 (QG)
- net at R4.1: now also U1.3 (QD); no longer U2.3 (QD)
- net at R2.1: now also U1.1 (QB); no longer U2.1 (QB)
- net at R6.1: now also U1.5 (QF); no longer U2.5 (QF)
- net at R5.1: now also U1.4 (QE); no longer U2.4 (QE)
- net at R3.1: now also U1.2 (QC); no longer U2.2 (QC)
- net at R8.1: now also U1.7 (QH); no longer U2.7 (QH)
- new net: U1.9 (QH'), U2.14 (SER)
