File: proj/usb/serial/serial.kicad_pcb (KiCad board)
At the start: 2 copper layers, 22 x 15 mm, 15 parts, among them J1 USB_A, J2 USB_C_Receptacle_USB2.0_16P, J3 OUT, Q1 BSS138, Q2 BSS138, U1 CH340K, U2 TS5A23159DGS, U3 AP7333

Commit message: -
Parts:
- added D1: POWER, LED_SMD:LED_0603_1608Metric, F.Cu at (105.8, 94.2)
- added R3: 10k, Resistor_SMD:R_0603_1608Metric, B.Cu at (105.8, 94.2)
Routing:
- net VCC: track 5.57 -> 4.51 mm
- net Net-(D1-A): vias 0 -> 1

Commit message: -
Other:
- outline, holes or cut-outs redrawn
- board text added: "5k1 x2"
- board text added: "AP7333"
- board text added: "USB Serial Writer"
- board text removed: "Vreg"
- board text removed: "Writer USB Serial"
- board text removed: "\5k1 x2/"
Changed lines of the file:
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@@
 		)
 		(fp_text user "E"
-			(at 0 0.5 0)
+			(at -0.7 -0.51 0)
 			(unlocked yes)
 			(layer "B.SilkS")
@@
 					(bold yes)
 				)
-				(justify left mirror)
+				(justify right mirror)
 			)
 		)
@@
 	(gr_line
 		(start 100 92.5)
+		(end 100 94)
+		(stroke
+			(width 0.1)
+			(type solid)
+		)
+		(layer "Edge.Cuts")
+	)
+	(gr_line
+		(start 100 92.5)
 		(end 122 92.5)
 		(stroke
@@
 	)
 	(gr_line
-		(start 100 92.5)
+		(start 100 106)
 		(end 100 107.5)
 		(stroke
@@
 			(font
 				(size 0.8 0.8)
-				(thickness 0.16)
-				(bold yes)
+				(thickness 0.1)
 			)
 			(justify left)
@@
 		(effects
 			(font
-				(size 0.5 0.5)
-				(thickness 0.1)
-				(bold yes)
+				(size 0.6 0.6)
+				(thickness 0.075)
 			)
 			(justify mirror)
 		)
 	)
-	(gr_text "Writer\nUSB Serial"
-		(at 117.75 100.25 90)
+	(gr_text "USB Serial\nWriter"
+		(at 118 100.5 90)
 		(layer "B.Mask")
 		(effects
@@
 		)
 	)
-	(gr_text "\\5k1 x2/"
+	(gr_text "5k1 x2"
 		(at 111.75 106.25 0)
 		(layer "B.Mask")
 		(effects
 			(font
-				(size 0.8 0.8)
-				(thickness 0.16)
-				(bold yes)
+				(size 0.6 0.6)
+				(thickness 0.075)
 			)
 			(justify mirror)
 		)
 	)
-	(gr_text "Vreg"
-		(at 112.5 94.5 90)
-		(layer "B.Mask")
-		(effects
-			(font
-				(size 0.8 0.8)
-				(thickness 0.16)
-				(bold yes)
+	(gr_text "AP7333"
+		(at 112.75 96.5 90)
+		(layer "B.Mask")
+		(effects
+			(font
+				(size 0.6 0.6)
+				(thickness 0.075)
+			)
+			(justify mirror)
+		)
+	)
+	(gr_text "0u1\nx3"
+		(at 108.25 98 0)
+		(layer "B.Mask")
+		(effects
+			(font
+				(size 0.6 0.6)
+				(thickness 0.075)
 			)
 			(justify left mirror)
 		)
 	)
-	(gr_text "0u1\nx3"
-		(at 107 98.25 0)
-		(layer "B.Mask")
-		(effects
-			(font
-				(size 0.8 0.8)
-				(thickness 0.16)
-				(bold yes)
-			)
-			(justify mirror)
-		)
-	)

Commit message: -
Routing:
- net VCC: vias 5 -> 3
Changed lines of the file:
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@@
-	)
-	(via
-		(at 111 97.25)
-		(size 0.3)
-		(drill 0.15)
-		(layers "F.Cu" "B.Cu")
-		(net 2)
 	)
 	(via
@@
 		(net 2)
 	)
-	(via
-		(at 110.75 97)
-		(size 0.3)
-		(drill 0.15)
-		(layers "F.Cu" "B.Cu")
-		(free yes)
-		(net 2)
-	)
