File: proj/7seg/clk/clk.kicad_sch (KiCad schematic)
At the start: 25 parts, among them J1 Conn_01x02_Pin, J2 USB_A, J3 USB_C_Receptacle_PowerOnly_6P, SW1 SW_Push, SW2 SW_Push, U1 LTC-4627JG, U2 74HC595, U3 74HC595, U4 ATtiny402-SS

Commit message: -
Parts:
- removed J2: USB_A, Library:USB_A_PLUG_USB-4AM103AS, symbol Connector:USB_A
- removed J3: USB_C_Receptacle_PowerOnly_6P, Connector_USB:USB_C_Receptacle_GCT_USB4125-xx-x_6P_TopMnt_Horizontal, symbol Connector:USB_C_Receptacle_PowerOnly_6P
- removed LS1: Speaker, Library:PKLCS1212E4001-R1, symbol Device:Speaker
- added BZ1: Buzzer, Buzzer_Beeper:Buzzer_TDK_PS1240P02BT_D12.2mm_H6.5mm, symbol Device:Buzzer
- added J2: Conn_01x04_Pin, Connector_PinHeader_2.54mm:PinHeader_1x04_P2.54mm_Vertical, symbol Connector:Conn_01x04_Pin
- C1: value C_Small -> C_RCLK
- C2: value C_Small -> C_SER
- R10: value R_Small -> R_SER
- R11, R12: value 5k1 -> R_I2C
- R9: value R_Small -> R_RCLK
- SW1, SW2: footprint Library:alps-skrp -> Library:alps-skrg
Connections:
- net SEG0 is gone; now on net SEG1: R1.2, U1.14 (A)
- net SEGC0 is gone; now on net SEGC1: U1.1 (CA1), U3.6 (QG)
- net _SEG0 is gone; now on net _SEG1: R1.1, U2.7 (QH)
- net GND: now also BZ1.2 (-), J2.1 (Pin_1); no longer R11.2, R12.2
- net SEG1: no longer R2.2, U1.16 (B)
- net SEG2: now also R2.2, U1.16 (B); no longer R3.2, U1.13 (C)
- net SEG3: now also R3.2, U1.13 (C); no longer R4.2, U1.3 (D)
- net SEG4: now also R4.2, U1.3 (D); no longer R5.2, U1.5 (E)
- net SEG5: now also R5.2, U1.5 (E); no longer R6.2, U1.11 (F)
- net SEG6: now also R6.2, U1.11 (F); no longer R7.2, U1.15 (G)
- net SEG7: now also R7.2, U1.15 (G); no longer R8.2, U1.7 (DP)
- net SEGC1: no longer U1.2 (CA2), U3.5 (QF)
- net SEGC2: now also U1.2 (CA2), U3.5 (QF); no longer U1.6 (CA3), U3.4 (QE)
- net SEGC3: now also U1.6 (CA3); no longer U1.8 (CA4)
- net SEGC4: now also U1.8 (CA4), U3.2 (QC); no longer U1.4 (CAL)
- net SPK: now also U4.3 (PA7), BZ1.1 (+); no longer U4.5 (PA2)
- net SRCLK: now also U4.2 (PA6); no longer U4.4 (PA1)
- net VCC: now also R11.1, R12.1, J2.2 (Pin_2)
- net _SEG1: no longer R2.1, U2.6 (QG)
- net _SEG2: now also R2.1, U2.6 (QG); no longer R3.1, U2.5 (QF)
- net _SEG3: now also R3.1, U2.5 (QF); no longer R4.1, U2.4 (QE)
- net _SEG4: now also R4.1, U2.4 (QE); no longer R5.1, U2.3 (QD)
- net _SEG5: now also R5.1, U2.3 (QD); no longer R6.1, U2.2 (QC)
- net _SEG6: now also R6.1, U2.2 (QC); no longer R7.1, U2.1 (QB)
- net _SEG7: now also R7.1, U2.1 (QB); no longer R8.1, U3.7 (QH)
- net BTN0 renamed PA1
- net PA1: now also R11.2, U4.4 (PA1), J2.3 (Pin_3); no longer U4.2 (PA6)
- net BTN1 renamed PA2
- net PA2: now also R12.2, U4.5 (PA2), J2.4 (Pin_4); no longer U4.3 (PA7)
- new net SEG8: R8.2, U1.7 (DP)
- new net SEGC:: U1.4 (CAL), U3.4 (QE)
- new net _SEG8: R8.1, U3.7 (QH)
- no-connect marks 7 -> 4
