File: proj/esp/c3-wroom-hat-clk/c3-wroom-hat-clk.kicad_pcb (KiCad board)
At the start: 2 copper layers, 72 x 47 mm, 27 parts, among them J1 IN1, J2 IN2, Q1 BPW40, SW1 SW_Push, SW2 SW_Push, U1 D168K, U2 74HC595, U3 74HC595, U4 D168K, U5 D168K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

Commit message: -
Parts:
- removed REF** (x4): MountingHole_3.2mm_M3, MountingHole:MountingHole_3.2mm_M3
- added ?: , Library:PCB.MCBEERINGI.DEV, B.Cu at (91.0, 122.0)
- added G***: LOGO, LOGO, B.Cu at (74.5, 122.0)
- added H1: MountingHole, MountingHole:MountingHole_3.2mm_M3, F.Cu at (67.0, 91.0)
- added H2: MountingHole, MountingHole:MountingHole_3.2mm_M3, F.Cu at (133.0, 91.0)
- added H3: MountingHole, MountingHole:MountingHole_3.2mm_M3, F.Cu at (67.0, 132.0)
- added H4: MountingHole, MountingHole:MountingHole_3.2mm_M3, F.Cu at (133.0, 132.0)
- J1, J2: moved to F.Cu
- moved SW1 41.9 mm to (68.0, 105.5), turned to 90 degrees
- moved SW2 24.0 mm to (68.0, 117.5), turned to 90 degrees
- moved J2 17.6 mm to (104.4, 112.7)
- moved J1 17.6 mm to (104.4, 130.5)
- moved Q1 17.3 mm to (130.0, 101.3), turned to 90 degrees
- moved R9 17.2 mm to (129.2, 106.0), turned to -90 degrees
- moved TH1 11.7 mm to (130.0, 108.4)
- moved R10 11.2 mm to (130.8, 106.0), turned to -90 degrees
- moved U3 3.20 mm to (105.0, 98.0)
- moved R8 3.00 mm to (109.0, 98.0)
- moved BZ1 0.82 mm to (82.4, 117.0)
- moved R1 0.20 mm to (123.4, 99.6)
- moved R2 0.20 mm to (123.4, 98.0)
- moved R3 0.20 mm to (123.4, 96.4)
Routing:
- net BTN1: track 10.3 -> 61.5 mm
- net IO0: track 2.74 -> 50.7 mm, vias 0 -> 1
- net BTN2: track 8.95 -> 52.4 mm
- net VBUS: track 24.9 -> 63.1 mm
- net +3.3V: track 15.2 -> 39.6 mm, vias 2 -> 0
- net IO10: track 23.8 -> 45.3 mm, vias 1 -> 0
- net IO1: track 26.3 -> 46.5 mm, vias 1 -> 2
- net IO2: track 29.7 -> 46.0 mm, vias 1 -> 2
- net IO3: track 34.6 -> 45.3 mm, vias 1 -> 2
- net IO6: track 25.3 -> 35.7 mm
- net IO7: track 33.5 -> 28.6 mm, vias 1 -> 0
- net SEG8: track 74.9 -> 78.6 mm
- net SEGC2: track 28.9 -> 25.2 mm
- net SEGC1: track 37.3 -> 34.1 mm
- net SEGC3: track 19.3 -> 16.3 mm
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Other:
- board text added: "74HC595 *2"
- board text added: "9 8 7 6 5 4 E v G"
- board text added: "C3_WROOM_CLK_EXT"
- board text added: "ESP32 C3 dev board"
- board text added: "G V 0 1 2 3 T R a"
- board text added: "IO10"
- board text added: "IO4"
- board text added: "IO5"
- board text added: "IO6"
- board text added: "IO7"
- board text added: "R_LED *8"
- board text added: "R_PHOTO"
- board text added: "R_THERMO"
- board text added: "SER: IO0 SERCLK: IO1 RCLK: IO2 OE#: IO3"
- board text added: "TH"
