File: paneled/c3-wroom-ext-clk-set/c3-wroom-ext-clk-set.kicad_pcb (KiCad board)
At the start: 2 copper layers, 94 x 95.2 mm, 88 parts, among them J1 IN1, J1 USB_C_Receptacle_USB2.0_16P, J2 IN2, J2 OUT1, J3 OUT2, Q1 BPW40, SW1 SW_BOOT, SW1 SW_Push, SW2 SW_Push, U1 D168K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

Commit message: -
Other:
- board text added: "JLCJLCJLCJLC"
Changed lines of the file:
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@@
+		)
+	)
+	(gr_text "JLCJLCJLCJLC"
+		(at 39.6 67.6 270)
+		(layer "F.SilkS")
+		(effects
+			(font
+				(size 1.5 1.5)
+				(thickness 0.3)
+				(bold yes)
+			)
 		)
 	)
