File: proj/esp/c3-wroom-ext-clk/c3-wroom-ext-clk.kicad_pcb (KiCad board)
At the start: 2 copper layers, 72 x 47 mm, 29 parts, among them J1 IN1, J2 IN2, Q1 BPW40, SW1 SW_Push, SW2 SW_Push, U1 D168K, U2 74HC595, U3 74HC595, U4 D168K, U5 D168K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

Commit message: -
Parts:
- moved BZ1 10.1 mm to (77.9, 126.0)
- moved G*** 5.32 mm to (78.0, 118.0)
- moved ? 4.12 mm to (92.0, 118.0)
Routing:
- net IO10: track 45.3 -> 53.5 mm
Changed lines of the file:
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@@
 	(footprint "Buzzer_Beeper:Buzzer_TDK_PS1240P02BT_D12.2mm_H6.5mm"
 		(layer "F.Cu")
-		(at 82.370785 117 180)
+		(at 77.870785 126 180)
 		(descr "Buzzer, D12.2mm height 6.5mm, https://product.tdk.com/info/en/catalog/datasheets/piezoelectronic_buzzer_ps_en.pdf")
 		(tags "buzzer")
@@
 	(footprint "Library:PCB.MCBEERINGI.DEV"
 		(layer "B.Cu")
-		(at 91 122 180)
+		(at 92 118 180)
 		(property "Reference" ""
 			(at 0 0 0)
@@
 	(footprint "LOGO"
 		(layer "B.Cu")
-		(at 74.5 122 180)
+		(at 78 118 180)
 		(property "Reference" "G***"
 			(at 0 0 0)
@@
 	)
 	(gr_text "C3_WROOM_CLK_EXT"
-		(at 87.5 131 0)
+		(at 85 129 0)
 		(layer "B.Mask")
 		(effects
@@
 	)
 	(gr_text "IO10"
-		(at 80 125 0)
+		(at 84 130 0)
 		(layer "F.SilkS")
 		(effects
@@
 	)
 	(segment
-		(start 123.9 112.7)
-		(end 124.765 112.7)
+		(start 92.4 111.4)
+		(end 77.870785 125.929215)
 		(width 0.2)
 		(layer "F.Cu")
@@
 	)
 	(segment
-		(start 122.6 111.4)
+		(start 124.765 112.7)
 		(end 123.9 112.7)
 		(width 0.2)
@@
 	)
 	(segment
-		(start 82.370785 117)
-		(end 87.970785 111.4)
+		(start 122.6 111.4)
+		(end 92.4 111.4)
 		(width 0.2)
 		(layer "F.Cu")
@@
 	)
 	(segment
-		(start 87.970785 111.4)
+		(start 77.870785 125.929215)
+		(end 77.870785 126)
+		(width 0.2)
+		(layer "F.Cu")
+		(net 1)
+	)
+	(segment
+		(start 123.9 112.7)
 		(end 122.6 111.4)
 		(width 0.2)

Commit message: -
Other:
- board text added: "> __43_21d _GFEDCBA"
Changed lines of the file:
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@@
+		)
+	)
+	(gr_text "> __43_21d _GFEDCBA"
+		(at 97 122.5 0)
+		(layer "F.SilkS")
+		(effects
+			(font
+				(size 1.5 1.5)
+				(thickness 0.3)
+				(bold yes)
+			)
 		)
 	)

Commit message: -
Routing:
- net SEGC2: track 25.2 -> 26.2 mm
- net IO10: track 53.5 -> 52.7 mm
- net SEG8: track 78.6 -> 79.2 mm
- net SEG4: track 83.7 -> 84.2 mm
- net GND: vias 2 -> 121
