File: proj/7seg/8x1_ext/8x1_ext.kicad_pcb (KiCad board)
At the start: 2 copper layers, 100 x 19 mm, 44 parts, among them J1 Conn_01x03_Pin, J2 grove, J3 UART, J4 UART, J9 USB_C, SW1 SW_Push, U1 74HC595, U10 D168K, U11 MCU_DISP, U12 MCU_CTL, U13 CH340E, U14 CH340K, U2 74HC595, U3 D168K, U4 D168K, U5 D168K, U6 D168K, U7 D168K, U8 D168K, U9 D168K

Commit message: -
Parts:
- removed ?: , Library:PCB.MCBEERINGI.DEV
- removed C1: 0.1u, Capacitor_SMD:C_0603_1608Metric
- removed C2: 1u, Capacitor_SMD:C_0603_1608Metric
- removed C3: 0u1, Capacitor_SMD:C_0603_1608Metric
- removed D1: NeoPixel, LED_SMD:LED_WS2812B-2020_PLCC4_2.0x2.0mm
- removed D3: LED_TNOW, LED_SMD:LED_0603_1608Metric
- removed J1: Conn_01x03_Pin, Connector_PinHeader_2.54mm:PinHeader_1x03_P2.54mm_Vertical
- removed J2: grove, Connector_PinHeader_2.54mm:PinHeader_1x04_P2.54mm_Vertical
- removed JP1, JP2: T:R, Jumper:SolderJumper-3_P1.3mm_Bridged12_RoundedPad1.0x1.5mm
- removed JP5, JP6: DISP:CTL, Jumper:SolderJumper-3_P1.3mm_Bridged12_RoundedPad1.0x1.5mm
- removed R1, R2, R3, R4, R5, R6, R7, R8: 1k, Resistor_SMD:R_0603_1608Metric
- removed R10, R11: 5k1, Resistor_SMD:R_0603_1608Metric
- removed R12, R13, R9: 10k, Resistor_SMD:R_0603_1608Metric
- removed SW1: SW_Push, Library:alps-skrp
- removed U1, U2: 74HC595, Package_SO:TSSOP-16_4.4x5mm_P0.65mm
- removed U11: MCU_DISP, Package_SO:SOIC-8_3.9x4.9mm_P1.27mm
- removed U12: MCU_CTL, Package_SO:SOIC-14_3.9x8.7mm_P1.27mm
- removed U13: CH340E, Package_SO:MSOP-10_3x3mm_P0.5mm
- removed U14: CH340K, Package_SO:SSOP-10-1EP_3.9x4.9mm_P1mm_EP2.1x3.3mm
Routing:
- net F: track 127.2 -> 0.00 mm, vias 9 -> 0
- net D: track 119.9 -> 0.00 mm, vias 9 -> 0
- net C: track 117.7 -> 0.00 mm, vias 8 -> 0
- net A: track 116.3 -> 0.00 mm, vias 9 -> 0
- net H: track 111.6 -> 0.00 mm, vias 9 -> 0
- net G: track 109.4 -> 0.00 mm, vias 8 -> 0
- net E: track 109.2 -> 0.00 mm, vias 9 -> 0
- net B: track 105.6 -> 0.00 mm, vias 9 -> 0
- net RXD_DISP: track 83.2 -> 0.00 mm, vias 4 -> 0
- net C7: track 81.8 -> 0.00 mm, vias 2 -> 0
- net TXD_DISP: track 78.8 -> 0.00 mm, vias 4 -> 0
- net C6: track 68.2 -> 0.00 mm, vias 2 -> 0
- net C5: track 55.0 -> 0.00 mm, vias 2 -> 0
- net C4: track 38.7 -> 0.00 mm, vias 2 -> 0
- net C3: track 36.8 -> 0.00 mm, vias 2 -> 0
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- removed copper zone on F.Cu, net VCC
Other:
- board text removed: "7seg *8 dev board"
- board text removed: "AVR_CTL"
- board text removed: "AVR_DISP"
- board text removed: "CH340"
- board text removed: "CTR:DISP"
- board text removed: "C_V3"
- board text removed: "C_VCC"
- board text removed: "DR_TNOW"
- board text removed: "GND VCC SDA SCL"
- board text removed: "PA3"
- board text removed: "PA7"
- board text removed: "R:T"
- board text removed: "R_CC *2"
- board text removed: "T:R"
- board text removed: "UPDI GND UPDI"

Commit message: -
Parts:
- added C1: 0.1u, Capacitor_SMD:C_0603_1608Metric, F.Cu at (84.2, 124.3)
- added C2: 1u, Capacitor_SMD:C_0603_1608Metric, F.Cu at (84.2, 126.8)
- added C3: 0u1, Capacitor_SMD:C_0603_1608Metric, F.Cu at (84.2, 129.3)
- added D1: NeoPixel, LED_SMD:LED_WS2812B-2020_PLCC4_2.0x2.0mm, F.Cu at (109.4, 129.1)
- added D3: LED_TNOW, LED_SMD:LED_0603_1608Metric, F.Cu at (110.4, 134.7)
- added J1: Conn_01x03_Pin, Connector_PinHeader_2.54mm:PinHeader_1x03_P2.54mm_Vertical, F.Cu at (104.9, 125.4)
- added J2: grove, Connector_PinHeader_2.54mm:PinHeader_1x04_P2.54mm_Vertical, F.Cu at (102.1, 142.4)
- added JP1: T:R, Jumper:SolderJumper-3_P1.3mm_Bridged12_RoundedPad1.0x1.5mm, F.Cu at (97.0, 135.2)
- added JP2: T:R, Jumper:SolderJumper-3_P1.3mm_Bridged12_RoundedPad1.0x1.5mm, F.Cu at (97.0, 139.0)
- added JP5: DISP:CTL, Jumper:SolderJumper-3_P1.3mm_Bridged12_RoundedPad1.0x1.5mm, F.Cu at (97.0, 142.9)
- added JP6: DISP:CTL, Jumper:SolderJumper-3_P1.3mm_Bridged12_RoundedPad1.0x1.5mm, F.Cu at (97.0, 146.7)
- added R1: 1k, Resistor_SMD:R_0603_1608Metric, F.Cu at (84.2, 131.8)
- added R10: 5k1, Resistor_SMD:R_0603_1608Metric, F.Cu at (92.2, 124.3)
- added R11: 5k1, Resistor_SMD:R_0603_1608Metric, F.Cu at (92.2, 126.8)
- added R12: 10k, Resistor_SMD:R_0603_1608Metric, F.Cu at (92.2, 129.3)
- added R13: 10k, Resistor_SMD:R_0603_1608Metric, F.Cu at (92.2, 131.8)
- added R2: 1k, Resistor_SMD:R_0603_1608Metric, F.Cu at (84.2, 134.4)
- added R3: 1k, Resistor_SMD:R_0603_1608Metric, F.Cu at (84.2, 136.9)
- added R4: 1k, Resistor_SMD:R_0603_1608Metric, F.Cu at (88.2, 124.3)
- added R5: 1k, Resistor_SMD:R_0603_1608Metric, F.Cu at (88.2, 126.8)
- added R6: 1k, Resistor_SMD:R_0603_1608Metric, F.Cu at (88.2, 129.3)
- added R7: 1k, Resistor_SMD:R_0603_1608Metric, F.Cu at (88.2, 131.8)
- added R8: 1k, Resistor_SMD:R_0603_1608Metric, F.Cu at (88.2, 134.4)
- added R9: 10k, Resistor_SMD:R_0603_1608Metric, F.Cu at (88.2, 136.9)
- added SW1: SW_Push, Library:alps-skrp, F.Cu at (110.6, 125.2)
- added U1: 74HC595, Package_SO:TSSOP-16_4.4x5mm_P0.65mm, F.Cu at (86.9, 141.4)
- added U11: MCU_DISP, Package_SO:SOIC-8_3.9x4.9mm_P1.27mm, F.Cu at (108.7, 143.4)
- added U12: MCU_CTL, Package_SO:SOIC-14_3.9x8.7mm_P1.27mm, F.Cu at (98.4, 128.3)
- added U13: CH340E, Package_SO:MSOP-10_3x3mm_P0.5mm, F.Cu at (108.1, 149.0)
- added U14: CH340K, Package_SO:SSOP-10-1EP_3.9x4.9mm_P1mm_EP2.1x3.3mm, F.Cu at (104.1, 136.9)
- added U2: 74HC595, Package_SO:TSSOP-16_4.4x5mm_P0.65mm, F.Cu at (86.9, 148.0)
- moved G*** 34.3 mm to (23.5, 100.0)
- moved U10 0.12 mm to (140.4, 107.6)
- moved U3 0.12 mm to (49.4, 107.6)
- moved U4 0.12 mm to (62.4, 107.6)
- moved U5 0.12 mm to (75.4, 107.6)
- moved U6 0.12 mm to (88.4, 107.6)
- moved U7 0.12 mm to (101.4, 107.6)
- moved U8 0.12 mm to (114.4, 107.6)
- moved U9 0.12 mm to (127.4, 107.6)
Routing:
- net A: track 0.00 -> 112.9 mm, vias 0 -> 8
- net D: track 0.00 -> 112.9 mm, vias 0 -> 8
- net F: track 0.00 -> 112.2 mm, vias 0 -> 8
- net C: track 0.00 -> 112.2 mm, vias 0 -> 8
- net E: track 0.00 -> 108.8 mm, vias 0 -> 8
- net B: track 0.00 -> 108.8 mm, vias 0 -> 8
- net H: track 0.00 -> 106.7 mm, vias 0 -> 8
- net G: track 0.00 -> 106.7 mm, vias 0 -> 8
Other:
- board text removed: "RC_SER"
- board text removed: "R_LED *8"

Commit message: -
Parts:
- added ?: , Library:PCB.MCBEERINGI.DEV_small, B.Cu at (57.7, 103.2)
- C1, C2, C3, D1, D3, J1, J2, JP1, JP2, JP5, JP6, R1, R10, R11, R12, R13, R2, R3, R4, R5, R6, R7, R8, R9, SW1, U1, U11, U12, U13, U14, U2: moved to B.Cu
- moved C3 65.7 mm to (140.4, 95.3), turned to -90 degrees
- moved JP6 60.0 mm to (130.0, 96.6)
- moved U13 57.6 mm to (138.5, 100.0), turned to 90 degrees
- moved R10 57.3 mm to (142.0, 95.9), turned to 90 degrees
- moved R13 55.1 mm to (134.0, 95.9), turned to -90 degrees
- moved JP1 55.1 mm to (56.4, 98.0), turned to -90 degrees
- moved JP5 54.6 mm to (130.0, 99.4)
- moved R11 54.1 mm to (141.2, 104.0), turned to 180 degrees
- moved U14 50.4 mm to (138.5, 100.0), turned to 180 degrees
- moved JP2 50.4 mm to (126.2, 98.0), turned to 90 degrees
- moved U2 49.5 mm to (80.0, 99.0)
- moved U11 47.1 mm to (101.0, 97.0), turned to 180 degrees
- moved D3 46.2 mm to (135.5, 95.9), turned to -90 degrees
- moved G*** 44.0 mm to (67.5, 100.0)
- moved U1 42.9 mm to (93.0, 99.0)
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Routing:
- net C7: track 0.00 -> 83.7 mm, vias 0 -> 2
- net RXD_DISP: track 0.00 -> 83.6 mm, vias 0 -> 4
- net TXD_DISP: track 0.00 -> 83.2 mm, vias 0 -> 4
- net C6: track 0.00 -> 68.2 mm, vias 0 -> 2
- net C5: track 0.00 -> 55.5 mm, vias 0 -> 2
- net C4: track 0.00 -> 39.9 mm, vias 0 -> 2
- net C0: track 0.00 -> 34.6 mm, vias 0 -> 2
- net C3: track 0.00 -> 25.5 mm, vias 0 -> 2
- net Net-(J4-Pin_3): track 0.00 -> 25.4 mm, vias 0 -> 1
- net SRCLK: track 0.00 -> 22.9 mm, vias 0 -> 2
- net OE#: track 0.00 -> 20.8 mm, vias 0 -> 2
- net PA7: track 0.00 -> 20.1 mm
- net /chain: track 0.00 -> 18.5 mm, vias 0 -> 2
- net RCLK: track 0.00 -> 15.8 mm, vias 0 -> 2
- net SDA: track 0.00 -> 15.3 mm, vias 0 -> 2
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- added copper zone on F.Cu, net VCC

Commit message: -
Parts:
- moved G*** 1.50 mm to (69.0, 100.0)
Routing:
- net GND: vias 7 -> 42
Other:
- board text added: "7seg *8 dev board"
- board text added: "AVR_CTL"
- board text added: "AVR_DISP"
- board text added: "CH340 [KE]"
- board text added: "CTL:DISP"
- board text added: "C_V3"
- board text added: "C_VCC"
- board text added: "G V S"
- board text added: "GND VCC SDA SCL"
- board text added: "PA3"
- board text added: "PA7"
- board text added: "R:T"
- board text added: "RC_SER"
- board text added: "R_LED *8"
- board text added: "S V G"
- board text added: "T:R"
- board text added: "TNOW"
- board text added: "UPDI GND UPDI"

Commit message: -
Connections:
- U11 pad 2: RXD_DISP -> TXD_DISP
- U11 pad 3: TXD_DISP -> RXD_DISP
- U12 pad 6: TXD_DISP -> RXD_DISP
- U12 pad 7: RXD_DISP -> TXD_DISP
Changed lines of the file:
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@@
 			(layers "B.Cu" "B.Mask" "B.Paste")
 			(roundrect_rratio 0.25)
-			(net 45 "TXD_DISP")
+			(net 46 "RXD_DISP")
 			(pinfunction "PB3")
 			(pintype "bidirectional")
@@
 			(layers "B.Cu" "B.Mask" "B.Paste")
 			(roundrect_rratio 0.25)
-			(net 46 "RXD_DISP")
+			(net 45 "TXD_DISP")
 			(pinfunction "PB2")
 			(pintype "bidirectional")
@@
 			(layers "B.Cu" "B.Mask" "B.Paste")
 			(roundrect_rratio 0.25)
-			(net 46 "RXD_DISP")
+			(net 45 "TXD_DISP")
 			(pinfunction "PA6")
 			(pintype "bidirectional")
@@
 			(layers "B.Cu" "B.Mask" "B.Paste")
 			(roundrect_rratio 0.25)
-			(net 45 "TXD_DISP")
+			(net 46 "RXD_DISP")
 			(pinfunction "PA7")
 			(pintype "bidirectional")

Commit message: -
Connections:
- net TXD_CTL renamed TXD_CTL_ALT
- JP1 pad 1: TXD_DISP -> RXD_CTL
- JP2 pad 3: TXD_DISP -> RXD_CTL
- JP5 pad 3: RXD_CTL -> RXD_CTL_ALT
- JP6 pad 1: TXD_DISP -> RXD_CTL
- U11 pad 2: TXD_DISP -> RXD_CTL
- U12 pad 12: RXD_CTL -> RXD_CTL_ALT
- U12 pad 6: RXD_DISP -> RXD_CTL
- U12 pad 7: TXD_DISP -> RXD_DISP
Routing:
- net TXD_DISP: track 83.2 -> 0.00 mm, vias 4 -> 0
- net (no net): track 0.00 -> 83.2 mm
- net RXD_CTL_ALT: track 0.00 -> 9.88 mm
- net RXD_CTL: track 9.88 -> 0.00 mm
- net RXD_DISP: vias 4 -> 8

Commit message: -
Parts:
- removed D1: NeoPixel, LED_SMD:LED_WS2812B-2020_PLCC4_2.0x2.0mm
- removed J9: USB_C, Connector_USB:USB_C_Receptacle_GCT_USB4105-xx-A_16P_TopMnt_Horizontal
- removed JP5, JP6: DISP:CTL, Jumper:SolderJumper-3_P1.3mm_Bridged12_RoundedPad1.0x1.5mm
- removed SW1: SW_Push, Library:alps-skrp
- removed U14: CH340K, Package_SO:SSOP-10-1EP_3.9x4.9mm_P1mm_EP2.1x3.3mm
- C1: value 0.1u -> 10n
- J1: value Conn_01x03_Pin -> UART; footprint Connector_PinHeader_2.54mm:PinHeader_1x03_P2.54mm_Vertical -> Connector_PinSocket_2.54mm:PinSocket_1x02_P2.54mm_Vertical
- J2: value grove -> COMM; footprint Connector_PinHeader_2.54mm:PinHeader_1x04_P2.54mm_Vertical -> Connector_JST:JST_ZH_B4B-ZR_1x04_P1.50mm_Vertical
- J3: value UART -> COMM; footprint Connector_PinHeader_2.54mm:PinHeader_1x03_P2.54mm_Vertical -> Connector_JST:JST_ZH_B4B-ZR_1x04_P1.50mm_Vertical
- J4: value UART -> USB_C_Receptacle_USB2.0_16P; footprint Connector_PinHeader_2.54mm:PinHeader_1x03_P2.54mm_Vertical -> Connector_USB:USB_C_Receptacle_GCT_USB4105-xx-A_16P_TopMnt_Horizontal
- JP1, JP2: value T:R -> pokayoke; footprint Jumper:SolderJumper-3_P1.3mm_Bridged12_RoundedPad1.0x1.5mm -> Library:pokayoke_1608
- R1, R2, R3, R4, R5, R6, R7, R8: value 1k -> 100R
- R12: value 10k -> R_TNOW
- R13: value 10k -> 4k7
- R9: value 10k -> 1k
- U11: value MCU_DISP -> MCU_DISP_X02
- U12: value MCU_CTL -> CH340E; footprint Package_SO:SOIC-14_3.9x8.7mm_P1.27mm -> Package_SO:MSOP-10_3x3mm_P0.5mm
- U13: value CH340E -> TS5A23159DGS; footprint Package_SO:MSOP-10_3x3mm_P0.5mm -> Package_SO:VSSOP-10_3x3mm_P0.5mm
- moved JP1 77.6 mm to (134.0, 97.0), turned to 45 degrees
- moved JP2 60.2 mm to (66.0, 97.0), turned to 45 degrees
- moved J2 33.8 mm to (140.4, 102.2), turned to 90 degrees
- moved C2 24.4 mm to (128.4, 100.0)
- moved U11 16.0 mm to (117.0, 98.0), turned to 0 degrees
- moved U2 16.0 mm to (96.0, 98.0)
- moved U12 14.2 mm to (134.0, 102.0), turned to 180 degrees
- moved G*** 14.0 mm to (83.0, 100.0), turned to 180 degrees
- moved U1 13.0 mm to (106.0, 98.0)
- moved U13 12.7 mm to (125.8, 100.0)
- moved R13 11.7 mm to (123.0, 100.0)
- moved C3 11.4 mm to (130.0, 100.0), turned to 90 degrees
- moved J1 10.9 mm to (117.0, 103.0)
- moved R9 10.5 mm to (112.4, 98.0)
- moved C1 10.4 mm to (110.8, 98.0), turned to 90 degrees
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Connections:
- C3 pad 2: V3 -> /V3
- D3 pad 2: Net-(D3-A) -> /TNOW
- J1 pad 1: UPDI_DISP -> GND
- J1 pad 2: GND -> UPDI
- J2 pad 3: SDA -> Net-(J2-Pin_3)
- J2 pad 4: SCL -> Net-(J2-Pin_4)
- JP1 pad 1: RXD_CTL -> Net-(J2-Pin_3)
- JP1 pad 2: Net-(J3-Pin_3) -> TXD_DISP|SDA
- JP1 pad 3: RXD_DISP -> Net-(J2-Pin_4)
- JP2 pad 1: RXD_DISP -> Net-(J3-Pin_3)
- JP2 pad 2: Net-(J4-Pin_3) -> TXD_DISP|SDA
- JP2 pad 3: RXD_CTL -> Net-(J3-Pin_4)
- R10 pad 1: Net-(J9-CC1) -> Net-(J4-CC1)
- R11 pad 1: Net-(J9-CC2) -> Net-(J4-CC2)
- R12 pad 1: Net-(D1-DIN) -> Net-(D3-K)
- R12 pad 2: LED_BUILTIN -> GND
- R13 pad 1: Net-(D3-K) -> Net-(R13-Pad1)
- R13 pad 2: GND -> UPDI
- U1 pad 1: /_B -> C6
- U1 pad 15: /_A -> C7
- U1 pad 2: /_C -> C5
- U1 pad 3: /_D -> C4
- U1 pad 4: /_E -> C3
- U1 pad 5: /_F -> C2
- U1 pad 6: /_G -> C1
- U1 pad 7: /_H -> C0
- U11 pad 2: RXD_CTL -> SRCLK
- U11 pad 3: RXD_DISP -> RCLK
- U11 pad 4: SRCLK -> TXD_DISP|SDA
- U11 pad 5: RCLK -> RXD_DISP|SCL
- U11 pad 6: UPDI_DISP -> UPDI
- U12 pad 1: VCC -> D+
- U12 pad 10: UPDI_CTL -> /V3
- U12 pad 2: PA4 -> D-
- U12 pad 3: PA5 -> GND
- U12 pad 4: PA6 -> RTS#
- U12 pad 5: PA7 -> unconnected-(U12-~{CTS}-Pad5)
- U12 pad 6: RXD_CTL -> /TNOW
- U12 pad 7: RXD_DISP -> VCC
- U12 pad 8: SDA -> TXD_USB
- U12 pad 9: SCL -> RXD_USB
- U13 pad 1: D+ -> RTS#
- U13 pad 10: V3 -> TXD_USB
- U13 pad 2: D- -> Net-(R13-Pad1)
- U13 pad 4: unconnected-(U13-~{RTS}-Pad4) -> UPDI
- U13 pad 5: unconnected-(U13-~{CTS}-Pad5) -> RTS#
- U13 pad 6: Net-(D3-A) -> RXD_USB
- U13 pad 7: VCC -> TXD_DISP|SDA
- U13 pad 8: TXD_USB -> VCC
- U13 pad 9: RXD_USB -> RXD_DISP|SCL
- U2 pad 1: C1 -> /_G
- U2 pad 15: C0 -> /_H
- U2 pad 2: C2 -> /_F
- U2 pad 3: C3 -> /_E
- U2 pad 4: C4 -> /_D
- U2 pad 5: C5 -> /_C
- U2 pad 6: C6 -> /_B
- U2 pad 7: C7 -> /_A
- U3 pad 3: unconnected-(U3-CC-Pad3) -> C0
- U3 pad 8: C0 -> unconnected-(U3-CC-Pad8)
Routing:
- net RXD_DISP: track 83.6 -> 0.00 mm, vias 8 -> 0
- net (no net): track 83.2 -> 0.00 mm
- net RXD_DISP|SCL: track 0.00 -> 75.3 mm, vias 0 -> 4
- net TXD_DISP|SDA: track 0.00 -> 75.3 mm, vias 0 -> 4
- net C7: track 83.7 -> 42.8 mm
- net C5: track 55.5 -> 22.7 mm
- net C1: track 15.1 -> 45.9 mm, vias 0 -> 2
- net C6: track 68.2 -> 38.9 mm
- net C4: track 39.9 -> 11.3 mm
- net Net-(J4-Pin_3): track 25.4 -> 0.00 mm, vias 1 -> 0
- net C0: track 34.6 -> 58.6 mm
- net C2: track 8.79 -> 32.4 mm, vias 0 -> 2
- net PA7: track 20.1 -> 0.00 mm
- net SDA: track 15.3 -> 0.00 mm, vias 2 -> 0
- net TXD_CTL_ALT: track 15.1 -> 0.00 mm
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Other:
- board text added: "0u1*2"
- board text added: "100R"
- board text added: "10k"
- board text added: "10n"
- board text added: "1k"
- board text added: "4k7"
- board text added: "74HC595"
- board text added: "ATtinyX02"
- board text added: "CH340E"
- board text added: "DR_TNOW"
- board text added: "G V X Y"
- board text added: "SER RC"
- board text added: "TS5A 23159"
- board text added: "UPDI GND"
- board text added: "Y RXD TXD SCL SDA X"
- board text removed: "595"
- board text removed: "AVR_CTL"
- board text removed: "AVR_DISP"
- board text removed: "CH340 [KE]"
- board text removed: "CTL:DISP"
- board text removed: "G V S"
- board text removed: "GND VCC SDA SCL"
- board text removed: "ISOLATE!"
- board text removed: "PA3"
- board text removed: "PA7"
- board text removed: "R:T"
- board text removed: "RC_SER"
- board text removed: "S V G"
- board text removed: "T:R"
- board text removed: "TNOW"
- board text removed: "UPDI GND UPDI"
