File: proj/avr/tx02/tx02.kicad_sch (KiCad schematic)
At the start: 14 parts, among them J1 USB-C, J2 OUT, SW1 SW_Push, SW2 SW_SPDT, U1 ATtiny202-SS, U2 CH340E

Commit message: -
Parts:
- removed C2: 1F5, Library:edlc, symbol Device:C
- removed J1: USB-C, Library:USB-C, symbol Library:USB-C
- removed R5, R6: 5k1, Resistor_SMD:R_0603_1608Metric, symbol Device:R
- removed SW2: SW_SPDT, Library:sw, symbol Switch:SW_SPDT
- added J3: USB_C_Receptacle_USB2.0_16P, Connector_USB:USB_C_Receptacle_GCT_USB4105-xx-A_16P_TopMnt_Horizontal, symbol Connector:USB_C_Receptacle_USB2.0_16P
- added R3, R4: 4k7, Resistor_SMD:R_0603_1608Metric, symbol Device:R_Small
- added U3: TS5A23159DGS, Package_SO:VSSOP-10_3x3mm_P0.5mm, symbol Analog_Switch:TS5A23159DGS
- renumbered C3 to C2
Connections:
- net D+: now also J3.A6 (D+), J3.B6 (D+)
- net D-: now also J3.A7 (D-), J3.B7 (D-)
- net GND: now also J3.A1 (GND), J3.A12 (GND), J3.B1 (GND), J3.B12 (GND), J3.S1 (SHIELD), R3.2, R4.2, U3.3 (GND)
- net PA6: now also U3.7
- net PA7: now also U3.9
- net UPDI: now also U3.4; no longer U2.9 (RXD)
- net VCC: now also J3.A4 (VBUS), J3.A9 (VBUS), J3.B4 (VBUS), J3.B9 (VBUS), U3.8 (VCC)
- net at R2.1: now also U3.2; no longer U2.8 (TXD)
- net RTS#: now reaches U2.4 (~{RTS})
- net RTS#: now also U3.1, U3.5
- new net: J3.A5 (CC1), R3.1
- new net: J3.B5 (CC2), R4.1
- new net RXD: U2.9 (RXD), U3.6
- new net TXD: U2.8 (TXD), U3.10
Other:
- moved on the sheet: C1, R2
