File: proj/matrix_led/2x1/2x1.kicad_pcb (KiCad board)
At the start: 2 copper layers, 64 x 32 mm, 44 parts, among them J1 I2C, J2 I2C, J3 USB_C_Receptacle_USB2.0_16P, SW1 SW_Push, U1 74HC595, U2 74HC595, U3 74HC595, U4 74HC595, U5 ATtiny202-SS, U6 ATtiny202-SS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

Commit message: -
Parts:
- added ?: LOGO, Library:mcbeeringi_icon_10mm, B.Cu at (127.0, 96.0)
- added ?: , Library:PCB.MCBEERINGI.DEV_small, B.Cu at (126.8, 107.0)
- C2, R20, U7: moved to B.Cu
- JP1: footprint Connector_PinHeader_1.27mm:PinHeader_1x03_P1.27mm_Vertical -> Connector_PinHeader_2.54mm:PinHeader_1x03_P2.54mm_Vertical
- moved R18 65.5 mm to (114.2, 98.4), turned to -90 degrees
- moved R19 65.2 mm to (114.2, 101.6), turned to 90 degrees
- moved C3 34.1 mm to (84.8, 100.0), turned to -90 degrees
- moved C4 30.6 mm to (82.6, 100.0), turned to -90 degrees
- moved SW1 27.2 mm to (87.4, 100.0), turned to 90 degrees
- moved U7 26.0 mm to (80.0, 94.0), turned to 0 degrees
- moved R20 15.7 mm to (75.2, 92.8), turned to 90 degrees
- moved R23 13.1 mm to (71.8, 106.2), turned to 0 degrees
- moved D3 11.6 mm to (73.6, 92.8), turned to -90 degrees
- moved R21 10.0 mm to (72.0, 92.8), turned to 90 degrees
- moved R24 9.05 mm to (74.4, 90.4), turned to 0 degrees
- moved C2 7.27 mm to (70.4, 92.8), turned to -90 degrees
- moved JP1 6.43 mm to (75.5, 108.8), turned to 90 degrees
- moved R22 3.35 mm to (75.0, 106.2)
- moved C1 2.13 mm to (112.6, 101.6)
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Routing:
- net UPDI: track 0.00 -> 24.6 mm
- net /COL14: track 61.2 -> 37.7 mm
- net /COL3: track 58.5 -> 37.4 mm
- net /COL5: track 58.4 -> 38.2 mm
- net /COL6: track 58.1 -> 38.7 mm, vias 2 -> 3
- net /COL11: track 56.2 -> 38.7 mm, vias 2 -> 3
- net /COL12: track 55.6 -> 38.1 mm
- net /COL13: track 55.1 -> 38.0 mm, vias 2 -> 3
- net /RTS#: track 0.00 -> 17.1 mm, vias 0 -> 1
- net /COL4: track 52.5 -> 38.1 mm, vias 2 -> 3
- net /RXD_USB: track 0.00 -> 14.0 mm, vias 0 -> 1
- net UPDI_CTL: track 4.82 -> 18.7 mm, vias 1 -> 2
- net /TXD_USB: track 0.00 -> 12.3 mm, vias 0 -> 1
- net /COL10: track 45.8 -> 37.4 mm, vias 2 -> 1
- net /COL7: track 43.3 -> 36.4 mm, vias 2 -> 1
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Other:
- board text added: "... 3RG 2RG 1RG | 8RG 7RG 6RG ..."
- board text added: "0u1 10k LED 4k7"
- board text added: "1 2 3 ..."
- board text added: "74HC595 *4"
- board text added: "> 4G 4R 3G 3R 2G 2R 1G 1R _ 5R 5G 6R 6G 7R 7G 8R 8G _ A1 A2 A3 A4 A5 A6 A7 A8 _ B1 B2 B3 B4 B5 B6 B7 B8"
- board text added: "AVR_CTL"
- board text added: "AVR_DISP"
- board text added: "B|A"
- board text added: "CH340E"
- board text added: "C_VCC *2"
- board text added: "DISP U CTL"
- board text added: "GVDC"
- board text added: "I2C PULLUP"
- board text added: "JST ZH"
- board text added: "LTP-12188M-07 *2"
- board text added: "NC(U2G)"
- board text added: "PA3"
- board text added: "RC SER"
- board text added: "R_LED *16"
- board text added: "TS5A 23159"
- board text added: "matrix x2 dev board"

Commit message: -
Routing:
- net GND: vias 7 -> 67
