File: proj/amp-spk/amp-spk.kicad_sch (KiCad schematic)
At the start: 13 parts, among them J1 ROUT, J2 LOUT, J3 AudioJack3, J4 ROUT, J5 LOUT, U1 PAM8408D

Commit message: -
Parts:
- removed J4: ROUT, Connector_JST:JST_ZH_B2B-ZR_1x02_P1.50mm_Vertical, symbol Connector:Conn_01x02_Socket
- removed J5: LOUT, Connector_JST:JST_ZH_B2B-ZR_1x02_P1.50mm_Vertical, symbol Connector:Conn_01x02_Socket
- added J6: IN, Connector_JST:JST_ZH_B4B-ZR_1x04_P1.50mm_Vertical, symbol Connector:Conn_01x04_Socket
- added R1: 10k, Resistor_SMD:R_0603_1608Metric, symbol Device:R_Small
- added R2, R3: 0R, Resistor_SMD:R_0603_1608Metric, symbol Device:R_Small
- added SW1, SW2: SW_Push, Library:alps-skrg, symbol Switch:SW_Push
- added SW3: SW_SPDT, Library:sw, symbol Switch:SW_SPDT
- J3: footprint (none) -> Library:MJ-8435
Connections:
- net GND: now also SW1.1, SW2.1, SW3.3 (C)
- net LINN: now also J6.1 (Pin_1)
- net LINP: now also J6.4 (Pin_4)
- net RINN: now also J6.2 (Pin_2)
- net RINP: now also J6.3 (Pin_3)
- net VCC: now also R1.1, R2.2, R3.2; no longer C5.2, C6.2
- net LOUTN: now reaches J2.1 (Pin_1), U1.11 (LOUTN)
- net LOUTP: now reaches J2.2 (Pin_2), U1.10 (LOUTP)
- net ROUTN: now reaches J1.1 (Pin_1), U1.14 (ROUTN)
- net ROUTP: now reaches J1.2 (Pin_2), U1.15 (ROUTP)
- net ~{SD}: now reaches U1.3 (~{SD})
- net ~{SD}: now also SW3.2 (B)
- net UP: now reaches U1.4 (UP)
- net UP: now also SW1.2
- net DN: now reaches U1.5 (DOWN)
- net DN: now also SW2.2
- new net: C6.2, R3.1
- new net: R1.2, SW3.1 (A)
- new net: C5.2, R2.1
- no-connect marks 1 -> 0
Other:
- moved on the sheet: J1, J2
