File: proj/esp/c3-wroom/c3-wroom.kicad_pcb (KiCad board)
At the start: 2 copper layers, 20.3 x 34.3 mm, 13 parts, among them J1 USB-C, J2 Conn_01x08_Pin, J3 Conn_01x01_Pin, J4 Conn_01x08_Pin, U1 ESP32-C3-WROOM-02, U2 LM1117MP-3.3, U3 WS2812C

Commit message: -
Parts:
- removed the ? at (100.0, 89.8)
- removed the G*** at (97.5, 68.2)
- removed the G*** at (102.5, 68.2)
- removed J4: Conn_01x08_Pin, Connector_PinHeader_2.54mm:PinHeader_1x08_P2.54mm_Vertical
- removed U3: WS2812C, Library:WS2812C-2020
- added ?: , Library:PCB.MCBEERINGI.DEV_small, B.Cu at (98.8, 77.8)
- added C1: 1u, Capacitor_SMD:C_0603_1608Metric, F.Cu at (105.2, 79.8)
- added C2: 1u, Capacitor_SMD:C_0603_1608Metric, F.Cu at (100.0, 79.8)
- added D1: WS2812B-2020, LED_SMD:LED_WS2812B-2020_PLCC4_2.0x2.0mm, F.Cu at (97.4, 79.8)
- added G***: LOGO, LOGO, B.Cu at (100.0, 68.8)
- added SW1: SW_BOOT, Library:alps-skrg, F.Cu at (100.0, 85.8)
- J1: value USB-C -> USB_C_Receptacle_USB2.0_16P; footprint Library:USB-C -> Connector_USB:USB_C_Receptacle_GCT_USB4105-xx-A_16P_TopMnt_Horizontal
- J2: value Conn_01x08_Pin -> OUT1; footprint Connector_PinHeader_2.54mm:PinHeader_1x08_P2.54mm_Vertical -> Connector_PinHeader_2.54mm:PinHeader_1x09_P2.54mm_Vertical
- J3: value Conn_01x01_Pin -> OUT2; footprint Connector_PinHeader_2.54mm:PinHeader_1x01_P2.54mm_Vertical -> Connector_PinHeader_2.54mm:PinHeader_1x09_P2.54mm_Vertical
- U1: footprint PCM_Espressif:ESP32-C3-WROOM-02 -> RF_Module:ESP32-C3-WROOM-02
- U2: value LM1117MP-3.3 -> AP7333; footprint Package_TO_SOT_SMD:SOT-223-3_TabPin2 -> Package_TO_SOT_SMD:SOT-23-3
- moved J3 13.9 mm to (108.9, 78.2)
- moved U2 6.75 mm to (102.6, 79.8), turned to -90 degrees
- moved R2 5.83 mm to (97.6, 90.4), turned to 180 degrees
- moved R3 5.83 mm to (102.4, 90.4), turned to 0 degrees
- moved U1 2.86 mm to (100.0, 69.2)
- moved J2 2.74 mm to (91.1, 78.2)
- moved R1 1.80 mm to (94.8, 79.8), turned to -90 degrees
- moved J1 0.78 mm to (100.0, 96.3), turned to 0 degrees
Connections:
- J2 pad 1: +3.3V -> GND
- J2 pad 2: EN -> +3.3V
- J2 pad 3: IO4 -> EN
- J2 pad 4: IO5 -> IO4
- J2 pad 5: IO6 -> IO5
- J2 pad 6: IO7 -> IO6
- J2 pad 7: IO8 -> IO7
- J2 pad 8: IO9 -> IO8
- J3 pad 1: +5V -> GND
- R2 pad 1: Net-(J1-CC2) -> Net-(J1-CC1)
- R3 pad 1: Net-(J1-CC1) -> Net-(J1-CC2)
- U2 pad 1: GND -> VBUS
- U2 pad 3: +5V -> GND
Routing:
- net +5V: track 29.3 -> 0.00 mm, vias 4 -> 0
- net GND: track 12.2 -> 2.72 mm, vias 27 -> 41
- net IO9: track 27.4 -> 34.0 mm, vias 1 -> 2
- net D+: track 36.0 -> 32.3 mm
- net TXD: track 22.6 -> 25.1 mm
- net RXD: track 24.3 -> 26.8 mm
- net IO10: track 25.9 -> 28.5 mm
- net IO5: track 20.8 -> 23.2 mm
- net IO6: track 22.4 -> 24.9 mm
- net IO7: track 24.1 -> 26.6 mm
- net IO2: track 22.3 -> 24.7 mm
- net IO3: track 23.9 -> 26.3 mm
- net IO4: track 19.2 -> 21.6 mm
- net IO0: track 19.1 -> 21.4 mm
- net IO1: track 21.0 -> 23.0 mm
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- added copper zone on F.Cu, net VBUS
- removed copper zone on B.Cu, net +3.3V
Other:
- board size 20.3 x 34.3 mm -> 20.8 x 37.8 mm
- board text added: "ESP32 C3 dev board"
- board text added: "ESP32-C3 WROOM-02"
- board text added: "G V 0 1 2 3 R T a"
- board text added: "G v E 4 5 6 7 8 9"
- board text removed: "G 0 1 2 3 T R a"
- board text removed: "JLCJLCJLCJLC"
- board text removed: "V E 4 5 6 7 8 9"
- board text removed: "Vin"

Commit message: -
Parts:
- J2, J3: moved to B.Cu
- turned J2 to 180 degrees
- turned J3 to 180 degrees

Commit message: -
Parts:
- added SW2: SW_BOOT, Library:alps-skrp, F.Cu at (100.0, 85.8)
- moved ? 1.80 mm to (98.8, 76.0)
- moved G*** 0.80 mm to (100.0, 68.0)
- turned SW1 to -45 degrees
Routing:
- net IO9: track 34.0 -> 37.2 mm, vias 2 -> 3
- net GND: vias 41 -> 38

Commit message: -
Parts:
- removed G***: LOGO, LOGO
- added ?: LOGO, Library:mcbeeringi_icon_10mm, B.Cu at (100.0, 85.6)
- J2, J3: footprint Connector_PinHeader_2.54mm:PinHeader_1x09_P2.54mm_Vertical -> Connector_PinHeader_2.54mm:PinHeader_1x10_P2.54mm_Vertical
- R2, R3: value 5.1k -> 4k7
- moved SW1 23.2 mm to (100.0, 109.0), turned to -135 degrees
- moved SW2 23.2 mm to (100.0, 109.0)
- moved R2 22.4 mm to (96.4, 112.8)
- moved R3 22.4 mm to (103.6, 112.8)
- moved D1 22.4 mm to (100.0, 102.0), turned to 180 degrees
- moved J1 22.1 mm to (100.0, 118.4)
- moved C1 19.4 mm to (102.6, 99.0)
- moved C2 19.4 mm to (97.4, 99.0)
- moved J2 19.2 mm to (91.1, 97.5)
- moved J3 19.2 mm to (108.9, 97.5)
- moved U1 19.2 mm to (100.0, 88.4)
- moved U2 18.4 mm to (100.0, 98.0)
- moved R1 17.6 mm to (95.8, 97.4), turned to 90 degrees
- moved ? 17.2 mm to (100.0, 93.2), turned to -90 degrees
Connections:
- D1 pad 1: unconnected-(D1-DOUT-Pad1) -> NP_OUT
- J2 pad 1: GND -> EN
- J2 pad 3: EN -> GND
- J2 pad 4: IO4 -> VBUS
- J2 pad 5: IO5 -> IO4
- J2 pad 6: IO6 -> IO5
- J2 pad 7: IO7 -> IO6
- J2 pad 8: IO8 -> IO7
- J2 pad 9: IO9 -> IO8
- J3 pad 2: VBUS -> NP_OUT
- J3 pad 3: IO0 -> VBUS
- J3 pad 4: IO1 -> IO0
- J3 pad 5: IO2 -> IO1
- J3 pad 6: IO3 -> IO2
- J3 pad 7: TXD -> IO3
- J3 pad 8: RXD -> TXD
- J3 pad 9: IO10 -> RXD
Routing:
- net NP_OUT: track 0.00 -> 9.03 mm
- net IO9: track 37.2 -> 42.5 mm, vias 3 -> 2
- net EN: track 23.6 -> 19.0 mm
- net IO4: track 21.6 -> 24.8 mm
- net IO1: track 23.0 -> 26.2 mm
- net IO2: track 24.7 -> 27.8 mm
- net IO6: track 24.9 -> 28.0 mm
- net IO3: track 26.3 -> 29.4 mm
- net IO5: track 23.2 -> 26.3 mm
- net IO0: track 21.4 -> 24.4 mm
- net IO7: track 26.6 -> 29.5 mm
- net TXD: track 25.1 -> 28.0 mm
- net RXD: track 26.8 -> 29.6 mm
- net GND: track 2.72 -> 0.00 mm, vias 38 -> 18
- net IO10: track 28.5 -> 31.2 mm
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- added copper zone on B.Cu, net VBUS
Other:
- board size 20.8 x 37.8 mm -> 21 x 41 mm
- board text added: "0"
- board text added: "1"
- board text added: "10"
- board text added: "10k"
- board text added: "1u"
- board text added: "2"
- board text added: "3"
- board text added: "3V3"
- board text added: "4"
- board text added: "4k7"
- board text added: "5"
- board text added: "5V"
- board text added: "6"
- board text added: "7"
- board text added: "8"
- board text added: "9"
- board text added: "@McbeEringi"
- board text added: "ALPS"
- board text added: "AP7333"
- board text added: "EN"
- board text added: "ESP32-C3 dev-board"
- board text added: "GND"
- board text added: "NPO"
- board text added: "RX"
- board text added: "SKRP SKRG"
- board text added: "TX"
- board text added: "WS2812-2020"
- board text removed: "ESP32 C3 dev board"
- board text removed: "ESP32-C3 WROOM-02"
- board text removed: "G V 0 1 2 3 R T a"
- board text removed: "G v E 4 5 6 7 8 9"

Commit message: -
Routing:
- net GND: vias 18 -> 38
Other:
- board text added: "IO8 IO9"
Changed lines of the file:
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@@
+		)
+	)
+	(gr_text "IO8\nIO9"
+		(at 100 104.6 0)
+		(layer "F.SilkS")
+		(effects
+			(font
+				(size 0.8 0.8)
+				(thickness 0.16)
+				(bold yes)
+			)
 		)
 	)
@@
 	)
 	(via
+		(at 91.4 96)
+		(size 0.5)
+		(drill 0.3)
+		(layers "F.Cu" "B.Cu")
+		(free yes)
+		(net 1)
+	)
+	(via
+		(at 96 111)
+		(size 0.5)
+		(drill 0.3)
+		(layers "F.Cu" "B.Cu")
+		(free yes)
+		(net 1)
+	)
+	(via
 		(at 96 107)
 		(size 0.5)
@@
 	)
 	(via
+		(at 109.6 96)
+		(size 0.5)
+		(drill 0.3)
+		(layers "F.Cu" "B.Cu")
+		(free yes)
+		(net 1)
+	)
+	(via
+		(at 100 95)
+		(size 0.5)
+		(drill 0.3)
+		(layers "F.Cu" "B.Cu")
+		(free yes)
+		(net 1)
+	)
+	(via
 		(at 103.8 101)
 		(size 0.5)
@@
 	)
 	(via
+		(at 90.4 96)
+		(size 0.5)
+		(drill 0.3)
+		(layers "F.Cu" "B.Cu")
+		(free yes)
+		(net 1)
+	)
+	(via
 		(at 103.2 114.4)
 		(size 0.5)
@@
 	)
 	(via
+		(at 98 81.8)
+		(size 0.5)
+		(drill 0.3)
+		(layers "F.Cu" "B.Cu")
+		(free yes)
+		(net 1)
+	)
+	(via
+		(at 106 81.8)
+		(size 0.5)
+		(drill 0.3)
+		(layers "F.Cu" "B.Cu")
+		(free yes)
+		(net 1)
+	)
+	(via
+		(at 104 111)
+		(size 0.5)
+		(drill 0.3)
+		(layers "F.Cu" "B.Cu")
+		(free yes)
+		(net 1)
+	)
+	(via
 		(at 103.8 107)
 		(size 0.5)
@@
 	)
 	(via
+		(at 93.4 83.6)
+		(size 0.5)
+		(drill 0.3)
+		(layers "F.Cu" "B.Cu")
+		(free yes)
+		(net 1)
+	)
+	(via
 		(at 96.8 115)
 		(size 0.5)
@@
 	)
 	(via
+		(at 102 81.8)
+		(size 0.5)
+		(drill 0.3)
+		(layers "F.Cu" "B.Cu")
+		(free yes)
+		(net 1)
+	)
+	(via
 		(at 96 95)
 		(size 0.5)
@@
 	)
 	(via
+		(at 98 121.2)
+		(size 0.5)
+		(drill 0.3)
+		(layers "F.Cu" "B.Cu")
+		(free yes)
+		(net 1)
+	)
+	(via
+		(at 94 121.2)
+		(size 0.5)
+		(drill 0.3)
+		(layers "F.Cu" "B.Cu")
+		(free yes)
+		(net 1)
+	)
+	(via
+		(at 100 94)
+		(size 0.5)
+		(drill 0.3)
+		(layers "F.Cu" "B.Cu")
+		(free yes)
+		(net 1)
+	)
+	(via
 		(at 97 107)
 		(size 0.5)
@@
 	)
 	(via
+		(at 108.2 96)
+		(size 0.5)
+		(drill 0.3)
+		(layers "F.Cu" "B.Cu")
+		(free yes)
+		(net 1)
+	)
+	(via
+		(at 94 81.8)
+		(size 0.5)
+		(drill 0.3)
+		(layers "F.Cu" "B.Cu")
+		(free yes)
+		(net 1)
+	)
+	(via
+		(at 94.4 88)
+		(size 0.5)
+		(drill 0.3)
+		(layers "F.Cu" "B.Cu")
+		(free yes)
+		(net 1)
+	)
+	(via
 		(at 98 103)
 		(size 0.5)
@@
 	)
 	(via
+		(at 101.8 111)
+		(size 0.5)
+		(drill 0.3)
+		(layers "F.Cu" "B.Cu")
+		(free yes)
+		(net 1)
+	)
+	(via
 		(at 102 101)
 		(size 0.5)
@@
 	)
 	(via
+		(at 105.8 88)
+		(size 0.5)
+		(drill 0.3)
+		(layers "F.Cu" "B.Cu")
+		(free yes)
+		(net 1)
+	)
+	(via
 		(at 102 103)
 		(size 0.5)
@@
 	)
 	(via
+		(at 102 121.2)
+		(size 0.5)
+		(drill 0.3)
+		(layers "F.Cu" "B.Cu")
+		(free yes)
+		(net 1)
+	)
+	(via
 		(at 96 94)
 		(size 0.5)
@@
 		(drill 0.3)
 		(layers "F.Cu" "B.Cu")
+		(net 1)
+	)
+	(via
+		(at 106 121.2)
+		(size 0.5)
+		(drill 0.3)
+		(layers "F.Cu" "B.Cu")
+		(free yes)
 		(net 1)
 	)
@@
 		(polygon
 			(pts
-				(xy 88.8 106.4) (xy 106 106.4) (xy 108.4 104) (xy 112.2 104) (xy 112.2 101) (xy 108 101) (xy 105 104)
-				(xy 88.8 104)
+				(xy 89.4 106.4) (xy 106 106.4) (xy 108.4 104) (xy 110.6 104) (xy 110.6 101) (xy 108 101) (xy 105 104)
+				(xy 89.4 104)
 			)
 		)
@@
 		(polygon
 			(pts
-				(xy 89.4 96.6) (xy 97 96.6) (xy 97 95.6) (xy 93.8 82.8) (xy 90.4 82.8) (xy 90.4 82) (xy 95.8 82)
-				(xy 99 94.8) (xy 99 95) (xy 99.8 95.8) (xy 99.8 98.2) (xy 98.8 99.2) (xy 94.2 99.2) (xy 92.2 101.2)
-				(xy 89.4 101.2)
+				(xy 89.4 96.6) (xy 97 96.6) (xy 97 95.8) (xy 93.8 83) (xy 90.4 83) (xy 90.4 82) (xy 95.8 82) (xy 99 94.8)
+				(xy 99 95) (xy 99.8 95.8) (xy 99.8 98.2) (xy 98.8 99.2) (xy 94.2 99.2) (xy 92.2 101.2) (xy 89.4 101.2)
 			)
 		)
