File: proj/esp/c3-wroom/c3-wroom.kicad_sch (KiCad schematic)
At the start: 10 parts, among them J1 USB-C, J2 Conn_01x08_Pin, J3 Conn_01x01_Pin, J4 Conn_01x08_Pin, U1 ESP32-C3-WROOM-02, U2 LM1117MP-3.3, U3 WS2812C

Commit message: -
Parts:
- removed J1: USB-C, Library:USB-C, symbol Library:USB-C
- removed J3: Conn_01x01_Pin, Connector_PinHeader_2.54mm:PinHeader_1x01_P2.54mm_Vertical, symbol Connector:Conn_01x01_Pin
- removed J4: Conn_01x08_Pin, Connector_PinHeader_2.54mm:PinHeader_1x08_P2.54mm_Vertical, symbol Connector:Conn_01x08_Pin
- removed U2: LM1117MP-3.3, Package_TO_SOT_SMD:SOT-223-3_TabPin2, symbol Regulator_Linear:LM1117MP-3.3
- removed U3: WS2812C, Library:WS2812C-2020, symbol Library:WS2812C-2020
- added C1, C2: 1u, Capacitor_SMD:C_0603_1608Metric, symbol Device:C_Small
- added D1: WS2812B-2020, LED_SMD:LED_WS2812B-2020_PLCC4_2.0x2.0mm, symbol LED:WS2812B-2020
- added J1: USB_C_Receptacle_USB2.0_16P, Connector_USB:USB_C_Receptacle_GCT_USB4105-xx-A_16P_TopMnt_Horizontal, symbol Connector:USB_C_Receptacle_USB2.0_16P
- added J3: OUT2, Connector_PinHeader_2.54mm:PinHeader_1x09_P2.54mm_Vertical, symbol Connector:Conn_01x09_Pin
- added SW1: SW_BOOT, Library:alps-skrg, symbol Switch:SW_Push
- added U2: AP7333, Package_TO_SOT_SMD:SOT-23-3, symbol Library:AP7333
- J2: value Conn_01x08_Pin -> OUT1; footprint Connector_PinHeader_2.54mm:PinHeader_1x08_P2.54mm_Vertical -> Connector_PinHeader_2.54mm:PinHeader_1x09_P2.54mm_Vertical; symbol Connector:Conn_01x08_Pin -> Connector:Conn_01x09_Pin
- U1: footprint PCM_Espressif:ESP32-C3-WROOM-02 -> RF_Module:ESP32-C3-WROOM-02
Connections:
- net +3.3V: now also J2.2 (Pin_2), C2.1, U2.2 (OUT); no longer J2.1 (Pin_1)
- net D+: now also J1.A6 (D+), J1.B6 (D+)
- net D-: now also J1.A7 (D-), J1.B7 (D-)
- net EN: now also J2.3 (Pin_3); no longer J2.2 (Pin_2)
- net GND: now also J2.1 (Pin_1), C1.2, C2.2, D1.2 (VSS), J1.A1 (GND), J1.A12 (GND), J1.B1 (GND), J1.B12 (GND), J1.S1 (SHIELD), J3.1 (Pin_1), SW1.2, U2.3 (GND)
- net IO0: now also J3.3 (Pin_3)
- net IO1: now also J3.4 (Pin_4)
- net IO10: now also J3.9 (Pin_9)
- net IO2: now also J3.5 (Pin_5)
- net IO3: now also J3.6 (Pin_6)
- net IO4: now also J2.4 (Pin_4); no longer J2.3 (Pin_3)
- net IO5: now also J2.5 (Pin_5); no longer J2.4 (Pin_4)
- net IO6: now also J2.6 (Pin_6); no longer J2.5 (Pin_5)
- net IO7: now also J2.7 (Pin_7); no longer J2.6 (Pin_6)
- net IO8: now also J2.8 (Pin_8), D1.3 (DIN); no longer J2.7 (Pin_7)
- net IO9: now also J2.9 (Pin_9), SW1.1; no longer J2.8 (Pin_8)
- net RXD: now also J3.8 (Pin_8)
- net TXD: now also J3.7 (Pin_7)
- net at R3.1: now also J1.B5 (CC2)
- net at R2.1: now also J1.A5 (CC1)
- new net VBUS: C1.1, D1.4 (VDD), J1.A4 (VBUS), J1.A9 (VBUS), J1.B4 (VBUS), J1.B9 (VBUS), J3.2 (Pin_2), U2.1 (IN)
- no-connect marks 0 -> 3
Other:
- moved on the sheet: R1, R2, R3

Commit message: -
Parts:
- added SW2: SW_BOOT, Library:alps-skrp, symbol Switch:SW_Push
Connections:
- net GND: now also SW2.2
- net IO9: now also SW2.1
Changed lines of the file:
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@@
+	)
+	(junction
+		(at 82.55 153.67)
+		(diameter 0)
+		(color 0 0 0 0)
 	)
 	(junction
@@
 		(pts
 			(xy 58.42 115.57) (xy 58.42 118.11)
+		)
+		(stroke
+			(width 0)
+			(type default)
+		)
+	)
+	(wire
+		(pts
+			(xy 82.55 153.67) (xy 82.55 156.21)
+		)
+		(stroke
+			(width 0)
+			(type default)
+		)
+	)
+	(wire
+		(pts
+			(xy 72.39 153.67) (xy 72.39 156.21)
 		)
 		(stroke
@@
 					(unit 1)
 				)
+			)
+		)
+	)
+	(symbol
+		(lib_id "Switch:SW_Push")
+		(at 77.47 156.21 0)
+		(mirror x)
+		(unit 1)
+		(exclude_from_sim no)
+		(in_bom yes)
+		(on_board yes)
+		(dnp no)
+		(property "Reference" "SW2"
+			(at 77.47 163.83 0)
+			(effects
+				(font
+					(size 1.27 1.27)
+				)
+			)
+		)
+		(property "Value" "SW_BOOT"
+			(at 77.47 161.29 0)
+			(effects
+				(font
+					(size 1.27 1.27)
+				)
+			)
+		)
+		(property "Footprint" "Library:alps-skrp"
+			(at 77.47 161.29 0)
+			(effects
+				(font
+					(size 1.27 1.27)
+				)
+				(hide yes)
+			)
+		)
+		(property "Datasheet" "~"
+			(at 77.47 161.29 0)
+			(effects
+				(font
+					(size 1.27 1.27)
+				)
+				(hide yes)
+			)
+		)
+		(property "Description" "Push button switch, generic, two pins"
+			(at 77.47 156.21 0)
+			(effects
+				(font
+					(size 1.27 1.27)
+				)
+				(hide yes)
+			)
+		)
+		(pin "2"
+		)
+		(pin "1"
+		)
+		(instances
+			(project "c3-wroom"
+				(path "/c16d87cc-6731-400b-81e0-d0681fc8ad9f"
+					(reference "SW2")
+					(unit 1)
+				)

Commit message: -
Parts:
- removed J2: OUT1, Connector_PinHeader_2.54mm:PinHeader_1x09_P2.54mm_Vertical, symbol Connector:Conn_01x09_Pin
- removed J3: OUT2, Connector_PinHeader_2.54mm:PinHeader_1x09_P2.54mm_Vertical, symbol Connector:Conn_01x09_Pin
- added J2: OUT1, Connector_PinHeader_2.54mm:PinHeader_1x10_P2.54mm_Vertical, symbol Connector:Conn_01x10_Pin
- added J3: OUT2, Connector_PinHeader_2.54mm:PinHeader_1x10_P2.54mm_Vertical, symbol Connector:Conn_01x10_Pin
- R2, R3: value 5.1k -> 4k7
Connections:
- net +3.3V: now also J2.2 (Pin_2)
- net EN: now also J2.1 (Pin_1)
- net GND: now also J2.3 (Pin_3), J3.1 (Pin_1)
- net IO0: now also J3.4 (Pin_4)
- net IO1: now also J3.5 (Pin_5)
- net IO10: now also J3.10 (Pin_10)
- net IO2: now also J3.6 (Pin_6)
- net IO3: now also J3.7 (Pin_7)
- net IO4: now also J2.5 (Pin_5)
- net IO5: now also J2.6 (Pin_6)
- net IO6: now also J2.7 (Pin_7)
- net IO7: now also J2.8 (Pin_8)
- net IO8: now also J2.9 (Pin_9)
- net IO9: now also J2.10 (Pin_10)
- net RXD: now also J3.9 (Pin_9)
- net TXD: now also J3.8 (Pin_8)
- net VBUS: now also J2.4 (Pin_4), J3.3 (Pin_3)
- net NP_OUT: now reaches D1.1 (DOUT)
- net NP_OUT: now also J3.2 (Pin_2)
- no-connect marks 3 -> 2
