File: proj/ir_remote/cosmo_wide21/cosmo_wide21.kicad_pcb (KiCad board)
At the start: 2 copper layers, 42.4 x 91.2 mm, 12 parts, among them J1 UPDI, Q1 BSS138, SW1 BTN1, U1 ATtiny202-SS

Commit message: -
Parts:
- added C2: 4u7, Capacitor_SMD:C_0603_1608Metric, B.Cu at (117.6, 61.2)
- moved D1 22.4 mm to (96.9, 65.1)
- moved D3 22.4 mm to (83.7, 65.1)
- moved D2 22.4 mm to (90.3, 65.1)
Connections:
- net Net-(D1-A) renamed /LED12
- net Net-(D2-A) renamed /LED23
- BT1 pad 1: Net-(BT1-+) -> VCC
- BT2 pad 1: VCC -> +6V
- BT2 pad 2: Net-(BT1-+) -> VCC
- D3 pad 2: VCC -> +6V
Routing:
- added copper zone on B.Cu, net +6V
- added copper zone on B.Cu, net /LED12
- added copper zone on B.Cu, net /LED23
- added copper zone on B.Cu, net VCC

Commit message: -
Parts:
- added H1: MountingHole, MountingHole:MountingHole_3.2mm_M3, F.Cu at (84.0, 84.0)
- added H2: MountingHole, MountingHole:MountingHole_3.2mm_M3, F.Cu at (84.0, 116.0)
- J1: moved to B.Cu
- moved J1 31.9 mm to (87.7, 68.0), turned to -90 degrees
- moved C2 24.6 mm to (93.0, 62.0), turned to 0 degrees
- moved Q1 20.4 mm to (98.0, 62.0), turned to 180 degrees
- moved U1 9.53 mm to (104.0, 64.0), turned to 180 degrees
- moved C1 7.38 mm to (104.0, 60.4), turned to 180 degrees
Routing:
- net BTN1: track 0.00 -> 46.6 mm, vias 0 -> 2
- net UPDI: track 0.00 -> 13.3 mm
- net WO: track 0.00 -> 3.71 mm
- net GND: vias 0 -> 26
- added copper zone on B.Cu, net /LED

Commit message: -
Parts:
- moved H1 12.0 mm to (84.0, 72.0)
- moved H2 12.0 mm to (84.0, 128.0)
Other:
- board text added: "4u7"
- board text added: "ALPS SKRG"
- board text added: "ATtinyX02"
- board text added: "BC-2001"
- board text added: "BSS138"
- board text added: "GND"
- board text added: "PA1"
- board text added: "PA3"
- board text added: "UPDI"
Changed lines of the file:
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@@
 	(footprint "MountingHole:MountingHole_3.2mm_M3"
 		(layer "F.Cu")
-		(at 84 116)
+		(at 84 128)
 		(descr "Mounting Hole 3.2mm, M3, no annular, generated by kicad-footprint-generator mountinghole.py")
 		(tags "mountinghole M3")
@@
 	(footprint "MountingHole:MountingHole_3.2mm_M3"
 		(layer "F.Cu")
-		(at 84 84)
+		(at 84 72)
 		(descr "Mounting Hole 3.2mm, M3, no annular, generated by kicad-footprint-generator mountinghole.py")
 		(tags "mountinghole M3")
@@
 		(layer "B.Fab")
 	)
+	(gr_text "ATtinyX02"
+		(at 104 64 90)
+		(layer "B.Mask")
+		(effects
+			(font
+				(size 0.5 0.5)
+				(thickness 0.1)
+				(bold yes)
+			)
+			(justify mirror)
+		)
+	)
+	(gr_text "PA3"
+		(at 98 58.4 0)
+		(layer "B.Mask")
+		(effects
+			(font
+				(size 0.5 0.5)
+				(thickness 0.1)
+				(bold yes)
+			)
+			(justify mirror)
+		)
+	)
+	(gr_text "4u7"
+		(at 93 61 0)
+		(layer "B.Mask")
+		(effects
+			(font
+				(size 0.5 0.5)
+				(thickness 0.1)
+				(bold yes)
+			)
+			(justify mirror)
+		)
+	)
+	(gr_text "ALPS SKRG"
+		(at 118 100 0)
+		(layer "B.Mask")
+		(effects
+			(font
+				(size 0.5 0.5)
+				(thickness 0.1)
+				(bold yes)
+			)
+			(justify mirror)
+		)
+	)
+	(gr_text "UPDI"
+		(at 90.2 70.2 0)
+		(layer "B.Mask")
+		(effects
+			(font
+				(size 0.5 0.5)
+				(thickness 0.1)
+				(bold yes)
+			)
+			(justify mirror)
+		)
+	)
 	(gr_text "IR Remote\ncosmo_wide21"
 		(at 100 108 0)
@@
 		)
 	)
+	(gr_text "BC-2001"
+		(at 86 118 0)
+		(layer "B.Mask")
+		(effects
+			(font
+				(size 0.5 0.5)
+				(thickness 0.1)
+				(bold yes)
+			)
+			(justify mirror)
+		)
+	)
+	(gr_text "BC-2001"
+		(at 86 82 0)
+		(layer "B.Mask")
+		(effects
+			(font
+				(size 0.5 0.5)
+				(thickness 0.1)
+				(bold yes)
+			)
+			(justify mirror)
+		)
+	)
+	(gr_text "4u7"
+		(at 104 59.2 0)
+		(layer "B.Mask")
+		(effects
+			(font
+				(size 0.5 0.5)
+				(thickness 0.1)
+				(bold yes)
+			)
+			(justify mirror)
+		)
+	)
+	(gr_text "GND"
+		(at 87.8 70.2 0)
+		(layer "B.Mask")
+		(effects
+			(font
+				(size 0.5 0.5)
+				(thickness 0.1)
+				(bold yes)
+			)
+			(justify mirror)
+		)
+	)
+	(gr_text "BSS138"
+		(at 98 59.4 0)
+		(layer "B.Mask")
+		(effects
+			(font
+				(size 0.5 0.5)
+				(thickness 0.1)
+				(bold yes)
+			)
+			(justify mirror)
+		)
+	)
+	(gr_text "PA1"
+		(at 118 96 0)
+		(layer "B.Mask")
+		(effects
+			(font
+				(size 0.5 0.5)
+				(thickness 0.1)
+				(bold yes)
+			)
+			(justify mirror)
+		)
+	)
 	(via
 		(at 118 88)
@@
 	)
 	(segment
-		(start 101.49 64.6)
-		(end 99.2 64.6)
+		(start 98.8 65)
+		(end 98.8 66.2)
 		(width 0.2)
 		(layer "B.Cu")
@@
 	)
 	(segment
-		(start 91.2 67)
-		(end 90.265 67.935)
+		(start 98.8 66.2)
+		(end 98 67)
 		(width 0.2)
 		(layer "B.Cu")
@@
 	)
 	(segment
-		(start 97.8 67)
+		(start 98 67)
 		(end 91.2 67)
 		(width 0.2)
@@
 	)
 	(segment
-		(start 98.8 65)
-		(end 98.8 66)
+		(start 101.49 64.6)
+		(end 99.2 64.6)
 		(width 0.2)
 		(layer "B.Cu")
@@
 	)
 	(segment
-		(start 98.8 66)
-		(end 97.8 67)
+		(start 91.2 67)
+		(end 90.265 67.935)
 		(width 0.2)
 		(layer "B.Cu")
