File: proj/card/25led/25led.kicad_pcb (KiCad board)
At the start: 2 copper layers, 100 x 80 mm, 43 parts, among them U1 ATtiny404-SS

Commit message: -
Parts:
- added J1: UPDI, Connector_PinSocket_2.54mm:PinSocket_1x02_P2.54mm_Vertical, B.Cu at (98.8, 133.6)
- added SW1: SW_SPDT, Button_Switch_THT:SW_Slide_SPDT_Straight_CK_OS102011MS2Q, B.Cu at (99.0, 144.8)
- moved D20 90.0 mm to (55.0, 70.0), turned to 180 degrees
- moved D5 90.0 mm to (145.0, 130.0), turned to 0 degrees
- moved D19 70.0 mm to (65.0, 70.0), turned to 180 degrees
- moved D4 70.0 mm to (135.0, 130.0), turned to 0 degrees
- moved D26 64.0 mm to (95.0, 130.0)
- moved D6 64.0 mm to (145.0, 80.0)
- moved D15 50.0 mm to (145.0, 70.0)
- moved D18 50.0 mm to (75.0, 70.0), turned to 180 degrees
- moved D25 50.0 mm to (55.0, 120.0)
- moved D27 50.0 mm to (85.0, 130.0)
- moved D3 50.0 mm to (125.0, 130.0), turned to 0 degrees
- moved D7 50.0 mm to (145.0, 90.0)
- moved D11 41.2 mm to (105.0, 70.0)
- moved D14 41.2 mm to (135.0, 70.0)
- moved D21 41.2 mm to (55.0, 80.0)
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Connections:
- BT1 pad 1: VCC -> +BATT
- BT2 pad 1: VCC -> +BATT
- U1 pad 11: ROW1 -> ROW2
- U1 pad 12: ROW2 -> ROW1
Routing:
- net /_COL5: track 154.3 -> 100.5 mm
- net /_COL6: track 102.4 -> 49.6 mm
- net /_COL3: track 101.9 -> 153.2 mm
- net /_COL2: track 50.8 -> 100.5 mm
- net UPDI: track 0.00 -> 9.77 mm
- net /_COL4: track 159.0 -> 153.2 mm
- net /_COL1: track 53.7 -> 49.6 mm
- net ROW4: track 248.3 -> 245.5 mm
- net ROW5: track 230.7 -> 228.4 mm
- net ROW2: track 276.4 -> 274.5 mm
- net ROW3: track 264.5 -> 262.8 mm
- net COL5: track 8.17 -> 7.12 mm
- net COL4: track 3.36 -> 2.34 mm
- net COL1: track 2.97 -> 1.96 mm
- net COL2: track 2.84 -> 1.98 mm
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- added copper zone on B.Cu, net +BATT

Commit message: -
Parts:
- SW1: footprint Button_Switch_THT:SW_Slide_SPDT_Straight_CK_OS102011MS2Q -> Library:sw_tht
- moved SW1 22.6 mm to (83.6, 128.2)
Connections:
- SW1 pad 2: +BATT -> VCC
- SW1 pad 3: VCC -> +BATT
