File: proj/card/25led/25led.kicad_sch (KiCad schematic)
At the start: 41 parts, among them U1 ATtiny404-SS

Commit message: -
Parts:
- added J1: UPDI, Connector_PinSocket_2.54mm:PinSocket_1x02_P2.54mm_Vertical, symbol Connector:Conn_01x02_Socket
- added SW1: SW_SPDT, Button_Switch_THT:SW_Slide_SPDT_Straight_CK_OS102011MS2Q, symbol Switch:SW_SPDT
Connections:
- net GND: now also J1.1 (Pin_1)
- net ROW1: now also U1.12 (PA2); no longer U1.11 (PA1)
- net ROW2: now also U1.11 (PA1); no longer U1.12 (PA2)
- net UPDI: now also J1.2 (Pin_2)
- net VCC: now also SW1.3 (C); no longer BT1.1 (+), BT2.1 (+)
- new net +BATT: BT1.1 (+), BT2.1 (+), SW1.2 (B)
- no-connect marks 0 -> 1

Commit message: -
Parts:
- SW1: footprint Button_Switch_THT:SW_Slide_SPDT_Straight_CK_OS102011MS2Q -> Library:sw_tht
Connections:
- net +BATT: now also SW1.3 (C); no longer SW1.2 (B)
- net VCC: now also SW1.2 (B); no longer SW1.3 (C)
Changed lines of the file:
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@@
 	(symbol
 		(lib_id "power:+BATT")
-		(at 24.13 109.22 90)
+		(at 34.29 111.76 270)
 		(unit 1)
 		(exclude_from_sim no)
@@
 		(fields_autoplaced yes)
 		(property "Reference" "#PWR013"
-			(at 27.94 109.22 0)
+			(at 30.48 111.76 0)
 			(effects
 				(font
@@
 		)
 		(property "Value" "+BATT"
-			(at 20.32 109.2199 90)
+			(at 38.1 111.7599 90)
 			(effects
 				(font
@@
 		)
 		(property "Footprint" ""
-			(at 24.13 109.22 0)
+			(at 34.29 111.76 0)
 			(effects
 				(font
@@
 		)
 		(property "Datasheet" ""
-			(at 24.13 109.22 0)
+			(at 34.29 111.76 0)
 			(effects
 				(font
@@
 		)
 		(property "Description" "Power symbol creates a global label with name \"+BATT\""
-			(at 24.13 109.22 0)
+			(at 34.29 111.76 0)
 			(effects
 				(font
@@
 	(symbol
 		(lib_id "power:VCC")
-		(at 34.29 111.76 270)
+		(at 24.13 109.22 90)
 		(unit 1)
 		(exclude_from_sim no)
@@
 		(fields_autoplaced yes)
 		(property "Reference" "#PWR014"
-			(at 30.48 111.76 0)
+			(at 27.94 109.22 0)
 			(effects
 				(font
@@
 		)
 		(property "Value" "VCC"
-			(at 38.1 111.7599 90)
-			(effects
-				(font
-					(size 1.27 1.27)
-				)
-				(justify left)
+			(at 22.86 106.68 90)
+			(effects
+				(font
+					(size 1.27 1.27)
+				)
 			)
 		)
 		(property "Footprint" ""
-			(at 34.29 111.76 0)
+			(at 24.13 109.22 0)
 			(effects
 				(font
@@
 		)
 		(property "Datasheet" ""
-			(at 34.29 111.76 0)
+			(at 24.13 109.22 0)
 			(effects
 				(font
@@
 		)
 		(property "Description" "Power symbol creates a global label with name \"VCC\""
-			(at 34.29 111.76 0)
+			(at 24.13 109.22 0)
 			(effects
 				(font
@@
 			)
 		)
-		(property "Footprint" "Button_Switch_THT:SW_Slide_SPDT_Straight_CK_OS102011MS2Q"
+		(property "Footprint" "Library:sw_tht"
 			(at 29.21 109.22 0)
 			(effects
