File: proj/usb/pd-fix/pd-fix.kicad_pcb (KiCad board)
At the start: 2 copper layers, 10 x 10 mm, 9 parts, among them J1 USB_C_Receptacle_PowerOnly_6P, J2 Conn_01x02_Pin, U1 CH221K

Commit message: -
Parts:
- removed G***: LOGO, LOGO
- added D1: PG, LED_SMD:LED_0603_1608Metric, F.Cu at (103.6, 96.2)
- added R5: 10k, Resistor_SMD:R_0603_1608Metric, B.Cu at (103.6, 96.2)
- J1: value USB_C_Receptacle_PowerOnly_6P -> USB_C_Receptacle_USB2.0_16P; footprint Connector_USB:USB_C_Receptacle_GCT_USB4125-xx-x_6P_TopMnt_Horizontal -> Connector_USB:USB_C_Receptacle_GCT_USB4105-xx-A_16P_TopMnt_Horizontal
- J2: footprint Connector_PinHeader_2.54mm:PinHeader_1x02_P2.54mm_Vertical -> Library:SolderPad_2P; moved to B.Cu
- moved R2 8.17 mm to (96.4, 103.2)
- moved R4 7.09 mm to (96.4, 98.4), turned to 180 degrees
- moved R3 6.44 mm to (96.4, 101.6), turned to 180 degrees
- moved C1 3.78 mm to (96.4, 100.0)
- moved J1 2.80 mm to (97.2, 100.0)
- moved J2 2.67 mm to (103.4, 100.0), turned to 0 degrees
- moved R1 2.64 mm to (96.4, 96.8), turned to 0 degrees
- moved U1 0.10 mm to (99.6, 100.0), turned to -90 degrees
Connections:
- U1 pad 3: unconnected-(U1-PG#-Pad3) -> Net-(U1-PG#)
Routing:
- net VBUS: track 1.28 -> 12.6 mm, vias 1 -> 3
- net VDD: track 7.53 -> 0.00 mm, vias 2 -> 0
- net CC1: track 5.07 -> 11.4 mm
- net Net-(U1-PG#): track 0.00 -> 3.78 mm
- net Net-(U1-CFG): track 2.68 -> 5.03 mm
- net CC2: track 3.74 -> 5.07 mm
- net Net-(D1-K): vias 0 -> 1
- added copper zone on B.Cu, net VDD
Other:
- board size 10 x 10 mm -> 11 x 11 mm
- board text added: "103 5 473 12 203 9 104 15 204 20"
- board text added: "1k ~0.28W CFG 1u 4k7 4k7"
- board text added: "@Mcbe Eringi"
- board text added: "PD TRG FIXED"
- board text removed: "PD FIX"

Commit message: -
Parts:
- removed D1: PG, LED_SMD:LED_0603_1608Metric
- removed R5: 10k, Resistor_SMD:R_0603_1608Metric
Connections:
- U1 pad 3: Net-(U1-PG#) -> unconnected-(U1-PG#-Pad3)
Routing:
- net Net-(U1-PG#): track 3.78 -> 0.00 mm
- net Net-(D1-K): vias 1 -> 0

Commit message: -
Other:
- board text added: "CH221K FIXED PD TRG"
- board text removed: "PD TRG FIXED"
Changed lines of the file:
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@@
 		)
 	)
-	(gr_text "PD TRG\nFIXED"
-		(at 103.2 96 -0)
+	(gr_text "CH221K\nFIXED\nPD TRG"
+		(at 103.4 96.2 0)
 		(layer "B.Mask")
 		(effects
 			(font
-				(size 0.6 0.6)
-				(thickness 0.12)
+				(size 0.5 0.5)
+				(thickness 0.1)
 				(bold yes)
 			)

Commit message: -
Other:
- board text added: "CH221K PD-FIX"
- board text removed: "CH221K FIXED PD TRG"
Changed lines of the file:
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@@
 		)
 	)
-	(gr_text "CH221K\nFIXED\nPD TRG"
+	(gr_text "CH221K\nPD-FIX"
 		(at 103.4 96.2 0)
 		(layer "B.Mask")

Commit message: -
Other:
- board size 11 x 11 mm -> 11 x 10 mm
Changed lines of the file:
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@@
 	)
 	(gr_line
-		(start 94.5 94.5)
-		(end 94.5 105.5)
+		(start 94.5 95)
+		(end 94.5 105)
 		(stroke
 			(width 0.05)
@@
 	)
 	(gr_line
-		(start 105.5 94.5)
-		(end 94.5 94.5)
+		(start 105.5 95)
+		(end 94.5 95)
 		(stroke
 			(width 0.05)
@@
 	)
 	(gr_line
-		(start 94.5 105.5)
-		(end 105.5 105.5)
+		(start 94.5 105)
+		(end 105.5 105)
 		(stroke
 			(width 0.05)
@@
 	)
 	(gr_line
-		(start 105.5 105.5)
-		(end 105.5 94.5)
+		(start 105.5 105)
+		(end 105.5 95)
 		(stroke
 			(width 0.05)
@@
 	)
 	(gr_text "@Mcbe\n Eringi"
-		(at 103.4 103.8 -0)
+		(at 103.4 103.6 180)
 		(layer "B.Mask")
 		(effects
@@
 	)
 	(gr_text "CH221K\nPD-FIX"
-		(at 103.4 96.2 0)
+		(at 103.4 96.4 0)
 		(layer "B.Mask")
 		(effects
@@
 		(polygon
 			(pts
-				(xy 94 94) (xy 106 94) (xy 106 106) (xy 94 106)
-			)
-		)
+				(xy 94 94.6) (xy 106 94.6) (xy 106 105.4) (xy 94 105.4)
+			)
+		)

Commit message: -
Routing:
- net GND: vias 3 -> 5
Changed lines of the file:
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@@
+	)
+	(via
+		(at 95.575 103.2)
+		(size 0.5)
+		(drill 0.3)
+		(layers "F.Cu" "B.Cu")
+		(net 2)
 	)
 	(via
@@
 		(size 0.5)
 		(drill 0.3)
+		(layers "F.Cu" "B.Cu")
+		(net 2)
+	)
+	(via
+		(at 95.625 100)
+		(size 0.5)
+		(drill 0.3)
