File: proj/audio/amp/pam8408/pam8408.kicad_pcb (KiCad board)
At the start: 2 copper layers, 36 x 18 mm, 15 parts, among them J1 ROUT, J2 LOUT, J3 AudioJack3, J4 PWR, SW1 VOL_UP, SW2 VOL_DOWN, U1 PAM8408D

Commit message: -
Other:
- board text added: "MJ-8435"
Changed lines of the file:
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@@
 		(layer "Edge.Cuts")
+	)
+	(gr_text "MJ-8435"
+		(at 90 96 0)
+		(layer "F.Mask")
+		(effects
+			(font
+				(size 0.5 0.5)
+				(thickness 0.1)
+				(bold yes)
+			)
+		)
 	)
 	(gr_text "PAM8408"

Commit message: -
Parts:
- moved ? 9.06 mm to (86.0, 104.2), turned to 90 degrees
- moved ? 7.07 mm to (90.6, 99.8), turned to 90 degrees
Routing:
- net INL: track 14.9 -> 13.9 mm
Changed lines of the file:
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@@
 		(fp_line
 			(start -3 1)
-			(end -3 3)
+			(end -3 4)
 			(stroke
 				(width 0.1)
@@
 		)
 		(fp_line
-			(start 3 3)
+			(start 3 4)
 			(end 3 1)
 			(stroke
@@
 		)
 		(fp_line
-			(start -3 6)
+			(start -3 7)
 			(end -3 10)
 			(stroke
@@
 		(fp_line
 			(start 3 10)
-			(end 3 6)
+			(end 3 7)
 			(stroke
 				(width 0.1)
@@
 		)
 		(pad "T" thru_hole roundrect
-			(at -2.75 4.5 90)
+			(at -2.75 5.5 90)
 			(size 1.8 2.1)
 			(drill oval 1 1.3)
@@
 		)
 		(pad "T" thru_hole roundrect
-			(at 2.75 4.5 90)
+			(at 2.75 5.5 90)
 			(size 1.8 2.1)
 			(drill oval 1 1.3)
@@
 	(footprint "Library:mcbeeringi_icon_5mm"
 		(layer "B.Cu")
-		(at 95.6 94.8 45)
+		(at 90.6 99.8 90)
 		(property "Reference" ""
-			(at 0 0 45)
+			(at 0 0 90)
 			(layer "B.SilkS")
 			(effects
@@
 		)
 		(property "Value" "mcbeeringi_icon"
-			(at 0.75 0 45)
+			(at 0.75 0 90)
 			(layer "B.SilkS")
 			(hide yes)
@@
 		)
 		(property "Datasheet" ""
-			(at 0 0 45)
+			(at 0 0 90)
 			(layer "B.Fab")
 			(hide yes)
@@
 		)
 		(property "Description" ""
-			(at 0 0 45)
+			(at 0 0 90)
 			(layer "B.Fab")
 			(hide yes)
@@
 	(footprint "Library:PCB.MCBEERINGI.DEV_small"
 		(layer "B.Cu")
-		(at 89.4 95.8 45)
+		(at 86 104.2 90)
 		(property "Reference" ""
-			(at 0 0 45)
+			(at 0 0 90)
 			(layer "B.SilkS")
 			(effects
@@
 		)
 		(property "Value" ""
-			(at 0 0 45)
+			(at 0 0 90)
 			(layer "B.Fab")
 			(effects
@@
 		)
 		(property "Datasheet" ""
-			(at 0 0 45)
+			(at 0 0 90)
 			(layer "B.Fab")
 			(hide yes)
@@
 		)
 		(property "Description" ""
-			(at 0 0 45)
+			(at 0 0 90)
 			(layer "B.Fab")
 			(hide yes)
@@
 		(fp_poly
 			(pts
-				(xy -1.374121 1.749526) (xy -1.374121 1.374121) (xy -1.749526 1.374121) (xy -2.12493 1.374121) (xy -2.12493 1.749526)
-				(xy -2.12493 2.12493) (xy -1.749526 2.12493) (xy -1.374121 2.12493)
+				(xy 2.620748 0.375404) (xy 2.620748 0.127496) (xy 2.500335 0.127496) (xy 2.379922 0.127496) (xy 2.379922 0.375404)
+				(xy 2.379922 0.623313) (xy 2.500335 0.623313) (xy 2.620748 0.623313)
 			)
 			(stroke
@@
 		(fp_poly
 			(pts
-				(xy 2.620748 0.375404) (xy 2.620748 0.127496) (xy 2.500335 0.127496) (xy 2.379922 0.127496) (xy 2.379922 0.375404)
-				(xy 2.379922 0.623313) (xy 2.500335 0.623313) (xy 2.620748 0.623313)
+				(xy 2.12493 1.749526) (xy 2.12493 1.374121) (xy 1.749526 1.374121) (xy 1.374122 1.374121) (xy 1.374122 1.749526)
+				(xy 1.374122 2.124929) (xy 1.749526 2.12493) (xy 2.12493 2.12493)
 			)
 			(stroke
@@
 		(fp_poly
 			(pts
-				(xy 2.12493 1.749526) (xy 2.12493 1.374121) (xy 1.749526 1.374121) (xy 1.374122 1.374121) (xy 1.374122 1.749526)
-				(xy 1.374122 2.124929) (xy 1.749526 2.12493) (xy 2.12493 2.12493)
+				(xy -1.374121 1.749526) (xy -1.374121 1.374121) (xy -1.749526 1.374121) (xy -2.12493 1.374121) (xy -2.12493 1.749526)
+				(xy -2.12493 2.12493) (xy -1.749526 2.12493) (xy -1.374121 2.12493)
 			)
 			(stroke
@@
 		(fp_poly
 			(pts
-				(xy -0.878304 1.756609) (xy -0.878304 0.878304) (xy -1.749526 0.878304) (xy -2.620747 0.878304)
-				(xy -2.620747 1.133296) (xy -2.38022 1.133296) (xy -1.756758 1.133296) (xy -1.133296 1.133296) (xy -1.133296 1.756758)
-				(xy -1.133296 2.38022) (xy -1.753067 2.376529) (xy -2.372839 2.372839) (xy -2.376529 1.753067) (xy -2.38022 1.133296)
-				(xy -2.620747 1.133296) (xy -2.620747 1.756609) (xy -2.620747 2.634913) (xy -1.749526 2.634913)
-				(xy -0.878304 2.634913)
+				(xy 2.620748 1.756609) (xy 2.620748 0.878304) (xy 1.749526 0.878304) (xy 0.878305 0.878304) (xy 0.878305 1.75661)
+				(xy 0.878305 1.756758) (xy 1.133296 1.756758) (xy 1.133296 1.133296) (xy 1.756758 1.133296) (xy 2.38022 1.133296)
+				(xy 2.376529 1.753067) (xy 2.372839 2.372839) (xy 1.753068 2.376529) (xy 1.133296 2.38022) (xy 1.133296 1.756758)
+				(xy 0.878305 1.756758) (xy 0.878305 2.634913) (xy 1.749526 2.634913) (xy 2.620748 2.634913)
 			)
 			(stroke
@@
 		(fp_poly
 			(pts
-				(xy 2.620748 1.756609) (xy 2.620748 0.878304) (xy 1.749526 0.878304) (xy 0.878305 0.878304) (xy 0.878305 1.75661)
-				(xy 0.878305 1.756758) (xy 1.133296 1.756758) (xy 1.133296 1.133296) (xy 1.756758 1.133296) (xy 2.38022 1.133296)
-				(xy 2.376529 1.753067) (xy 2.372839 2.372839) (xy 1.753068 2.376529) (xy 1.133296 2.38022) (xy 1.133296 1.756758)
-				(xy 0.878305 1.756758) (xy 0.878305 2.634913) (xy 1.749526 2.634913) (xy 2.620748 2.634913)
+				(xy -0.878304 1.756609) (xy -0.878304 0.878304) (xy -1.749526 0.878304) (xy -2.620747 0.878304)
+				(xy -2.620747 1.133296) (xy -2.38022 1.133296) (xy -1.756758 1.133296) (xy -1.133296 1.133296) (xy -1.133296 1.756758)
+				(xy -1.133296 2.38022) (xy -1.753067 2.376529) (xy -2.372839 2.372839) (xy -2.376529 1.753067) (xy -2.38022 1.133296)
+				(xy -2.620747 1.133296) (xy -2.620747 1.756609) (xy -2.620747 2.634913) (xy -1.749526 2.634913)
+				(xy -0.878304 2.634913)
 			)
 			(stroke
@@
 	)
 	(gr_text "PAM8408\n2x3W AMP"
-		(at 94.6 99.8 225)
+		(at 84.6 95.8 270)
 		(layer "B.Mask")
 		(effects
@@
 	)
 	(gr_text "IN"
-		(at 82.6 95.8 270)
+		(at 90 95.8 270)
 		(layer "B.SilkS")
 		(effects
@@
 				(bold yes)
 			)
-			(justify bottom mirror)
+			(justify mirror)
 		)
 	)
@@
 	)
 	(gr_text "PWR"
-		(at 82.6 104.2 270)
+		(at 91.6 103.8 270)
 		(layer "B.SilkS")
 		(effects
@@
 	)
 	(segment
-		(start 86.4 93.0625)
-		(end 86.3875 93.05)
+		(start 94.2 98.6)
+		(end 95.025 98.6)
 		(width 0.2)
 		(layer "F.Cu")
@@
 	)
 	(segment
-		(start 86.3875 98.55)
-		(end 86.4 98.5375)
+		(start 87.3875 98.5875)
+		(end 88 99.2)
 		(width 0.2)
 		(layer "F.Cu")
@@
 	)
 	(segment
-		(start 95.025 98.6)
-		(end 94.2 98.6)
+		(start 88 99.2)
+		(end 93.6 99.2)
 		(width 0.2)
 		(layer "F.Cu")
@@
 	)
 	(segment
-		(start 87 99.2)
-		(end 86.3875 98.5875)
+		(start 87.3875 98.55)
+		(end 87.3875 98.5875)
 		(width 0.2)
 		(layer "F.Cu")
@@
 	)
 	(segment
-		(start 86.4 98.5375)
-		(end 86.4 93.0625)
+		(start 87.4 93.0625)
+		(end 87.4 98.5375)
 		(width 0.2)
 		(layer "F.Cu")
@@
 	(segment
 		(start 93.6 99.2)
-		(end 87 99.2)
+		(end 94.2 98.6)
 		(width 0.2)
 		(layer "F.Cu")
@@
 	)
 	(segment
-		(start 95.2 98.425)
-		(end 95.025 98.6)
+		(start 87.3875 93.05)
+		(end 87.4 93.0625)
 		(width 0.2)
 		(layer "F.Cu")
@@
 	)
 	(segment
-		(start 94.2 98.6)
-		(end 93.6 99.2)
+		(start 87.4 98.5375)
+		(end 87.3875 98.55)
 		(width 0.2)
 		(layer "F.Cu")
@@
 	)
 	(segment
-		(start 86.3875 98.5875)
-		(end 86.3875 98.55)
+		(start 95.025 98.6)
+		(end 95.2 98.425)
 		(width 0.2)
 		(layer "F.Cu")
