File: proj/card/30led/30led.kicad_pcb (KiCad board)
At the start: 2 copper layers, 100 x 80 mm, 45 parts, among them J1 UPDI, SW1 SW_SPDT, U1 ATtiny404-SS

Commit message: -
Parts:
- added ?: LOGO, Library:mcbeeringi_icon_20mm, B.Cu at (108.0, 100.0)
- added ?: , Library:PCB.MCBEERINGI.DEV, B.Cu at (90.0, 100.0)
- moved SW1 3.01 mm to (86.6, 128.0)
- moved C1 1.00 mm to (91.6, 123.0)
- moved C2 1.00 mm to (93.6, 123.0)
Routing:
- net ROW1: track 302.7 -> 299.4 mm, vias 9 -> 11
Other:
- board text added: "card 30led"

Commit message: -
Other:
- board text added: "100R *6"
- board text added: "100u"
- board text added: "4u7"
- board text added: "ATtinyX04"
- board text added: "BC-2001"
- board text added: "CR2032 *2"
- board text added: "GND"
- board text added: "I"
- board text added: "O"
- board text added: "UPDI"
Changed lines of the file:
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@@
+		)
+	)
+	(gr_text "CR2032 *2"
+		(at 74 103 0)
+		(layer "B.Mask")
+		(effects
+			(font
+				(size 2 2)
+				(thickness 0.4)
+				(bold yes)
+			)
+			(justify mirror)
+		)
+	)
+	(gr_text "ATtinyX04"
+		(at 105.6 122.6 0)
+		(layer "B.Mask")
+		(effects
+			(font
+				(size 0.5 0.5)
+				(thickness 0.1)
+				(bold yes)
+			)
+			(justify mirror)
+		)
+	)
+	(gr_text "100u"
+		(at 91.6 125.7 0)
+		(layer "B.Mask")
+		(effects
+			(font
+				(size 0.5 0.5)
+				(thickness 0.1)
+				(bold yes)
+			)
+			(justify mirror)
+		)
+	)
+	(gr_text "BC-2001"
+		(at 87 111 -0)
+		(layer "B.Mask")
+		(effects
+			(font
+				(size 0.5 0.5)
+				(thickness 0.1)
+				(bold yes)
+			)
+			(justify mirror)
+		)
+	)
+	(gr_text "BC-2001"
+		(at 113 111 -0)
+		(layer "B.Mask")
+		(effects
+			(font
+				(size 0.5 0.5)
+				(thickness 0.1)
+				(bold yes)
+			)
+			(justify mirror)
+		)
+	)
+	(gr_text "GND"
+		(at 96 134 0)
+		(layer "B.Mask")
+		(effects
+			(font
+				(size 0.5 0.5)
+				(thickness 0.1)
+				(bold yes)
+			)
+			(justify mirror)
+		)
+	)
+	(gr_text "4u7"
+		(at 93.6 124.9 0)
+		(layer "B.Mask")
+		(effects
+			(font
+				(size 0.5 0.5)
+				(thickness 0.1)
+				(bold yes)
+			)
+			(justify mirror)
+		)
+	)
+	(gr_text "UPDI"
+		(at 104 134 0)
+		(layer "B.Mask")
+		(effects
+			(font
+				(size 0.5 0.5)
+				(thickness 0.1)
+				(bold yes)
+			)
+			(justify mirror)
+		)
+	)
+	(gr_text "100R *6"
+		(at 107.5 126 0)
+		(layer "B.Mask")
+		(effects
+			(font
+				(size 0.5 0.5)
+				(thickness 0.1)
+				(bold yes)
+			)
+			(justify mirror)
 		)
 	)
@@
 			)
 			(justify mirror)
+		)
+	)
+	(gr_text "O"
+		(at 92 128 0)
+		(layer "B.SilkS")
+		(effects
+			(font
+				(size 2 2)
+				(thickness 0.25)
+			)
+			(justify mirror)
+		)
+	)
+	(gr_text "I"
+		(at 81 128 0)
+		(layer "B.SilkS")
+		(effects
+			(font
+				(size 2 2)
+				(thickness 0.25)
+			)
+			(justify mirror)

Commit message: -
Parts:
- added C3: 0u1, Capacitor_SMD:C_0603_1608Metric, F.Cu at (153.1, 145.1)
- added J2: USB_C_Receptacle_USB2.0_16P, Connector_USB:USB_C_Receptacle_GCT_USB4105-xx-A_16P_TopMnt_Horizontal, B.Cu at (175.1, 87.3)
- added R7: 4k7, Resistor_SMD:R_0603_1608Metric, F.Cu at (153.1, 147.6)
- added R8: 4k7, Resistor_SMD:R_0603_1608Metric, F.Cu at (153.1, 150.1)
- added SW2: SW_Push, Library:alps-skrp, F.Cu at (188.7, 110.5)
- added U2: CH340K, Package_SO:SSOP-10-1EP_3.9x4.9mm_P1mm_EP2.1x3.3mm, F.Cu at (166.4, 154.5)
- C1: value 100u -> 10u; footprint Capacitor_SMD:C_1206_3216Metric -> Capacitor_SMD:C_0603_1608Metric; moved to F.Cu
- C2: value 4u7 -> 0u1; moved to F.Cu
- J1: moved to F.Cu
- R1, R2, R3, R4, R5, R6: value 100R -> Rled
- SW1: value SW_SPDT -> SW_Push; footprint Library:sw_tht -> Library:alps-skrp; moved to F.Cu
- moved SW1 104.4 mm to (188.7, 106.3), turned to 0 degrees
- moved ? 100.0 mm to (207.5, 82.5)
- moved G*** 100.0 mm to (180.0, 95.0)
- moved C1 96.2 mm to (187.4, 113.9), turned to 0 degrees
- moved U1 79.2 mm to (176.6, 105.9)
- moved J1 68.7 mm to (167.2, 127.7), turned to 0 degrees
- moved C2 62.6 mm to (153.1, 142.5), turned to 0 degrees
- moved D1 41.8 mm to (146.8, 130.6), turned to 90 degrees
- moved D26 41.8 mm to (53.2, 130.6), turned to 90 degrees
- moved D30 39.8 mm to (94.8, 130.6), turned to 90 degrees
- moved D5 39.8 mm to (105.2, 130.6), turned to 90 degrees
- moved ? 32.2 mm to (81.2, 82.2)
- moved ? 29.5 mm to (67.4, 81.0)
- moved D2 21.4 mm to (136.4, 130.6), turned to 90 degrees
- moved D27 21.4 mm to (63.6, 130.6), turned to 90 degrees
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Connections:
- C1 pad 1: VCC -> +BATT
- C2 pad 1: VCC -> Net-(U2-V3)
- SW1 pad 1: unconnected-(SW1-A-Pad1) -> GND
- SW1 pad 2: VCC -> ROW5
- U1 pad 1: VCC -> +BATT
Routing:
- net ROW1: track 299.4 -> 0.00 mm, vias 11 -> 3
- net ROW2: track 274.9 -> 0.00 mm, vias 9 -> 3
- net ROW3: track 262.8 -> 0.00 mm, vias 9 -> 3
- net ROW4: track 245.5 -> 0.00 mm, vias 9 -> 3
- net ROW5: track 228.4 -> 0.00 mm, vias 9 -> 3
- net /_COL4: track 153.2 -> 0.00 mm, vias 1 -> 0
- net /_COL3: track 153.2 -> 41.6 mm, vias 1 -> 0
- net /_COL5: track 100.5 -> 0.00 mm, vias 1 -> 0
- net /_COL2: track 100.5 -> 43.5 mm, vias 1 -> 0
- net /_COL6: track 49.6 -> 0.00 mm, vias 1 -> 0
- net UPDI: track 9.77 -> 0.00 mm
- net /_COL1: track 49.6 -> 41.6 mm, vias 1 -> 0
- net COL3: track 7.59 -> 0.00 mm
- net COL6: track 7.21 -> 0.00 mm
- net COL5: track 7.12 -> 0.00 mm
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- removed copper zone on B.Cu, net VCC
Other:
- board size 100 x 80 mm -> 100 x 75 mm
- board text added: "10u"
- board text added: "Rled *6"
- board text removed: "100R *6"
- board text removed: "100u"
- board text removed: "4u7"
- board text removed: "I"
- board text removed: "O"

Commit message: -
Parts:
- moved J2 85.0 mm to (100.0, 127.2)
- moved R3 46.2 mm to (95.2, 73.8), turned to 90 degrees
- moved R4 46.2 mm to (104.8, 73.8), turned to 90 degrees
- moved R2 45.7 mm to (96.8, 73.8), turned to 90 degrees
- moved R5 45.7 mm to (103.2, 73.8), turned to 90 degrees
- moved R1 45.3 mm to (98.4, 73.8), turned to 90 degrees
- moved R6 45.3 mm to (101.6, 73.8), turned to 90 degrees
- turned D1 to -90 degrees
- turned D10 to -90 degrees
- turned D11 to -90 degrees
- turned D12 to -90 degrees
- turned D13 to -90 degrees
- turned D14 to -90 degrees
- turned D15 to -90 degrees
- turned D16 to -90 degrees
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Routing:
- net ROW5: track 0.00 -> 142.8 mm
- net ROW4: track 0.00 -> 141.9 mm
- net ROW3: track 0.00 -> 132.5 mm
- net ROW2: track 0.00 -> 123.1 mm
- net ROW1: track 0.00 -> 114.4 mm
- net /_COL1: track 41.6 -> 43.0 mm
Other:
- outline, holes or cut-outs redrawn
- board text added: "${REFERENCE}"

Commit message: -
Parts:
- C1, C2, C3, J1, R7, R8, SW1, SW2, U2: moved to B.Cu
- moved C1 103.1 mm to (93.0, 72.4), turned to 180 degrees
- moved SW1 96.1 mm to (96.0, 81.0), turned to 180 degrees
- moved SW2 89.7 mm to (104.0, 81.0), turned to 180 degrees
- moved U1 82.6 mm to (100.0, 75.0)
- moved J1 78.1 mm to (89.8, 117.6), turned to 180 degrees
- moved U2 75.7 mm to (100.0, 118.0), turned to 180 degrees
- moved R8 64.4 mm to (93.8, 124.8), turned to 90 degrees
- moved R7 52.1 mm to (106.2, 124.8), turned to 90 degrees
- moved C2 50.6 mm to (109.4, 117.0), turned to 180 degrees
- moved C3 49.4 mm to (109.6, 121.6), turned to 180 degrees
- moved R3 11.8 mm to (107.0, 74.0), turned to 0 degrees
- moved R4 11.8 mm to (93.0, 74.0), turned to 180 degrees
- moved R2 10.4 mm to (107.0, 75.6), turned to 0 degrees
- moved R5 10.4 mm to (93.0, 75.6), turned to 180 degrees
- moved R1 9.25 mm to (107.0, 77.2), turned to 0 degrees
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Connections:
- SW1 pad 2: ROW5 -> ROW1
- SW2 pad 2: ROW4 -> ROW3
- U1 pad 11: ROW2 -> ROW3
- U1 pad 13: COL4 -> COL6
- U1 pad 2: COL5 -> COL4
- U1 pad 3: COL6 -> COL5
- U1 pad 4: ROW3 -> ROW2
- U1 pad 8: COL2 -> COL1
- U1 pad 9: COL1 -> COL2
Routing:
- net ROW5: track 142.8 -> 302.4 mm, vias 3 -> 9
- net /_COL6: track 0.00 -> 144.0 mm, vias 0 -> 1
- net ROW3: track 132.5 -> 276.4 mm, vias 3 -> 9
- net ROW4: track 141.9 -> 279.7 mm, vias 3 -> 9
- net ROW1: track 114.4 -> 241.4 mm, vias 3 -> 7
- net ROW2: track 123.1 -> 243.4 mm, vias 3 -> 9
- net /_COL1: track 43.0 -> 143.9 mm, vias 0 -> 1
- net /_COL5: track 0.00 -> 94.3 mm, vias 0 -> 1
- net /_COL2: track 43.5 -> 94.3 mm, vias 0 -> 1
- net /_COL4: track 0.00 -> 47.0 mm, vias 0 -> 1
- net COL5: track 0.00 -> 7.02 mm
- net Net-(J2-CC1): track 0.00 -> 6.25 mm
- net Net-(J2-CC2): track 0.00 -> 6.04 mm
- net /_COL3: track 41.6 -> 47.0 mm, vias 0 -> 1
- net COL6: track 0.00 -> 4.84 mm
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Other:
- outline, holes or cut-outs redrawn
- board text added: "CR2032 x2"
- board text removed: "${REFERENCE}"
- board text removed: "CR2032 *2"

Commit message: -
Parts:
- removed the ? at (207.5, 82.5)
- removed G***: LOGO, LOGO
- removed the J1 at (89.8, 117.6)
- added TP1: PRG_GND, TestPoint:TestPoint_Pad_1.5x1.5mm, B.Cu at (91.7, 79.0)
- added TP2: PRG_UPDI, TestPoint:TestPoint_Pad_D1.5mm, B.Cu at (94.3, 79.0)
- moved C1 14.9 mm to (107.0, 77.6), turned to 0 degrees
- moved C3 14.2 mm to (95.4, 120.8), turned to 90 degrees
- moved C2 14.0 mm to (95.4, 117.0), turned to -90 degrees
- moved R7 5.28 mm to (102.0, 121.6), turned to 0 degrees
- moved R8 5.12 mm to (97.8, 121.6), turned to 180 degrees
- moved SW1 2.24 mm to (98.0, 82.0), turned to 90 degrees
- moved SW2 2.24 mm to (102.0, 82.0), turned to -90 degrees
- moved R1 2.00 mm to (107.0, 75.2)
- moved R2 2.00 mm to (107.0, 73.6)
- moved R3 2.00 mm to (107.0, 72.0)
- moved R4 2.00 mm to (93.0, 72.0)
- moved R5 2.00 mm to (93.0, 73.6)
- moved R6 2.00 mm to (93.0, 75.2)
- moved ? 1.00 mm to (78.0, 80.0)
- moved ? 1.00 mm to (62.0, 80.0)
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- renumbered J2 to J1
Connections:
- SW1 pad 2: ROW1 -> ROW4
- SW2 pad 2: ROW3 -> ROW2
- U1 pad 13: COL6 -> COL3
- U1 pad 2: COL4 -> COL1
- U1 pad 3: COL5 -> COL2
- U1 pad 7: COL3 -> COL6
- U1 pad 8: COL1 -> COL4
- U1 pad 9: COL2 -> COL5
Routing:
- net UPDI: track 3.05 -> 121.2 mm
- net ROW3: track 276.4 -> 261.5 mm
- net ROW1: track 241.4 -> 229.0 mm
- net ROW2: track 243.4 -> 255.5 mm
- net ROW4: track 279.7 -> 291.5 mm
- net D-: track 0.00 -> 10.7 mm
- net D+: track 0.00 -> 9.96 mm
- net ROW5: track 302.4 -> 307.3 mm
- net Net-(J1-CC1): track 6.25 -> 1.95 mm
- net Net-(J1-CC2): track 6.04 -> 2.08 mm
- net COL3: track 3.27 -> 6.19 mm
- net COL5: track 7.02 -> 4.61 mm
- net COL2: track 4.65 -> 6.96 mm
- net /_COL4: track 47.0 -> 44.8 mm
- net /_COL3: track 47.0 -> 44.8 mm
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- added copper zone on B.Cu, net VBUS
Other:
- board text added: "0u1"
- board text added: "4k7 *2"
- board text added: "ALPS SKRP *2"
- board text added: "CH340K"
- board text added: "NFC tag sticker"
- board text added: "Rled *3"
- board text added: "USB4105"
- board text removed: "6ca.me"
- board text removed: "McbeEringi"
- board text removed: "Rled *6"

Commit message: -
Routing:
- net VBUS: track 0.00 -> 2.75 mm
- net GND: track 0.00 -> 2.72 mm
Changed lines of the file:
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@@
 	)
 	(segment
+		(start 103.775 124.095)
+		(end 103.2 123.52)
+		(width 0.5)
+		(layer "B.Cu")
+		(net 1)
+	)
+	(segment
+		(start 104.32 124.095)
+		(end 103.775 124.095)
+		(width 0.5)
+		(layer "B.Cu")
+		(net 1)
+	)
+	(segment
+		(start 95.68 124.095)
+		(end 96.225 124.095)
+		(width 0.5)
+		(layer "B.Cu")
+		(net 1)
+	)
+	(segment
+		(start 96.225 124.095)
+		(end 96.8 123.52)
+		(width 0.5)
+		(layer "B.Cu")
+		(net 1)
+	)
+	(segment
 		(start 102.54 76.06)
 		(end 102.54 77.475)
@@
 	)
 	(segment
-		(start 98.73 74.67)
-		(end 98.095 75.305)
-		(width 0.2)
-		(layer "B.Cu")
-		(net 12)
-	)
-	(segment
 		(start 65.8 126.2)
 		(end 59.8 120.2)
@@
 	)
 	(segment
-		(start 97.502 80.8)
-		(end 98.095 80.207)
+		(start 83.8 118.6)
+		(end 76.2 126.2)
 		(width 0.2)
 		(layer "B.Cu")
@@
 	)
 	(segment
-		(start 83.8 118.6)
-		(end 76.2 126.2)
+		(start 97.502 80.8)
+		(end 98.095 80.207)
 		(width 0.2)
 		(layer "B.Cu")
@@
 	)
 	(segment
-		(start 98.095 80.207)
-		(end 98.095 78.4)
+		(start 97.3625 118)
+		(end 96.4 118)
 		(width 0.2)
 		(layer "B.Cu")
@@
 	)
 	(segment
-		(start 97.3625 118)
-		(end 96.4 118)
+		(start 81.8 93.8)
+		(end 94.8 80.8)
 		(width 0.2)
 		(layer "B.Cu")
@@
 	)
 	(segment
-		(start 98.095 78.4)
-		(end 98.095 78.456968)
+		(start 94.8 80.8)
+		(end 97.502 80.8)
 		(width 0.2)
 		(layer "B.Cu")
@@
 	)
 	(segment
-		(start 81.8 93.8)
-		(end 94.8 80.8)
+		(start 98.095 80.207)
+		(end 98.095 75.305)
 		(width 0.2)
 		(layer "B.Cu")
@@
 	)
 	(segment
-		(start 98.095 75.305)
-		(end 98.095 78.4)
+		(start 96.4 118)
+		(end 95.8 118.6)
 		(width 0.2)
 		(layer "B.Cu")
@@
 	)
 	(segment
-		(start 94.8 80.8)
-		(end 97.502 80.8)
+		(start 98.73 74.67)
+		(end 98.73 72.525)
 		(width 0.2)
 		(layer "B.Cu")
@@
 	)
 	(segment
-		(start 96.4 118)
-		(end 95.8 118.6)
+		(start 98.095 75.305)
+		(end 98.73 74.67)
 		(width 0.2)
 		(layer "B.Cu")
@@
 	)
 	(segment
-		(start 98.73 72.525)
-		(end 98.73 74.67)
-		(width 0.2)
-		(layer "B.Cu")
-		(net 12)
-	)
-	(segment
 		(start 94.285 79.045)
 		(end 94.285 80.285)
@@
 	)
 	(segment
+		(start 95.8 119)
+		(end 97.3625 119)
+		(width 0.2)
+		(layer "B.Cu")
+		(net 22)
+	)
+	(segment
+		(start 95.4 119.4)
+		(end 95.8 119)
+		(width 0.2)
+		(layer "B.Cu")
+		(net 22)
+	)
+	(segment
+		(start 95.4 120.025)
+		(end 95.4 119.4)
+		(width 0.2)
+		(layer "B.Cu")
+		(net 22)
+	)
+	(segment

Commit message: -
Routing:
- net GND: vias 16 -> 60
