File: proj/dcdc/buckboost/tps631000/tps631000.kicad_pcb (KiCad board)
At the start: 2 copper layers, 10 x 8 mm, 8 parts, among them J1 POW, U1 TPS631000

Commit message: -
Parts:
- L1: footprint Inductor_SMD:L_1210_3225Metric -> Inductor_SMD:L_1008_2520Metric
- moved R1 0.20 mm to (106.0, 97.8)
Changed lines of the file:
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@@
 		)
 	)
-	(footprint "Inductor_SMD:L_1210_3225Metric"
+	(footprint "Inductor_SMD:L_1008_2520Metric"
 		(layer "F.Cu")
 		(at 106 100.8 -90)
-		(descr "Inductor SMD 1210 (3225 Metric), square (rectangular) end terminal, IPC-7351 nominal, (Body size source: http://www.tortai-tech.com/upload/download/2011102023233369053.pdf), generated with kicad-footprint-generator")
+		(descr "Inductor SMD 1008 (2520 Metric), square (rectangular) end terminal, IPC-7351 nominal, (Body size source: https://ecsxtal.com/store/pdf/ECS-MPI2520-SMD-POWER-INDUCTOR.pdf), generated with kicad-footprint-generator")
 		(tags "inductor")
 		(property "Reference" "L1"
-			(at 0 -2.28 90)
+			(at 0 -2.05 270)
 			(layer "F.SilkS")
 			(hide yes)
@@
 		)
 		(property "Value" "1u"
-			(at 0 2.28 90)
+			(at 0 2.05 270)
 			(layer "F.Fab")
 			(hide yes)
@@
 		)
 		(property "Datasheet" "~"
-			(at 0 0 90)
+			(at 0 0 270)
 			(layer "F.Fab")
 			(hide yes)
@@
 		)
 		(property "Description" "Inductor, small symbol"
-			(at 0 0 90)
+			(at 0 0 270)
 			(layer "F.Fab")
 			(hide yes)
@@
 		(attr smd)
 		(fp_line
-			(start -0.602064 1.36)
-			(end 0.602064 1.36)
+			(start -0.261252 1.11)
+			(end 0.261252 1.11)
 			(stroke
 				(width 0.12)
@@
 		)
 		(fp_line
-			(start -0.602064 -1.36)
-			(end 0.602064 -1.36)
+			(start -0.261252 -1.11)
+			(end 0.261252 -1.11)
 			(stroke
 				(width 0.12)
@@
 		)
 		(fp_rect
-			(start -2.28 -1.58)
-			(end 2.28 1.58)
+			(start -1.95 -1.35)
+			(end 1.95 1.35)
 			(stroke
 				(width 0.05)
@@
 		)
 		(fp_rect
-			(start -1.6 -1.25)
-			(end 1.6 1.25)
+			(start -1.25 -1)
+			(end 1.25 1)
 			(stroke
 				(width 0.1)
@@
 		)
 		(fp_text user "${REFERENCE}"
-			(at 0 0 90)
-			(layer "F.Fab")
-			(effects
-				(font
-					(size 0.8 0.8)
-					(thickness 0.12)
+			(at 0 0 270)
+			(layer "F.Fab")
+			(effects
+				(font
+					(size 0.62 0.62)
+					(thickness 0.09)
 				)
 			)
 		)
 		(pad "1" smd roundrect
-			(at -1.4 0 270)
-			(size 1.25 2.65)
+			(at -1.075 0 270)
+			(size 1.25 2.2)
 			(layers "F.Cu" "F.Mask" "F.Paste")
 			(roundrect_rratio 0.2)
@@
 		)
 		(pad "2" smd roundrect
-			(at 1.4 0 270)
-			(size 1.25 2.65)
+			(at 1.075 0 270)
+			(size 1.25 2.2)
 			(layers "F.Cu" "F.Mask" "F.Paste")
 			(roundrect_rratio 0.2)
@@
 		)
 		(embedded_fonts no)
-		(model "${KICAD9_3DMODEL_DIR}/Inductor_SMD.3dshapes/L_1210_3225Metric.step"
+		(model "${KICAD9_3DMODEL_DIR}/Inductor_SMD.3dshapes/L_1008_2520Metric.step"
 			(offset
 				(xyz 0 0 0)
 			)
 			(scale
-				(xyz 1 1 0.5)
+				(xyz 1 1 1)
 			)
 			(rotate
-				(xyz -0 -0 -0)
+				(xyz 0 0 0)
 			)
 		)
@@
 	(footprint "Resistor_SMD:R_0603_1608Metric"
 		(layer "F.Cu")
-		(at 106 97.6)
+		(at 106 97.8)
 		(descr "Resistor SMD 0603 (1608 Metric), square (rectangular) end terminal, IPC-7351 nominal, (Body size source: IPC-SM-782 page 72, https://www.pcb-3d.com/wordpress/wp-content/uploads/ipc-sm-782a_amendment_1_and_2.pdf), generated with kicad-footprint-generator")
 		(tags "resistor")
@@
 	(segment
 		(start 103.575 97.8)
-		(end 104.975 97.8)
-		(width 0.2)
-		(layer "F.Cu")
-		(net 2)
-	)
-	(segment
-		(start 104.975 97.8)
-		(end 105.175 97.6)
+		(end 105.175 97.8)
 		(width 0.2)
 		(layer "F.Cu")
@@
 	)
 	(segment
-		(start 106.825 97.6)
-		(end 106.8 97.6)
+		(start 106.8 97.8)
+		(end 106.825 97.8)
 		(width 0.2)
 		(layer "F.Cu")
@@
 	)
 	(segment
-		(start 106.8 97.6)
-		(end 106 98.4)
+		(start 106 98.6)
+		(end 106.8 97.8)
 		(width 0.2)
 		(layer "F.Cu")
@@
 	)
 	(segment
-		(start 106 98.4)
-		(end 104.4 98.4)
+		(start 104.6 98.6)
+		(end 106 98.6)
+		(width 0.2)
+		(layer "F.Cu")
+		(net 4)
+	)
+	(segment
+		(start 104.4 98.4)
+		(end 104.6 98.6)
 		(width 0.2)
 		(layer "F.Cu")
@@
 		(polygon
 			(pts
-				(xy 107.4 98.8) (xy 107.4 99.9) (xy 103.4 99.9) (xy 103.4 99.4) (xy 104.2 99.4) (xy 104.2 98.8)
+				(xy 107.2 99) (xy 107.2 99.9) (xy 103.4 99.9) (xy 103.4 99.4) (xy 104.2 99.4) (xy 104.2 99)
 			)
 		)
@@
 		(polygon
 			(pts
-				(xy 107.4 102.8) (xy 107.4 100.1) (xy 103.4 100.1) (xy 103.4 100.6) (xy 104.2 100.6) (xy 104.2 102.8)
-			)
-		)
+				(xy 107.2 102.6) (xy 107.2 100.1) (xy 103.4 100.1) (xy 103.4 100.6) (xy 104.2 100.6) (xy 104.2 102.6)
+			)
+		)
