File: proj/dcdc/boost/tps61322-batt/tps61322-batt.kicad_sch (KiCad schematic)
At the start: 7 parts, among them J1 Conn_02x02_Odd_Even, J2 Conn_01x02_Pin, P1 USB_C_Plug, U1 TPS613222ADBV

Commit message: -
Parts:
- L1: footprint Inductor_SMD:L_1210_3225Metric -> Inductor_SMD:L_1008_2520Metric
Changed lines of the file:
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@@
 			)
 		)
-		(property "Footprint" "Inductor_SMD:L_1210_3225Metric"
+		(property "Footprint" "Inductor_SMD:L_1008_2520Metric"
 			(at 83.82 53.34 0)
 			(effects

Commit message: -
Parts:
- added JP1: BC, Resistor_SMD:R_0603_1608Metric, symbol Jumper:Jumper_2_Open
- added R1: 56k, Resistor_SMD:R_0603_1608Metric, symbol Device:R_Small
- P1: footprint Library:USB_C_PLUG_00402-UCAM002-X -> Library:USB_C_PLUG_00402-UCAM001-X
Connections:
- net at P1.A5 (CC): now also R1.2
- net at P1.A6 (D+): now also JP1.1 (A)
- net at P1.A7 (D-): now also JP1.2 (B)
- net Vout renamed +5V
- net +5V: now also R1.1
- no-connect marks 16 -> 13
