File: proj/avr/musicbox/musicbox.kicad_sch (KiCad schematic)
At the start: 55 parts, among them J1 USB, J2 UPDI, J3 NiMh*2, J4 OUT1, J5 OUT1, Q1 AO3401A, SW1 SW, SW2 SW, U1 CH340E, U2 BQ25172, U3 ATtiny402-SS, U4 ATtiny1604-SS, U5 TPS613222ADBV, U6 CH213K, U7 CH213K, U8 alps-rk10j12e, U9 PAM8406D

Commit message: -
Connections:
- net GND: now also C2.2; no longer C2.1
- net at U1.10 (V3): now also C2.1; no longer C2.2
Changed lines of the file:
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@@
 	(wire
 		(pts
+			(xy 31.75 116.84) (xy 31.75 119.38)
+		)
+		(stroke
+			(width 0)
+			(type default)
+		)
+	)
+	(wire
+		(pts
 			(xy 135.89 148.59) (xy 149.86 148.59)
 		)
@@
 	(wire
 		(pts
+			(xy 29.21 115.57) (xy 29.21 119.38)
+		)
+		(stroke
+			(width 0)
+			(type default)
+		)
+	)
+	(wire
+		(pts
 			(xy 149.86 142.24) (xy 149.86 140.97)
 		)
@@
 	(symbol
 		(lib_id "power:VBUS")
-		(at 29.21 119.38 0)
+		(at 29.21 115.57 0)
 		(unit 1)
 		(exclude_from_sim no)
@@
 		(fields_autoplaced yes)
 		(property "Reference" "#PWR05"
-			(at 29.21 123.19 0)
+			(at 29.21 119.38 0)
 			(effects
 				(font
@@
 		)
 		(property "Value" "VBUS"
-			(at 29.21 114.3 0)
+			(at 29.21 110.49 0)
 			(effects
 				(font
@@
 		)
 		(property "Footprint" ""
-			(at 29.21 119.38 0)
+			(at 29.21 115.57 0)
 			(effects
 				(font
@@
 		)
 		(property "Datasheet" ""
-			(at 29.21 119.38 0)
+			(at 29.21 115.57 0)
 			(effects
 				(font
@@
 		)
 		(property "Description" "Power symbol creates a global label with name \"VBUS\""
-			(at 29.21 119.38 0)
+			(at 29.21 115.57 0)
 			(effects
 				(font
@@
 	(symbol
 		(lib_id "Device:C_Small")
+		(at 34.29 116.84 90)
+		(unit 1)
+		(exclude_from_sim no)
+		(in_bom yes)
+		(on_board yes)
+		(dnp no)
+		(fields_autoplaced yes)
+		(property "Reference" "C2"
+			(at 34.2963 110.49 90)
+			(effects
+				(font
+					(size 1.27 1.27)
+				)
+			)
+		)
+		(property "Value" "0u1"
+			(at 34.2963 113.03 90)
+			(effects
+				(font
+					(size 1.27 1.27)
+				)
+			)
+		)
+		(property "Footprint" "Capacitor_SMD:C_0603_1608Metric"
+			(at 34.29 116.84 0)
+			(effects
+				(font
+					(size 1.27 1.27)
+				)
+				(hide yes)
+			)
+		)
+		(property "Datasheet" "~"
+			(at 34.29 116.84 0)
+			(effects
+				(font
+					(size 1.27 1.27)
+				)
+				(hide yes)
+			)
+		)
+		(property "Description" "Unpolarized capacitor, small symbol"
+			(at 34.29 116.84 0)
+			(effects
+				(font
+					(size 1.27 1.27)
+				)
+				(hide yes)
+			)
+		)
+		(pin "2"
+		)
+		(pin "1"
+		)
+		(instances
+			(project ""
+				(path "/450caee3-b68b-423d-a829-37eac74bf274"
+					(reference "C2")
+					(unit 1)
+				)
+			)
+		)
+	)
+	(symbol
+		(lib_id "Device:C_Small")
 		(at 162.56 148.59 90)
 		(mirror x)
@@
 	)
 	(symbol
-		(lib_id "Device:C_Small")
-		(at 31.75 116.84 0)
-		(mirror y)
-		(unit 1)
-		(exclude_from_sim no)
-		(in_bom yes)
-		(on_board yes)
-		(dnp no)
-		(property "Reference" "C2"
-			(at 34.29 118.1165 0)
-			(effects
-				(font
-					(size 1.27 1.27)
-				)
-				(justify right)
-			)
-		)
-		(property "Value" "0u1"
-			(at 34.29 115.5765 0)
-			(effects
-				(font
-					(size 1.27 1.27)
-				)
-				(justify right)
-			)
-		)
-		(property "Footprint" "Capacitor_SMD:C_0603_1608Metric"
-			(at 31.75 116.84 0)
-			(effects
-				(font
-					(size 1.27 1.27)
-				)
-				(hide yes)
-			)
-		)
-		(property "Datasheet" "~"
-			(at 31.75 116.84 0)
-			(effects
-				(font
-					(size 1.27 1.27)
-				)
-				(hide yes)
-			)
-		)
-		(property "Description" "Unpolarized capacitor, small symbol"
-			(at 31.75 116.84 0)
-			(effects
-				(font
-					(size 1.27 1.27)
-				)
-				(hide yes)
-			)
-		)
-		(pin "2"
-		)
-		(pin "1"
-		)
-		(instances
-			(project "musicbox"
-				(path "/450caee3-b68b-423d-a829-37eac74bf274"
-					(reference "C2")
-					(unit 1)
-				)
-			)
-		)
-	)
-	(symbol
 		(lib_id "power:VBUS")
 		(at 20.32 146.05 0)
@@
 	(symbol
 		(lib_id "power:GND")
-		(at 31.75 114.3 90)
+		(at 36.83 116.84 90)
 		(unit 1)
 		(exclude_from_sim no)
@@
 		(fields_autoplaced yes)
 		(property "Reference" "#PWR06"
-			(at 38.1 114.3 0)
+			(at 43.18 116.84 0)
 			(effects
 				(font
@@
 		)
 		(property "Value" "GND"
-			(at 35.56 114.2999 90)
+			(at 40.64 116.8399 90)
 			(effects
 				(font
@@
 		)
 		(property "Footprint" ""
-			(at 31.75 114.3 0)
+			(at 36.83 116.84 0)
 			(effects
 				(font
@@
 		)
 		(property "Datasheet" ""
-			(at 31.75 114.3 0)
+			(at 36.83 116.84 0)
 			(effects
 				(font
@@
 		)
 		(property "Description" "Power symbol creates a global label with name \"GND\" , ground"
-			(at 31.75 114.3 0)
+			(at 36.83 116.84 0)
 			(effects
 				(font

Commit message: -
Parts:
- removed J5: OUT1, Connector_JST:JST_ZH_S2B-ZR-SM4A-TF_1x02-1MP_P1.50mm_Horizontal, symbol Connector_Generic_MountingPin:Conn_01x02_MountingPin
- added JP1: BATT, Resistor_SMD:R_0603_1608Metric, symbol Jumper:Jumper_2_Open
- added R17: 10k, Resistor_SMD:R_0603_1608Metric, symbol Device:R_Small
- added SW3: POW, Library:IS-1245T-G, symbol Switch:SW_SPDT
- J4: footprint Connector_JST:JST_XH_S2B-XH-A_1x02_P2.50mm_Horizontal -> Connector_JST:JST_ZH_S2B-ZR-SM4A-TF_1x02-1MP_P1.50mm_Horizontal; symbol Connector:Conn_01x02_Socket -> Connector_Generic_MountingPin:Conn_01x02_MountingPin
Connections:
- net +BATT: now also JP1.1 (A)
- net GND: now also J4.MP (MountPin)
- net VBUS: now also SW3.3 (C); no longer Q1.1 (G)
- net +5V: no longer names the net of C6.1, Q1.2 (S), U5.4 (VOUT)
- net +5V: now also JP1.2 (B), SW3.1 (A)
- new net: R17.1, SW3.2 (B)
- new net: Q1.1 (G), R17.2
Other:
- moved on the sheet: C6, J3, L1, Q1, R11, TP1, TP2, U5, U6, U7

Commit message: -
Parts:
- removed J2: UPDI, Connector_PinSocket_2.54mm:PinSocket_1x02_P2.54mm_Vertical, symbol Connector:Conn_01x02_Socket
- removed R17: 10k, Resistor_SMD:R_0603_1608Metric, symbol Device:R_Small
- added R15: 10k, Resistor_SMD:R_0603_1608Metric, symbol Device:R_Small
- added TP1: GND, TestPoint:TestPoint_Pad_1.5x1.5mm, symbol Connector:TestPoint
- added TP2: UPDI, TestPoint:TestPoint_Pad_D1.5mm, symbol Connector:TestPoint
- R12: renamed from R15; value NC(2k2) -> NC(1k)
- R13: renamed from R16; value NC(2k2) -> NC(1k)
- renumbered C9 to C10, C8 to C11, C10 to C12, C5 to C4, C4 to C5, C11 to C7, C12 to C8, C7 to C9, J3 to J2, J4 to J3, R12 to R10, R13 to R11, R10 to R14, R11 to R16, R14 to R17, TP1 to TP3, TP2 to TP4, U8 to U6, U6 to U8
Connections:
- net GND: now also TP1.1
- net UPDI: now also TP2.1
- net VBUS: now also R15.2; no longer SW3.3 (C)
- net at SW3.2 (B): now also Q1.1 (G)
- new net: R15.1, SW3.3 (C)
Other:
- moved on the sheet: Q1, SW3, U7, U8

Commit message: -
Parts:
- removed SW2: SW, Library:alps-skrp, symbol Switch:SW_Push
- SW1: footprint Library:alps-skrg -> Library:alps-skr[gp]
Changed lines of the file:
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@@
-		)
-	)
-	(global_label "BTN"
-		(shape output)
-		(at 151.13 171.45 90)
-		(fields_autoplaced yes)
-		(effects
-			(font
-				(size 1.27 1.27)
-			)
-			(justify left)
-		)
-		(property "Intersheetrefs" "${INTERSHEET_REFS}"
-			(at 151.13 164.8967 90)
-			(effects
-				(font
-					(size 1.27 1.27)
-				)
-				(justify left)
-				(hide yes)
-			)
 		)
 	)
@@
 			)
 		)
-		(property "Footprint" "Library:alps-skrg"
+		(property "Footprint" "Library:alps-skr[gp]"
 			(at 147.32 176.53 0)
 			(effects
@@
 				(path "/450caee3-b68b-423d-a829-37eac74bf274"
 					(reference "#PWR024")
-					(unit 1)
-				)
-			)
-		)
-	)
-	(symbol
-		(lib_id "power:GND")
-		(at 151.13 181.61 0)
-		(unit 1)
-		(exclude_from_sim no)
-		(in_bom yes)
-		(on_board yes)
-		(dnp no)
-		(fields_autoplaced yes)
-		(property "Reference" "#PWR037"
-			(at 151.13 187.96 0)
-			(effects
-				(font
-					(size 1.27 1.27)
-				)
-				(hide yes)
-			)
-		)
-		(property "Value" "GND"
-			(at 151.13 186.69 0)
-			(effects
-				(font
-					(size 1.27 1.27)
-				)
-			)
-		)
-		(property "Footprint" ""
-			(at 151.13 181.61 0)
-			(effects
-				(font
-					(size 1.27 1.27)
-				)
-				(hide yes)
-			)
-		)
-		(property "Datasheet" ""
-			(at 151.13 181.61 0)
-			(effects
-				(font
-					(size 1.27 1.27)
-				)
-				(hide yes)
-			)
-		)
-		(property "Description" "Power symbol creates a global label with name \"GND\" , ground"
-			(at 151.13 181.61 0)
-			(effects
-				(font
-					(size 1.27 1.27)
-				)
-				(hide yes)
-			)
-		)
-		(pin "1"
-		)
-		(instances
-			(project "musicbox"
-				(path "/450caee3-b68b-423d-a829-37eac74bf274"
-					(reference "#PWR037")
 					(unit 1)
 				)
@@
 					(unit 1)
 				)
-			)
-		)
-	)
-	(symbol
-		(lib_id "Switch:SW_Push")
-		(at 151.13 176.53 270)
-		(mirror x)
-		(unit 1)
-		(exclude_from_sim no)
-		(in_bom yes)
-		(on_board yes)
-		(dnp no)
-		(property "Reference" "SW2"
-			(at 149.86 175.2599 90)
-			(effects
-				(font
-					(size 1.27 1.27)
-				)
-				(justify right)
-			)
-		)
-		(property "Value" "SW"
-			(at 149.86 177.7999 90)
-			(effects
-				(font
-					(size 1.27 1.27)
-				)
-				(justify right)
-			)
-		)
-		(property "Footprint" "Library:alps-skrp"
-			(at 156.21 176.53 0)
-			(effects
-				(font
-					(size 1.27 1.27)
-				)
-				(hide yes)
-			)
-		)
-		(property "Datasheet" "~"
-			(at 156.21 176.53 0)
-			(effects
-				(font
-					(size 1.27 1.27)
-				)
-				(hide yes)
-			)
-		)
-		(property "Description" "Push button switch, generic, two pins"
-			(at 151.13 176.53 0)
-			(effects
-				(font
-					(size 1.27 1.27)
-				)
-				(hide yes)
-			)
-		)
-		(pin "2"
-		)
-		(pin "1"
-		)
-		(instances
-			(project "musicbox"
-				(path "/450caee3-b68b-423d-a829-37eac74bf274"
-					(reference "SW2")
-					(unit 1)
-				)

Commit message: -
Connections:
- net at C7.1, R12.1: now also U6.2; no longer U6.2'
- net at C8.1, R13.2: now also U6.2'; no longer U6.2
- net at U6.3: now also R10.2; no longer R11.2
- net at U6.3': now also R11.2; no longer R10.2
Changed lines of the file:
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@@
 	)
 	(junction
+		(at 143.51 140.97)
+		(diameter 0)
+		(color 0 0 0 0)
+	)
+	(junction
 		(at 149.86 133.35)
 		(diameter 0)
@@
 	)
 	(junction
-		(at 143.51 140.97)
-		(diameter 0)
-		(color 0 0 0 0)
-	)
-	(junction
 		(at 140.97 25.4)
 		(diameter 0)
@@
 	(wire
 		(pts
-			(xy 143.51 140.97) (xy 149.86 140.97)
-		)
-		(stroke
-			(width 0)
-			(type default)
-		)
-	)
-	(wire
-		(pts
 			(xy 40.64 35.56) (xy 40.64 38.1)
 		)
@@
 	(wire
 		(pts
-			(xy 143.51 140.97) (xy 143.51 146.05)
+			(xy 143.51 140.97) (xy 143.51 135.89)
 		)
 		(stroke
@@
 	(wire
 		(pts
+			(xy 143.51 140.97) (xy 149.86 140.97)
+		)
+		(stroke
+			(width 0)
+			(type default)
+		)
+	)
+	(wire
+		(pts
 			(xy 149.86 134.62) (xy 149.86 133.35)
 		)
@@
 		(lib_id "Library:alps-rk10j12e")
 		(at 135.89 140.97 90)
+		(mirror x)
 		(unit 1)
 		(exclude_from_sim no)
@@
 		(dnp no)
 		(property "Reference" "U6"
-			(at 130.048 133.858 90)
+			(at 130.048 148.082 90)
 			(effects
 				(font
@@
 		)
 		(property "Value" "alps-rk10j12e"
-			(at 130.302 129.032 90)
+			(at 130.302 152.908 90)
 			(effects
 				(font
@@
 	(symbol
 		(lib_id "power:GND")
-		(at 143.51 140.97 180)
+		(at 143.51 140.97 0)
+		(mirror y)
 		(unit 1)
 		(exclude_from_sim no)
@@
 		(dnp no)
 		(property "Reference" "#PWR036"
-			(at 143.51 134.62 0)
+			(at 143.51 147.32 0)
 			(effects
 				(font
@@
 		)
 		(property "Value" "GND"
-			(at 143.51 135.89 0)
+			(at 143.51 146.05 0)
 			(effects
 				(font

Commit message: -
Parts:
- R10, R11: value 10k -> 47k
Changed lines of the file:
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@@
 			)
 		)
-		(property "Value" "10k"
+		(property "Value" "47k"
 			(at 128.27 146.05 90)
 			(effects
@@
 			)
 		)
-		(property "Value" "10k"
+		(property "Value" "47k"
 			(at 128.27 135.89 90)
 			(effects

Commit message: -
Parts:
- added R7: 56k, Resistor_SMD:R_0603_1608Metric, symbol Device:R_Small
- R6: value 27k -> 56k
- renumbered R9 to R10, R10 to R11, R11 to R12, R12 to R13, R13 to R14, R14 to R15, R15 to R16, R16 to R17, R17 to R18, R7 to R8, R8 to R9, SW3 to SW2
Connections:
- net GND: now also R7.2
- net VSET: now also R7.1
Other:
- moved on the sheet: R5, R6

Commit message: -
Parts:
- removed D1: TNOW, LED_SMD:LED_0603_1608Metric, symbol Device:LED_Small
- renumbered D2 to D1, D3 to D2, R11 to R10, R12 to R11, R13 to R12, R14 to R13, R4 to R14, R5 to R4, R6 to R5, R7 to R6, R8 to R7, R9 to R8, R10 to R9
Connections:
- net VBUS: now also U8.3 (VO-); no longer U8.2 (VO-)
- net VCC: now also U7.2 (VO+), U8.2 (VO+); no longer U7.3 (VO+), U8.3 (VO+)
- net at D2.2 (A), R15.2: now also R14.2
- net at Q1.3 (D): now also U7.3 (VO-); no longer U7.2 (VO-)
Other:
- moved on the sheet: D2, R14
