File: proj/avr/n_scale_pu/n_scale_pu.kicad_pcb (KiCad board)
At the start: 2 copper layers, 40 parts, among them J1 USB_C_Receptacle_USB2.0_16P, J2 feeder, J3 UPDI, J4 tcn, SW1 SW_Push, SW2 SW_Push, SW3 SW_Push, SW4 SW_Push, SW5 SW_Push, U1 CH221K, U2 ATtiny1604-SS, U3 AM2837, U4 AP2204K-5.0

Commit message: -
Parts:
- removed D10, D11, D12, D13, D14, D9: WS2812B-2020, LED_SMD:LED_WS2812B-2020_PLCC4_2.0x2.0mm
- removed R5: 2k2, Resistor_SMD:R_0603_1608Metric
- removed RV1: volume, Potentiometer_SMD:Potentiometer_Bourns_TC33X_Vertical
- removed SW5: SW_Push, Library:alps-skrg
- added C5: 1u, Capacitor_SMD:C_0603_1608Metric, F.Cu at (140.5, 95.0)
- added C6: 1u, Capacitor_SMD:C_0603_1608Metric, F.Cu at (140.5, 97.5)
- added R8: 4k7, Resistor_SMD:R_0603_1608Metric, F.Cu at (140.5, 100.0)
- added U5: AQM0802A-RN-GBW, Library:AQM0802A-RN-GBW, F.Cu at (154.2, 79.7)
- U4: value AP2204K-5.0 -> AP7375; footprint Package_TO_SOT_SMD:SOT-23-5 -> Package_TO_SOT_SMD:SOT-23-3
- moved U4 61.8 mm to (145.0, 95.9)
- moved D1 31.6 mm to (183.5, 112.2)
- moved D2 31.6 mm to (183.5, 115.7)
- moved D3 31.6 mm to (183.5, 119.2)
- moved D6 31.6 mm to (187.8, 112.2)
- moved D7 31.6 mm to (187.8, 115.7)
- moved D8 31.6 mm to (187.8, 119.2)
- moved D4 31.6 mm to (183.5, 122.8)
- moved D5 31.6 mm to (183.5, 126.3)
Connections:
- BZ1 pad 1: Net-(BZ1-+) -> SPK
- D8 pad 1: Net-(D8-DOUT) -> unconnected-(D8-DOUT-Pad1)
- R6 pad 1: VBUS -> Net-(R6-Pad1)
- U2 pad 1: +5V -> +3V3
- U2 pad 3: BTN5 -> V_SENSE
- U2 pad 4: ~{PG} -> NP
- U2 pad 5: V_SENSE -> SPK
- U2 pad 6: NP -> WO0
- U2 pad 8: WO1 -> SDA_3V3
- U2 pad 9: WO0 -> SCL_3V3
- U3 pad 2: WO1 -> WO2
- U4 pad 2: GND -> +5V
- U4 pad 3: VBUS -> GND

Commit message: -
Parts:
- added R8: 4k7, Resistor_SMD:R_0603_1608Metric, F.Cu at (85.0, 156.1)
- added R9: 4k7, Resistor_SMD:R_0603_1608Metric, F.Cu at (85.0, 158.6)
- renumbered C4 to C1, C1 to C2, C2 to C3, C3 to C4, J3 to J2, J2 to J3, R4 to R3, R3 to R4, R8 to R5, U4 to U2, U2 to U3, U5 to U4, U3 to U5

Commit message: -
Parts:
- removed J4: tcn, Connector_PinHeader_2.54mm:PinHeader_1x02_P2.54mm_Vertical
- added ?: , Library:PCB.MCBEERINGI.DEV_small, B.Cu at (112.0, 105.0)
- added ?: LOGO, Library:mcbeeringi_icon_10mm, B.Cu at (112.0, 98.0)
- BZ1, C2, C3, C4, C5, C6, J1, J3, R1, R2, R3, R4, R5, R6, R7, U1, U2, U3, U5: moved to B.Cu
- R8, R9: value 4k7 -> 10k; moved to B.Cu
- SW1, SW2, SW3, SW4: footprint Library:alps-skrg -> Library:alps-skr[gp]
- moved D1 97.5 mm to (86.0, 111.0), turned to 180 degrees
- moved D2 93.6 mm to (90.0, 111.0), turned to 180 degrees
- moved D3 89.9 mm to (94.0, 111.0), turned to 180 degrees
- moved D4 86.3 mm to (98.0, 111.0), turned to 180 degrees
- moved D5 82.9 mm to (102.0, 111.0), turned to 180 degrees
- moved D6 81.8 mm to (106.0, 111.0), turned to 180 degrees
- moved D7 77.9 mm to (110.0, 111.0), turned to 180 degrees
- moved D8 74.3 mm to (114.0, 111.0), turned to 180 degrees
- moved BZ1 58.2 mm to (87.4, 104.0), turned to -90 degrees
- moved U5 58.1 mm to (106.0, 94.0), turned to 90 degrees
- moved U4 56.6 mm to (100.0, 96.0)
- moved SW2 51.0 mm to (80.4, 109.0), turned to 90 degrees
- moved R9 50.9 mm to (104.0, 111.4), turned to 90 degrees
- moved SW1 50.3 mm to (80.4, 99.0), turned to -90 degrees
- moved R8 49.2 mm to (105.6, 111.4), turned to 90 degrees
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Connections:
- U1 pad 3: ~{PG} -> unconnected-(U1-PG#-Pad3)
- U3 pad 11: BTN1 -> BTN4
- U3 pad 12: BTN2 -> NP
- U3 pad 13: BTN3 -> BTN2
- U3 pad 2: BTN4 -> BTN1
- U3 pad 3: V_SENSE -> SPK
- U3 pad 4: NP -> BTN3
- U3 pad 5: SPK -> V_SENSE
- U5 pad 1: WO0 -> WO2
- U5 pad 2: WO2 -> WO0
Routing:
- net +3V3: track 0.00 -> 33.6 mm, vias 0 -> 4
- net UPDI: track 0.00 -> 30.6 mm
- net BTN3: track 0.00 -> 25.2 mm, vias 0 -> 1
- net BTN4: track 0.00 -> 25.0 mm, vias 0 -> 1
- net BTN1: track 0.00 -> 22.6 mm, vias 0 -> 1
- net BTN2: track 0.00 -> 22.4 mm, vias 0 -> 1
- net VBUS: track 0.00 -> 17.5 mm, vias 0 -> 10
- net NP: track 0.00 -> 16.8 mm, vias 0 -> 1
- net SPK: track 0.00 -> 15.2 mm
- net CC1: track 0.00 -> 10.3 mm
- net CC2: track 0.00 -> 9.48 mm
- net SCL_3V3: track 0.00 -> 8.47 mm
- net WO0: track 0.00 -> 7.15 mm
- net WO2: track 0.00 -> 6.68 mm
- net SDA_3V3: track 0.00 -> 4.85 mm
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- added copper zone on B.Cu, net +3V3
- added copper zone on F.Cu, net +3V3
- added copper zone on F.Cu, net +5V
- added copper zone on B.Cu, net GND
- added copper zone on F.Cu, net GND
- added copper zone on B.Cu, net Net-(J3-Pin_1)
- added copper zone on B.Cu, net Net-(J3-Pin_2)
- added copper zone on F.Cu, net VBUS
Other:
- board outline added: 48 x 28 mm
- board text added: "10k"
- board text added: "10k *2"
- board text added: "1k"
- board text added: "1u"
- board text added: "1u *2"
- board text added: "470u"
- board text added: "47k"
- board text added: "4k7"
- board text added: "4k7 *2"
- board text added: "4u7"
- board text added: "ALPS-SKR[GP]"
- board text added: "AM2837"
- board text added: "AP7375"
- board text added: "AQM0802A-RN-GBW"
- board text added: "ATtiny X04"
- board text added: "AVR N_SCALE_PU"
- board text added: "CH221K"
- board text added: "GND"
- board text added: "PA1"
- board text added: "PA2"
- board text added: "PA3"
- board text added: "PA4"
- board text added: "PA6"
- board text added: "PKLCS1212E4001-R1"
- board text added: "UPDI"
- board text added: "USB4105"
- board text added: "WS2812C-2020"

Commit message: -
Parts:
- R5: value 4k7 -> 10k
Changed lines of the file:
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@@
 		)
 		(fp_rect
+			(start -15.8 -3)
+			(end -15 3)
+			(stroke
+				(width 0.1)
+				(type solid)
+			)
+			(fill no)
+			(layer "F.Fab")
+		)
+		(fp_rect
 			(start -15 -6.75)
 			(end 15 12.75)
@@
 			)
 		)
+		(fp_text user "BACKLIGHT_LENS"
+			(at -15.4 0 270)
+			(unlocked yes)
+			(layer "F.Fab")
+			(effects
+				(font
+					(size 0.4 0.4)
+					(thickness 0.05)
+				)
+			)
+		)
 		(pad "1" thru_hole roundrect
 			(at -6 12.9)
@@
 			)
 		)
-		(property "Value" "4k7"
+		(property "Value" "10k"
 			(at 0 -1.43 90)
 			(layer "B.Fab")
@@
 		)
 	)
-	(gr_text "4k7"
+	(gr_text "10k"
 		(at 101.8 93.4 0)
 		(layer "B.Mask")

Commit message: -
Parts:
- removed the C1 at (119.6, 88.7)
- removed J2: UPDI, Connector_PinSocket_2.54mm:PinSocket_1x02_P2.54mm_Vertical
- removed J3: feeder, Connector_PinHeader_2.54mm:PinHeader_1x02_P2.54mm_Vertical
- removed the R6 at (102.6, 98.4)
- added C2: 0u1, Capacitor_SMD:C_0603_1608Metric, B.Cu at (115.6, 94.6)
- added C5: 47u, Capacitor_SMD:C_1210_3225Metric, B.Cu at (101.4, 98.0)
- added C6: 47u, Capacitor_SMD:C_1210_3225Metric, B.Cu at (98.0, 98.0)
- added C7: 47u, Capacitor_SMD:C_1210_3225Metric, B.Cu at (94.6, 98.0)
- added D1: SK6112-SIDE-RG-A, Library:SK6112-SIDE-RG-A, F.Cu at (84.0, 100.0)
- added R4: 4k7, Resistor_SMD:R_0603_1608Metric, B.Cu at (112.4, 94.6)
- added TP1: GND, TestPoint:TestPoint_Pad_1.5x1.5mm, B.Cu at (106.0, 108.4)
- added TP2: UPDI, TestPoint:TestPoint_Pad_D1.5mm, B.Cu at (106.0, 105.6)
- added TP3: OUT_A, TestPoint:TestPoint_Pad_1.5x1.5mm, B.Cu at (107.4, 88.0)
- added TP4: OUT_B, TestPoint:TestPoint_Pad_D1.5mm, B.Cu at (104.6, 88.0)
- added U1: CH340E, Package_SO:MSOP-10_3x3mm_P0.5mm, B.Cu at (114.0, 92.0)
- J1: footprint Connector_USB:USB_C_Receptacle_GCT_USB4105-xx-A_16P_TopMnt_Horizontal -> Connector_USB:USB_C_Receptacle_GCT_USB4110
- moved C4 25.8 mm to (86.0, 97.0)
- moved U2 25.5 mm to (89.0, 96.4)
- moved C1 24.6 mm to (92.0, 98.0)
- moved D2 22.0 mm to (86.0, 89.0), turned to -90 degrees
- moved D3 22.0 mm to (90.0, 89.0), turned to -90 degrees
- moved D4 22.0 mm to (94.0, 89.0), turned to -90 degrees
- moved D5 22.0 mm to (98.0, 89.0), turned to -90 degrees
- moved D6 22.0 mm to (102.0, 89.0), turned to -90 degrees
- moved D7 22.0 mm to (106.0, 89.0), turned to -90 degrees
- moved D8 22.0 mm to (110.0, 89.0), turned to -90 degrees
- moved D9 22.0 mm to (114.0, 89.0), turned to -90 degrees
- moved C3 19.6 mm to (82.4, 88.6), turned to 90 degrees
- moved R3 16.8 mm to (85.0, 88.0), turned to 180 degrees
- moved R5 14.6 mm to (82.4, 91.6), turned to -90 degrees
- moved U3 13.6 mm to (85.0, 91.0), turned to -90 degrees
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- renumbered C3 to C1, C2 to C3, C5 to C8, C6 to C9, D1 to D2, D2 to D3, D3 to D4, D4 to D5, D5 to D6, D6 to D7, D7 to D8, D8 to D9, R4 to R5, R5 to R6, U1 to U3, U3 to U4, U4 to U5, U5 to U6
Connections:
- net SCL_3V3 renamed SCL
- net SDA_3V3 renamed SDA
- C8 pad 1: +3V3 -> +5V
- D2 pad 3: NP -> Net-(D1-DOUT)
- J1 pad A6: unconnected-(J1-D+-PadA6) -> D+
- J1 pad A7: unconnected-(J1-D--PadA7) -> D-
- J1 pad B6: unconnected-(J1-D+-PadB6) -> D+
- J1 pad B7: unconnected-(J1-D--PadB7) -> D-
- R6 pad 2: Net-(R5-Pad2) -> V_SENSE
- R8 pad 1: +3V3 -> +5V
- R9 pad 1: +3V3 -> +5V
- U4 pad 1: +3V3 -> +5V
- U5 pad 5: +3V3 -> +5V
- U5 pad 9: +3V3 -> +5V
Routing:
- net +3V3: track 33.6 -> 0.00 mm, vias 4 -> 0
- net D-: track 0.00 -> 23.4 mm, vias 0 -> 2
- net D+: track 0.00 -> 22.0 mm, vias 0 -> 2
- net Net-(D1-DOUT): track 0.00 -> 11.3 mm
- net CC2: track 9.48 -> 15.3 mm
- net NP: track 16.8 -> 21.6 mm
- net Net-(U1-TXD): track 0.00 -> 4.45 mm
- net BTN1: track 22.6 -> 26.7 mm
- net UPDI: track 30.6 -> 26.5 mm
- net VBUS: track 17.5 -> 14.1 mm, vias 10 -> 13
- net BTN3: track 25.2 -> 27.8 mm
- net CC1: track 10.3 -> 12.8 mm
- net Net-(R5-Pad2): track 2.01 -> 0.00 mm
- net SPK: track 15.2 -> 13.5 mm
- net Net-(U1-V3): track 0.00 -> 1.71 mm
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- added copper zone on B.Cu, net +5V
- added copper zone on B.Cu, net VBUS
- removed copper zone on F.Cu, net +3V3
Other:
- board text added: "0u1"
- board text added: "47u *3"
- board text added: "CH340E"
- board text added: "PKLCS1212E 4001-R1"
- board text added: "SK6112-SIDE-RG-A"
- board text added: "USB4110"
- board text added: "↑ WS2812C-2020 *8 ↑"
- board text added: "↓ AQM0802A-RN-GBW ↓"
- board text removed: "470u"
- board text removed: "AQM0802A-RN-GBW"
- board text removed: "PA3"
- board text removed: "PKLCS1212E4001-R1"
- board text removed: "USB4105"
- board text removed: "WS2812C-2020"

Commit message: -
Parts:
- added C1: 0u1, Capacitor_SMD:C_0603_1608Metric, B.Cu at (114.0, 90.4)
- added C6: 4u7, Capacitor_SMD:C_0603_1608Metric, B.Cu at (94.6, 106.0)
- moved ? 1.00 mm to (115.0, 109.0)
- moved ? 1.00 mm to (115.0, 101.0)
- moved C3 1.00 mm to (115.6, 95.6)
- moved R4 1.00 mm to (112.4, 95.6)
- moved U1 1.00 mm to (114.0, 93.0)
- renumbered C8 to C10, C9 to C11, C1 to C2, C2 to C3, C3 to C4, C4 to C5, C5 to C7, C6 to C8, C7 to C9
Routing:
- net +5V: track 1.35 -> 3.12 mm
- net UPDI: track 26.5 -> 25.5 mm

Commit message: -
Routing:
- net GND: vias 41 -> 43
Changed lines of the file:
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@@
+	)
+	(via
+		(at 115 95.6)
+		(size 0.5)
+		(drill 0.3)
+		(layers "F.Cu" "B.Cu")
+		(net 1)
 	)
 	(via
@@
 		(size 0.5)
 		(drill 0.3)
+		(layers "F.Cu" "B.Cu")
+		(free yes)
+		(net 1)
+	)
+	(via
+		(at 114 93)
+		(size 0.5)
+		(drill 0.3)
