File: proj/usb/nimh-5v/nimh-5v.kicad_pcb (KiCad board)
At the start: 2 copper layers, 44 x 19 mm, 26 parts, among them J1 USB, J2 USB_A, Q1 AO3401A, SW1 SW_Push, U1 BQ25172, U2 TPS613222ADBV, U3 CH213K, U4 CH213K

Commit message: -
Connections:
- U3 pad 2: Net-(Q1-D) -> VCC
- U3 pad 3: VCC -> Net-(Q1-D)
- U4 pad 2: VBUS -> VCC
- U4 pad 3: VCC -> VBUS
Routing:
- net VCC: vias 4 -> 6
- net VBUS: vias 11 -> 9
Changed lines of the file:
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@@
 			(layers "F.Cu" "F.Mask" "F.Paste")
 			(roundrect_rratio 0.25)
-			(net 12 "Net-(Q1-D)")
-			(pinfunction "VO-")
+			(net 11 "VCC")
+			(pinfunction "VO+")
 			(pintype "passive")
 		)
@@
 			(layers "F.Cu" "F.Mask" "F.Paste")
 			(roundrect_rratio 0.25)
-			(net 11 "VCC")
-			(pinfunction "VO+")
+			(net 12 "Net-(Q1-D)")
+			(pinfunction "VO-")
 			(pintype "passive")
 		)
@@
 			(layers "F.Cu" "F.Mask" "F.Paste")
 			(roundrect_rratio 0.25)
-			(net 3 "VBUS")
-			(pinfunction "VO-")
+			(net 11 "VCC")
+			(pinfunction "VO+")
 			(pintype "passive")
 		)
@@
 			(layers "F.Cu" "F.Mask" "F.Paste")
 			(roundrect_rratio 0.25)
-			(net 11 "VCC")
-			(pinfunction "VO+")
+			(net 3 "VBUS")
+			(pinfunction "VO-")
 			(pintype "passive")
 		)
@@
 	)
 	(via
-		(at 92.4 108)
-		(size 0.5)
-		(drill 0.3)
-		(layers "F.Cu" "B.Cu")
-		(net 3)
-	)
-	(via
 		(at 84.8 101.6)
 		(size 0.5)
@@
 	(via
 		(at 90.2 108)
-		(size 0.5)
-		(drill 0.3)
-		(layers "F.Cu" "B.Cu")
-		(net 3)
-	)
-	(via
-		(at 91.8 108)
 		(size 0.5)
 		(drill 0.3)
@@
 	)
 	(via
+		(at 92.4 108)
+		(size 0.5)
+		(drill 0.3)
+		(layers "F.Cu" "B.Cu")
+		(net 11)
+	)
+	(via
 		(at 98 106.2)
 		(size 0.5)
@@
 		(net 11)
 	)
+	(via
+		(at 91.8 108)
+		(size 0.5)
+		(drill 0.3)
+		(layers "F.Cu" "B.Cu")
+		(net 11)
+	)

Commit message: -
Parts:
- moved R8 4.53 mm to (91.6, 104.0)
- moved U3 1.08 mm to (94.2, 103.4), turned to 90 degrees
- moved Q1 0.72 mm to (92.6, 100.8), turned to 0 degrees
- turned U4 to 180 degrees
Routing:
- net Net-(Q1-G): track 13.6 -> 15.8 mm
- net VCC: vias 6 -> 4
- net VBUS: vias 9 -> 11
Other:
- board text added: "TPS613222A"
- board text removed: "TPS61 3222A"

Commit message: -
Parts:
- removed the ? at (87.4, 94.0)
- removed U3, U4: CH213K, Package_TO_SOT_SMD:SOT-23
- added ?: pcb.6ca.me, Library:pcb.6ca.me_5mm, F.Cu at (84.5, 91.5)
- added D2: CUHS20S30, Library:US2H, F.Cu at (93.2, 106.2)
- added D3: CUHS20S30, Library:US2H, F.Cu at (93.2, 108.0)
- moved R8 3.93 mm to (92.6, 100.2), turned to 180 degrees
- moved Q1 2.40 mm to (92.6, 103.2), turned to -90 degrees
Routing:
- net Net-(Q1-G): track 15.8 -> 11.7 mm
- removed copper zone on F.Cu, net VCC
Other:
- board text added: "CUHS20S30 *2"
- board text removed: "CH213K"
