File: proj/usb/nimh-5v/nimh-5v.kicad_sch (KiCad schematic)
At the start: 24 parts, among them J1 USB, J2 USB_A, Q1 AO3401A, SW1 SW_Push, U1 BQ25172, U2 TPS613222ADBV, U3 CH213K, U4 CH213K

Commit message: -
Connections:
- net VBUS: now also U4.3 (VO-); no longer U4.2 (VO-)
- net VCC: now also U3.2 (VO+), U4.2 (VO+); no longer U3.3 (VO+), U4.3 (VO+)
- net at Q1.3 (D): now also U3.3 (VO-); no longer U3.2 (VO-)

Commit message: -
Parts:
- removed U3, U4: CH213K, Package_TO_SOT_SMD:SOT-23, symbol Library:CH213K
- added D2, D3: CUHS20S30, Library:US2H, symbol Device:D_Schottky
Connections:
- net VBUS: now also D3.2 (A)
- net VCC: now also D2.1 (K), D3.1 (K)
- net at Q1.3 (D): now also D2.2 (A)
