File: proj/musicbox/cube/cube.kicad_pcb (KiCad board)
At the start: 2 copper layers, 44 x 44 mm, 73 parts, among them J1 USB, J2 NiMh*2, J3 OUT1, Q1 AO3401A, SW1 SW, SW2 POW, U1 CH340E, U2 TPS56124x, U3 ATtiny402-SS, U4 ATtiny1604-SS, U5 alps-rk10j12e, U6 BQ25172, U7 TPS613222ADBV, U8 PAM8406D

Commit message: -
Parts:
- removed RV1: 10k, Potentiometer_SMD:Potentiometer_Bourns_TC33X_Vertical
- added R21: 10k, Resistor_SMD:R_0603_1608Metric, F.Cu at (83.4, 110.6)
- added R6: 10k, Resistor_SMD:R_0603_1608Metric, F.Cu at (85.8, 88.0)
- added R7: 10k, Resistor_SMD:R_0603_1608Metric, F.Cu at (83.8, 88.0)
- R8: renamed from R6; value 1k -> 4k7
- moved C8 1.80 mm to (86.6, 99.8)
- moved C9 1.80 mm to (86.6, 112.2)
- moved R8 1.60 mm to (82.2, 88.0)
- moved R18 1.28 mm to (83.4, 99.8), turned to 180 degrees
- moved R19 1.28 mm to (83.4, 112.2), turned to 180 degrees
- renumbered R8 to R10, R9 to R11, R10 to R12, R11 to R13, R12 to R14, R13 to R15, R14 to R16, R15 to R17, R16 to R18, R17 to R19, R18 to R20, R19 to R22, R20 to R23, R7 to R9
Routing:
- net Net-(U2-FB): track 14.1 -> 9.79 mm
- net ~{SD}: track 15.9 -> 18.2 mm
- net Net-(R6-Pad2): track 0.00 -> 2.02 mm
- net AMP1: track 2.24 -> 4.15 mm
- net Net-(C9-Pad1): track 38.5 -> 36.7 mm
- net Net-(C8-Pad1): track 45.4 -> 43.6 mm
- net AMP0: track 2.24 -> 3.94 mm
- net VBOOST: track 17.6 -> 18.2 mm
Other:
- board text added: "10k *2"
- board text added: "56k"
- board text removed: "1k"
- board text removed: "56k *2"
- board text removed: "V_{CHG}"
