File: proj/musicbox/cube/cube.kicad_sch (KiCad schematic)
At the start: 68 parts, among them J1 USB, J2 NiMh*2, J3 OUT1, Q1 AO3401A, SW1 SW, SW2 POW, U1 CH340E, U2 TPS56124x, U3 ATtiny402-SS, U4 ATtiny1604-SS, U5 alps-rk10j12e, U6 BQ25172, U7 TPS613222ADBV, U8 PAM8406D

Commit message: -
Parts:
- added R6: 1k, Resistor_SMD:R_0603_1608Metric, symbol Device:R_Small
- RV1: value R_FB -> 10k
- renumbered C11 to C10, C12 to C11, C13 to C12, C14 to C13, C15 to C14, C16 to C15, C8 to C7, C9 to C8, C10 to C9, R9 to R10, R10 to R11, R11 to R12, R12 to R13, R13 to R14, R14 to R15, R15 to R16, R16 to R17, R17 to R18, R18 to R19, R19 to R20, R6 to R7, R7 to R8, R8 to R9
Connections:
- net GND: now also R6.2; no longer RV1.3
- net at RV1.2, U2.6 (FB): now also RV1.3, R6.1
Other:
- moved on the sheet: C6, RV1

Commit message: -
Parts:
- removed RV1: 10k, Potentiometer_SMD:Potentiometer_Bourns_TC33X_Vertical, symbol Device:R_Potentiometer
- added R21, R6, R7: 10k, Resistor_SMD:R_0603_1608Metric, symbol Device:R_Small
- R8: renamed from R6; value 1k -> 4k7
- renumbered R8 to R10, R9 to R11, R10 to R12, R11 to R13, R12 to R14, R13 to R15, R14 to R16, R15 to R17, R16 to R18, R17 to R19, R18 to R20, R19 to R22, R20 to R23, R7 to R9
Connections:
- net GND: now also R21.2
- net VREG: now also R6.1
- net ~{SD}: now also R21.1
- net at R8.1, U2.6 (FB): now also R7.2
- new net: R6.2, R7.1
Other:
- moved on the sheet: C6, L1, R20, R8
