File: proj/musicbox/slim/slim.kicad_pcb (KiCad board)
At the start: 2 copper layers, 66 parts, among them J1 USB, J2 NiMh*3, J3 OUT0, J4 OUT2, Q1 AO3401A, SW1 SW, SW2 SW, SW3 SW, SW4 SW, SW5 POW, U1 CH340E, U2 TPS56124x, U3 AQM0802A-RN-GBW, U4 ATtiny1604-SS, U5 alps-rk10j12e, U6 BQ25172, U7 PAM8406D

Commit message: -
Parts:
- removed the C6 at (78.3, 106.2)
- removed the C8 at (82.3, 93.7)
- removed the R6 at (90.3, 96.2)
- removed the R7 at (90.3, 98.7)
- removed the U3 at (92.7, 78.4)
- added J2: I2C, Connector_JST:JST_ZH_B4B-ZR_1x04_P1.50mm_Vertical, F.Cu at (134.2, 97.6)
- added R10: 4k7, Resistor_SMD:R_0603_1608Metric, F.Cu at (133.7, 104.6)
- added R9: 4k7, Resistor_SMD:R_0603_1608Metric, F.Cu at (133.7, 102.1)
- J4: renamed from J3; moved to B.Cu
- J5: renamed from J4; moved to B.Cu
- moved J1 161.6 mm to (233.7, 59.1)
- moved R2 160.3 mm to (242.0, 63.0)
- moved R3 160.3 mm to (242.0, 65.5)
- moved C1 154.3 mm to (231.8, 78.4)
- moved R1 150.6 mm to (232.6, 70.6)
- moved R4 150.6 mm to (232.6, 73.1)
- moved C2 147.8 mm to (225.0, 78.2)
- moved C7 140.3 mm to (220.7, 119.1)
- moved C5 134.3 mm to (212.2, 93.6)
- moved C8 133.4 mm to (215.1, 116.9)
- moved C3 129.3 mm to (207.6, 95.0)
- moved C6 124.6 mm to (201.8, 92.2)
- moved R5 122.7 mm to (212.7, 85.0)
- moved R11 119.9 mm to (210.1, 115.9)
- moved R12 118.5 mm to (210.0, 119.4)
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- renumbered C11 to C10, C13 to C11, C14 to C12, C15 to C13, C16 to C14, C7 to C6, C9 to C7, C12 to C8, C10 to C9, J2 to J3, R3 to R1, R18 to R15, R17 to R16, R21 to R17, R22 to R18, R15 to R19, R1 to R2, R16 to R20, R23 to R21, R24 to R22, R19 to R23, R20 to R24, R2 to R3, R8 to R6, R9 to R7, R10 to R8, U4 to U3, U6 to U4, U7 to U6
Connections:
- R21 pad 1: GND -> ~{SD}
- R21 pad 2: ~{SD} -> GND
- U3 pad 11: MODE -> LED
- U3 pad 12: ~{SD} -> BTN1
- U3 pad 13: LED -> BTN2
- U3 pad 2: BTN1 -> BTN3
- U3 pad 3: BTN2 -> BTN4
- U3 pad 4: BTN3 -> MODE
- U3 pad 5: BTN4 -> ~{SD}
- U3 pad 8: SDA -> SCL
- U3 pad 9: SCL -> SDA

Commit message: -
Parts:
- removed the J2 at (134.2, 97.6)
- removed the R10 at (133.7, 104.6)
- removed the R13 at (210.0, 121.9)
- removed the R9 at (133.7, 102.1)
- removed the SW4 at (140.5, 178.9)
- added C9: 22u, Capacitor_SMD:C_0603_1608Metric, F.Cu at (240.8, 110.6)
- added JP2: SW, Resistor_SMD:R_0603_1608Metric, F.Cu at (168.4, 145.6)
- added L2: 4u7, Inductor_SMD:L_1008_2520Metric, F.Cu at (247.1, 108.7)
- added R11: 56k, Resistor_SMD:R_0603_1608Metric, F.Cu at (204.0, 126.8)
- added R16: 10k, Resistor_SMD:R_0603_1608Metric, F.Cu at (125.4, 148.4)
- added U2: TS5A23159DGS, Package_SO:TSSOP-10_3x3mm_P0.5mm, F.Cu at (228.4, 82.6)
- added U6: TPS613222ADBV, Package_TO_SOT_SMD:SOT-23-5, F.Cu at (247.2, 104.6)
- J2: renamed from J3; value NiMh*3 -> NiMh*2
- J4: renamed from J5; value OUT2 -> OUT1
- R10: renamed from R12; value 10k -> 56k
- R6: value 1k -> 10k
- R7: value 4k7 -> 10k
- R8: value 1k -> 4k7
- moved R2 73.8 mm to (173.8, 93.8), turned to 180 degrees
- moved R1 71.9 mm to (177.0, 93.8)
- moved J1 70.4 mm to (176.3, 100.0), turned to 90 degrees
- moved H1 38.8 mm to (175.4, 40.6)
- moved H2 31.4 mm to (175.4, 72.6)
- moved U8 25.4 mm to (41.8, 122.4)
- moved U7 21.8 mm to (118.1, 88.4), turned to -90 degrees
- moved R5 13.0 mm to (238.0, 82.4)
- moved R19 9.81 mm to (108.6, 88.6), turned to -90 degrees
- moved R20 7.83 mm to (108.6, 85.4), turned to -90 degrees
- moved C10 6.21 mm to (65.4, 156.4)
- moved R23 6.21 mm to (69.4, 160.1)
- moved C11 6.21 mm to (65.5, 161.1)
- moved R22 6.21 mm to (69.4, 157.6)
- renumbered C9 to C10, C10 to C11, C11 to C12, C12 to C13, C13 to C14, C14 to C15, C7 to C4, C8 to C6, C6 to C7, C4 to C8, D4 to D2, D5 to D3, D2 to D4, D3 to D5, J4 to J3, R2 to R1, R14 to R12, R16 to R13, R15 to R14, R17 to R15, R22 to R17, R3 to R2, R23 to R22, R24 to R23, R4 to R3, R5 to R4, R1 to R5, R11 to R9, SW5 to SW4, U2 to U3, U3 to U5, U5 to U7, U6 to U8
Connections:
- net AMP-OUT2+ renamed AMP-OUT1+
- net AMP-OUT2- renamed AMP-OUT1-
- net AMP2 renamed AMP1
- D2 pad 1: Net-(D4-K) -> Net-(D2-K)
- D3 pad 1: Net-(D4-K) -> Net-(D2-K)
- D3 pad 2: VBUS -> VREG
- Q1 pad 2: Net-(D4-K) -> VBOOST
- R10 pad 2: Net-(R12-Pad2) -> GND
- R5 pad 1: Net-(U1-TXD) -> Net-(R5-Pad1)
- SW4 pad 1: Net-(D4-K) -> VBOOST
- U1 pad 4: unconnected-(U1-~{RTS}-Pad4) -> ~{RTS}
- U1 pad 8: Net-(U1-TXD) -> USB_TXD
- U1 pad 9: UPDI -> USB_RXD
- U5 pad 11: LED -> AVR_TXD
- U5 pad 12: BTN1 -> AVR_RXD
- U5 pad 13: BTN2 -> Net-(U5-PA3)
- U5 pad 2: BTN3 -> BTN1
- U5 pad 3: BTN4 -> BTN2
- U5 pad 4: MODE -> BTN3
- U5 pad 5: ~{SD} -> LED
- U5 pad 6: WO0 -> ~{SD}
- U5 pad 7: WO2 -> MODE
- U5 pad 8: SCL -> WO1
- U5 pad 9: SDA -> WO0
- U7 pad 3': WO2 -> WO1
Routing:
- net Net-(J1-CC1): track 0.00 -> 9.33 mm
- net Net-(J1-CC2): track 0.00 -> 5.79 mm
Other:
- board outline added: 44 x 44 mm
