File: proj/musicbox/slim/slim.kicad_pcb (KiCad board)
At the start: 2 copper layers, 44 x 44 mm, 66 parts, among them J1 USB, J2 NiMh*2, J3 OUT0, J4 OUT1, Q1 AO3401A, SW1 SW, SW2 SW, SW3 SW, SW4 POW, U1 CH340E, U2 TS5A23159DGS, U3 TPS56124x, U4 BQ25172, U5 ATtiny1604-SS, U6 TPS613222ADBV, U7 alps-rk10j12e, U8 PAM8406D

Commit message: -
Parts:
- removed JP1: CHG, Resistor_SMD:R_0603_1608Metric
- removed JP2: SW, Resistor_SMD:R_0603_1608Metric
- J1, SW4, U7: moved to B.Cu
- U4: footprint Package_SON:WSON-8-1EP_2x2mm_P0.5mm_EP0.9x1.6mm -> Package_SON:Texas_DSG0008A_WSON-8-1EP_2x2mm_P0.5mm_EP0.9x1.6mm
- moved D3 125.2 mm to (57.0, 101.3)
- moved D2 125.2 mm to (57.0, 98.7)
- moved H2 105.8 mm to (80.0, 118.4)
- moved J1 104.4 mm to (72.0, 96.0)
- moved SW4 92.8 mm to (83.4, 90.8)
- moved SW1 70.4 mm to (112.0, 92.0)
- moved SW2 70.0 mm to (112.0, 100.0)
- moved SW3 69.5 mm to (112.0, 108.0)
- moved R19 34.9 mm to (142.8, 95.4)
- moved R20 34.9 mm to (142.8, 92.2)
- moved U7 13.8 mm to (126.2, 99.6), turned to 90 degrees
Connections:
- D2 pad 1: Net-(D2-K) -> VCC
- D2 pad 2: +BATT -> Net-(D2-A)
- D3 pad 1: Net-(D2-K) -> VCC
- D3 pad 2: VREG -> VBUS
- L2 pad 1: Net-(D2-K) -> +BATT
- Q1 pad 3: VCC -> Net-(D2-A)
Routing:
- net Net-(J1-CC1): track 9.33 -> 0.00 mm
- net Net-(J1-CC2): track 5.79 -> 0.00 mm
Other:
- board size 44 x 44 mm -> 64 x 24 mm

Commit message: -
Parts:
- removed the D2 at (57.0, 98.7)
- removed the D3 at (57.0, 101.3)
- removed J3: OUT0, Connector_JST:JST_ZH_S2B-ZR-SM4A-TF_1x02-1MP_P1.50mm_Horizontal
- added D4: CUHS20S30, Library:US2H, F.Cu at (36.2, 115.5)
- added D5: CUHS20S30, Library:US2H, F.Cu at (36.2, 118.2)
- added R24: 10k, Resistor_SMD:R_0603_1608Metric, F.Cu at (35.9, 120.8)
- added TP1: OUT0-, TestPoint:TestPoint_Pad_1.5x1.5mm, B.Cu at (126.6, 123.4)
- added TP2: OUT0+, TestPoint:TestPoint_Pad_D1.5mm, B.Cu at (131.2, 123.4)
- H1, H2, J2, R1, R2: moved to B.Cu
- J4: footprint Connector_JST:JST_ZH_S2B-ZR-SM4A-TF_1x02-1MP_P1.50mm_Horizontal -> Connector_JST:JST_ZH_B2B-ZR_1x02_P1.50mm_Vertical
- moved U2 102.8 mm to (125.7, 85.2)
- moved U1 96.7 mm to (131.2, 85.2), turned to 90 degrees
- moved J4 91.7 mm to (123.2, 123.3)
- moved R19 88.2 mm to (163.7, 177.9)
- moved R18 88.2 mm to (163.7, 181.1)
- moved U8 86.6 mm to (128.0, 115.0), turned to -90 degrees
- moved J2 85.1 mm to (120.3, 78.8), turned to -90 degrees
- moved C11 77.2 mm to (123.0, 109.6), turned to 90 degrees
- moved C14 76.1 mm to (129.4, 109.6), turned to -90 degrees
- moved R22 76.0 mm to (126.2, 109.6), turned to -90 degrees
- moved C13 75.3 mm to (127.8, 109.6), turned to -90 degrees
- moved H1 73.3 mm to (113.0, 79.0), turned to 180 degrees
- moved C12 72.8 mm to (127.8, 120.4), turned to 90 degrees
- moved R20 70.3 mm to (129.4, 120.4), turned to -90 degrees
- moved C15 70.2 mm to (124.6, 109.6), turned to -90 degrees
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- renumbered C5 to C4, C7 to C5, C8 to C6, C4 to C7, C6 to C8, D4 to D2, D5 to D3, R13 to R12, R12 to R13, R18 to R17, R19 to R18, R20 to R19, R21 to R20, R22 to R21, R23 to R22, R17 to R23, U5 to U4, U4 to U5, U7 to U6, U6 to U7
Connections:
- net Net-(U8-VREF) renamed /VREF
- R23 pad 2: GND -> VBUS
- U6 pad 2: Net-(C10-Pad1) -> Net-(C11-Pad1)
- U6 pad 2': Net-(C11-Pad1) -> Net-(C10-Pad1)
- U6 pad 3: WO0 -> WO1
- U6 pad 3': WO1 -> WO0
- U8 pad 1: AMP-OUT0+ -> AMP-OUT1+
- U8 pad 10: AMP1 -> AMP0
- U8 pad 14: AMP-OUT1- -> AMP-OUT0-
- U8 pad 16: AMP-OUT1+ -> AMP-OUT0+
- U8 pad 3: AMP-OUT0- -> AMP-OUT1-
- U8 pad 7: AMP0 -> AMP1
Routing:
- net VCC: track 0.00 -> 7.82 mm, vias 0 -> 6
- net ~{SD}: track 0.00 -> 5.61 mm
- net Net-(C11-Pad1): track 0.00 -> 5.29 mm
- net Net-(C10-Pad2): track 0.00 -> 3.76 mm
- net Net-(C10-Pad1): track 0.00 -> 3.33 mm
- net AMP1: track 0.00 -> 2.67 mm
- net AMP0: track 0.00 -> 2.67 mm
- net /VREF: track 0.00 -> 2.58 mm
- net MODE: track 0.00 -> 2.53 mm
- net D-: track 0.00 -> 2.44 mm
- net AMP-OUT0+: track 0.00 -> 1.00 mm, vias 0 -> 2
- net AMP-OUT1-: vias 0 -> 2
- net AMP-OUT1+: vias 0 -> 2
- net AMP-OUT0-: vias 0 -> 2
- added copper zone on B.Cu, net AMP-OUT0+
- added copper zone on B.Cu, net AMP-OUT0-
- added copper zone on F.Cu, net AMP-OUT0-
- added copper zone on B.Cu, net AMP-OUT1+
- added copper zone on F.Cu, net AMP-OUT1+
- added copper zone on B.Cu, net AMP-OUT1-
- added copper zone on F.Cu, net AMP-OUT1-
- added copper zone on B.Cu, net VCC
Other:
- board size 64 x 24 mm -> 24 x 49 mm

Commit message: -
Parts:
- moved R24 133.7 mm to (167.9, 142.2)
- moved D4 131.4 mm to (166.2, 135.5)
- moved D5 131.4 mm to (166.2, 138.2)
- moved U4 50.2 mm to (120.0, 103.0)
- moved C12 1.13 mm to (128.6, 119.6), turned to 180 degrees
- moved R20 1.13 mm to (128.6, 121.2), turned to 0 degrees
Routing:
- net ~{SD}: track 5.61 -> 13.3 mm, vias 0 -> 1
- net MODE: track 2.53 -> 9.49 mm, vias 0 -> 1
- net Net-(C11-Pad2): track 0.00 -> 3.86 mm
- net GND: track 0.00 -> 2.93 mm, vias 0 -> 7
- net VCC: track 7.82 -> 5.49 mm
- added copper zone on B.Cu, net GND
- added copper zone on F.Cu, net GND
- added copper zone on F.Cu, net VCC

Commit message: -
Parts:
- removed H2: MountingHole_Pad, MountingHole:MountingHole_3.2mm_M3_Pad
- R18, R19: moved to B.Cu
- moved C4 97.3 mm to (122.2, 56.5)
- moved C3 94.7 mm to (122.2, 54.0)
- moved R4 93.5 mm to (122.2, 61.5)
- moved U7 89.6 mm to (159.3, 87.5)
- moved L1 89.6 mm to (126.2, 55.1), turned to 180 degrees
- moved C7 87.7 mm to (147.9, 70.1)
- moved C5 86.2 mm to (122.2, 59.0)
- moved R11 84.3 mm to (138.9, 73.3)
- moved L2 84.2 mm to (164.4, 92.8)
- moved U5 83.8 mm to (148.3, 73.5)
- moved R6 83.5 mm to (118.3, 55.5)
- moved R7 83.5 mm to (118.3, 58.0)
- moved R8 83.5 mm to (118.3, 60.6)
- moved C8 83.4 mm to (147.7, 67.9)
- moved R14 83.3 mm to (138.9, 68.7)
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Routing:
- net BTN1: track 0.00 -> 32.8 mm, vias 0 -> 1
- net BTN2: track 0.00 -> 11.5 mm, vias 0 -> 1
- net BTN3: track 0.00 -> 11.0 mm, vias 0 -> 1
- net WO0: track 0.00 -> 6.34 mm
- net ~{SD}: track 13.3 -> 19.3 mm, vias 1 -> 2
- net WO1: track 0.00 -> 3.35 mm
- net AMP1: track 2.92 -> 5.69 mm
- net D+: track 0.00 -> 2.44 mm
- net Net-(C11-Pad1): track 5.29 -> 7.55 mm
- net Net-(C10-Pad1): track 3.33 -> 5.40 mm
- net GND: track 2.93 -> 1.93 mm, vias 7 -> 10
- net MODE: track 9.49 -> 9.35 mm, vias 1 -> 2

Commit message: -
Parts:
- moved R16 33.3 mm to (113.2, 113.0)
- moved C15 2.53 mm to (127.0, 108.8), turned to 180 degrees
- moved R22 2.53 mm to (124.6, 109.6), turned to -90 degrees
- moved C6 0.40 mm to (111.4, 122.6)
Routing:
- net BTN2: track 11.5 -> 25.5 mm
- net LED: track 0.00 -> 11.1 mm, vias 0 -> 1
- net BTN3: track 11.0 -> 18.0 mm
- net AMP1: track 5.69 -> 2.19 mm
- net /VREF: track 2.58 -> 5.55 mm
- net Net-(C11-Pad2): track 3.86 -> 1.62 mm
- net VCC: vias 6 -> 8
- net GND: vias 10 -> 9

Commit message: -
Parts:
- removed the D2 at (146.0, 122.0)
- removed the D3 at (148.1, 65.3)
- removed the R15 at (140.1, 65.3)
- removed the R3 at (159.8, 68.0)
- added JP1: AMP_AB, Resistor_SMD:R_0603_1608Metric, B.Cu at (118.6, 122.2)
- D1: value TNOW -> WS2812B-2020; footprint LED_SMD:LED_0603_1608Metric -> LED_SMD:LED_WS2812B-2020_PLCC4_2.0x2.0mm
- moved D1 47.6 mm to (128.0, 100.0)
- moved R11 29.5 mm to (125.0, 103.8)
- moved R14 4.73 mm to (117.6, 111.2)
- moved C1 3.47 mm to (156.2, 71.0)
- renumbered D4 to D2, D5 to D3, J4 to J3, R11 to R10, R12 to R11, R13 to R12, R14 to R13, R16 to R14, R17 to R15, R18 to R16, R19 to R17, R20 to R18, R21 to R19, R22 to R20, R23 to R21, R24 to R22, R4 to R3, R5 to R4, R6 to R5, R7 to R6, R8 to R7, R9 to R8, R10 to R9
Connections:
- D1 pad 1: GND -> unconnected-(D1-DOUT-Pad1)
- D1 pad 2: Net-(D1-A) -> GND
- R11 pad 2: Net-(D2-A) (its old number) -> Net-(D1-DIN)
- R19 pad 2: AMP0 -> AMP1
- R20 pad 2: AMP1 -> AMP2
- TP1 pad 1: AMP-OUT0- -> AMP-OUT2-
- TP2 pad 1: AMP-OUT0+ -> AMP-OUT2+
- U1 pad 6: TNOW -> unconnected-(U1-TNOW-Pad6)
- U4 pad 7: MODE -> WO2
- U4 pad 9: WO0 -> STAT
- U6 pad 3: WO1 -> WO2
- U6 pad 3': WO0 -> WO1
- U8 pad 1: AMP-OUT1+ -> AMP-OUT2+
- U8 pad 10: AMP0 -> AMP1
- U8 pad 14: AMP-OUT0- -> AMP-OUT1-
- U8 pad 16: AMP-OUT0+ -> AMP-OUT1+
- U8 pad 3: AMP-OUT1- -> AMP-OUT2-
- U8 pad 7: AMP1 -> AMP2
Routing:
- net STAT: track 0.00 -> 20.5 mm, vias 0 -> 1
- net LED: track 11.1 -> 2.32 mm
- net WO2: track 0.00 -> 8.30 mm
- net Net-(SW4-C): track 0.00 -> 6.56 mm
- net UPDI: track 0.00 -> 6.50 mm, vias 0 -> 1
- net WO0: track 6.34 -> 0.00 mm
- net Net-(U4-PA3): track 0.00 -> 6.14 mm, vias 0 -> 1
- net AVR_TXD: track 0.00 -> 5.30 mm, vias 0 -> 1
- net AVR_RXD: track 0.00 -> 5.07 mm, vias 0 -> 1
- net Net-(D1-DIN): track 0.00 -> 4.53 mm
- net Net-(Q1-G): track 0.00 -> 3.90 mm
- net AMP0: track 2.67 -> 0.00 mm
- net BTN1: track 32.4 -> 34.6 mm
- net AMP2: track 0.00 -> 2.19 mm
- net WO1: track 3.35 -> 5.35 mm
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- added copper zone on B.Cu, net AMP-OUT2+
- added copper zone on B.Cu, net AMP-OUT2-
- added copper zone on F.Cu, net AMP-OUT2-
- removed copper zone on B.Cu, net AMP-OUT0+
- removed copper zone on B.Cu, net AMP-OUT0-
- removed copper zone on F.Cu, net AMP-OUT0-
