File: proj/usb/c-test/c-test.kicad_pcb (KiCad board)
At the start: 2 copper layers, 13 parts, among them J1 USB_C_Receptacle_USB2.0_16P, P1 USB_C_Plug, U1 INA181, U2 AP7375, U3 ATtiny404-SS

Commit message: -
Parts:
- removed C3: 0u1, Capacitor_SMD:C_0603_1608Metric
- added J2: Conn_01x03, Connector_PinHeader_2.54mm:PinHeader_1x03_P2.54mm_Vertical, F.Cu at (146.2, 124.0)
- added R5: 47k, Resistor_SMD:R_0603_1608Metric, F.Cu at (107.8, 107.4)
- added R6: 56k, Resistor_SMD:R_0603_1608Metric, F.Cu at (111.0, 107.4)
- added RV1: 10k, Potentiometer_SMD:Potentiometer_Bourns_TC33X_Vertical, F.Cu at (111.4, 111.0)
- added SW1: SW_Push, Library:alps-skr[gp], F.Cu at (124.9, 114.3)
- added U2: MCP6L91T-EOT, Package_TO_SOT_SMD:SOT-23-5, F.Cu at (107.8, 110.4)
- R1, R4: value 10k -> 47k
- R3: value 4k7 -> 10k
- R7: renamed from R5; value 7m -> 8m; footprint Resistor_SMD:R_0603_1608Metric -> Resistor_SMD:R_0805_2012Metric
- U1: renamed from U2; value AP7375 -> AP7375-33
- U3: value ATtiny404-SS -> ATtiny402-SS; footprint Package_SO:SOIC-14_3.9x8.7mm_P1.27mm -> Package_SO:SOIC-8_3.9x4.9mm_P1.27mm
- moved U3 58.1 mm to (123.4, 127.9)
- moved R1 55.5 mm to (132.6, 104.8)
- moved R2 55.5 mm to (132.6, 107.3)
- moved R3 55.5 mm to (132.6, 109.8)
- moved C1 43.7 mm to (97.2, 111.4), turned to 180 degrees
- moved C2 38.7 mm to (97.2, 108.6), turned to 180 degrees
- moved P1 33.3 mm to (111.4, 98.8), turned to 90 degrees
- moved R7 32.2 mm to (104.0, 112.8)
- moved R4 30.4 mm to (104.6, 107.4)
- moved U1 29.1 mm to (99.8, 110.0), turned to 180 degrees
- moved U4 24.7 mm to (104.0, 110.0)
- moved J1 14.5 mm to (86.5, 101.7), turned to -90 degrees
- renumbered U1 to U4
Connections:
- C2 pad 1: +5V -> +3V3
- R4 pad 1: VREF_PWM -> +3V3
- R4 pad 2: VREF -> Net-(R4-Pad2)
- U1 pad 2: +5V -> +3V3
- U3 pad 1: +5V -> +3V3
- U3 pad 2: I_SENSE -> SOUT
- U3 pad 3: V_SENSE -> I_SENSE
- U3 pad 4: unconnected-(U3-PA6-Pad4) -> SDA
- U3 pad 5: VREF -> SCL
- U3 pad 6: VREF_PWM -> UPDI
- U3 pad 7: unconnected-(U3-PB2-Pad7) -> V_SENSE
- U3 pad 8: SDA -> GND
- U4 pad 6: +5V -> +3V3
