File: proj/audio/mini-dexed/mini-dexed.kicad_pcb (KiCad board)
At the start: 2 copper layers, 100 x 95 mm, 42 parts, among them J1 Raspberry_Pi_2_3, J3 OLED, J4 Conn_01x05_Pin, J5 Conn_01x05_Socket, Q1 AO3401A, SW1 RotaryEncoder_Switch_MP, SW2 POW, U1 TPS613222ADBV, U2 PCM5102A

Commit message: -
Parts:
- removed BT1: Battery, Library:BH-321-1P_{24}
- removed the C1 at (88.2, 154.8)
- removed the C2 at (91.8, 154.8)
- removed the C3 at (90.8, 146.0)
- removed the R1 at (88.2, 153.2)
- removed the R2 at (91.8, 153.2)
- removed the R3 at (89.2, 146.0)
- added C12: 1u, Capacitor_SMD:C_0603_1608Metric, F.Cu at (245.8, 106.0)
- added C13: 1u, Capacitor_SMD:C_0603_1608Metric, F.Cu at (245.8, 108.5)
- added C14: 1u, Capacitor_THT:C_Disc_D5.0mm_W2.5mm_P5.00mm, F.Cu at (228.9, 118.9)
- added C15: 1u, Capacitor_THT:C_Disc_D5.0mm_W2.5mm_P5.00mm, F.Cu at (228.9, 106.7)
- added C16: 1u, Capacitor_THT:C_Disc_D5.0mm_W2.5mm_P5.00mm, F.Cu at (228.9, 110.8)
- added C17: 1u, Capacitor_THT:C_Disc_D5.0mm_W2.5mm_P5.00mm, F.Cu at (228.9, 114.8)
- added D2: mute, LED_SMD:LED_0603_1608Metric, F.Cu at (248.3, 122.2)
- added J1: BATT, Connector_JST:JST_XH_B2B-XH-A_1x02_P2.50mm_Vertical, F.Cu at (230.8, 138.6)
- added JP3: pokayoke, Library:pokayoke_1608, F.Cu at (215.8, 138.8)
- added R10: 1k, Resistor_SMD:R_0603_1608Metric, F.Cu at (249.8, 111.0)
- added R11: 10k, Resistor_SMD:R_0603_1608Metric, F.Cu at (249.8, 116.0)
- added R12: 10k, Resistor_SMD:R_0603_1608Metric, F.Cu at (249.8, 113.5)
- added R13: 10k, Resistor_SMD:R_0603_1608Metric, F.Cu at (245.8, 118.5)
- added R14: 10k, Resistor_SMD:R_0603_1608Metric, F.Cu at (249.8, 106.0)
- added R5: 56k, Resistor_SMD:R_0603_1608Metric, F.Cu at (245.8, 113.5)
- added R6: 56k, Resistor_SMD:R_0603_1608Metric, F.Cu at (245.8, 116.0)
- added R9: 1k, Resistor_SMD:R_0603_1608Metric, F.Cu at (249.8, 108.5)
- added RV1: VOL_L, Potentiometer_SMD:Potentiometer_Bourns_TC33X_Vertical, F.Cu at (216.9, 134.3)
- added RV2: VOL_R, Potentiometer_SMD:Potentiometer_Bourns_TC33X_Vertical, F.Cu at (216.9, 129.6)
- added SW3: SW_Push, Library:alps-skr[gp], F.Cu at (217.5, 116.0)
- added SW4: SW_Push, Library:alps-skr[gp], F.Cu at (217.5, 123.5)
- added SW5: mute, Library:IS-1245T-G, F.Cu at (232.6, 130.9)
- added TP1: D-, TestPoint:TestPoint_Pad_D4.0mm, F.Cu at (224.3, 107.7)
- added TP2: D+, TestPoint:TestPoint_Pad_D4.0mm, F.Cu at (224.3, 113.8)
- added TP3: ID, TestPoint:TestPoint_Pad_D4.0mm, F.Cu at (224.3, 119.8)
- added TP4: +OUT_L, TestPoint:TestPoint_Pad_D2.0mm, F.Cu at (223.3, 124.9)
- added TP5: -OUT_L, TestPoint:TestPoint_Pad_2.0x2.0mm, F.Cu at (223.3, 133.0)
- added TP6: -OUT_R, TestPoint:TestPoint_Pad_2.0x2.0mm, F.Cu at (223.3, 137.0)
- added TP7: +OUT_R, TestPoint:TestPoint_Pad_D2.0mm, F.Cu at (223.3, 128.9)
- added U3: PAM8406D, Package_SO:SOIC-16_3.9x9.9mm_P1.27mm, F.Cu at (242.1, 126.8)
- J4: value Conn_01x05_Pin -> USB_C_Receptacle_USB2.0_16P; footprint Connector_PinHeader_2.54mm:PinHeader_1x05_P2.54mm_Vertical -> Connector_USB:USB_C_Receptacle_GCT_USB4110
- J5: value Conn_01x05_Socket -> AudioJack3; footprint Connector_PinSocket_2.54mm:PinSocket_1x05_P2.54mm_Vertical -> Library:MJ-8435; moved to F.Cu
- SW1: value RotaryEncoder_Switch_MP -> POW; footprint Rotary_Encoder:RotaryEncoder_Alps_EC12E-Switch_Vertical_H20mm -> Library:IS-1245T-G
- SW2: value POW -> SW_Push; footprint Button_Switch_THT:SW_Push_2P2T_Toggle_CK_PVA2xxH3xxxxxxV2 -> Library:alps-skr[gp]
- moved J4 165.2 mm to (245.1, 137.8)
- moved SW1 149.0 mm to (232.6, 123.8), turned to 0 degrees
- moved J5 121.5 mm to (239.6, 107.8), turned to 0 degrees
- moved JP1 112.7 mm to (245.8, 111.0)
- moved SW2 47.4 mm to (217.5, 108.5)
- renumbered C4 to C1, C12 to C10, C13 to C11, C14 to C2, C5 to C3, C6 to C4, C10 to C5, C11 to C6, J1 to J2, R4 to R1, R9 to R2, R5 to R3, R6 to R4
Connections:
- J2 pad 12: unconnected-(J1-GPIO18/PWM0-Pad12) -> BCK
- J2 pad 19: CLK -> BTN2
- J2 pad 21: DT -> BTN1
- J2 pad 23: SW -> BTN3
- J2 pad 35: unconnected-(J1-GPIO19/MISO1-Pad35) -> LCK
- J2 pad 40: unconnected-(J1-GPIO21/SCLK1-Pad40) -> DIN
- R1 pad 1: Net-(SW2A-C) -> Net-(SW1-C)
- SW2 pad 1: +BATT -> BTN1
- SW2 pad 2: Net-(Q1-G) -> GND
- U2 pad 12: unconnected-(U2-SCK-Pad12) -> GND
- U2 pad 13: unconnected-(U2-BCK-Pad13) -> BCK
- U2 pad 14: unconnected-(U2-DIN-Pad14) -> DIN
- U2 pad 15: unconnected-(U2-LRCK-Pad15) -> LCK
Routing:
- net RE_B: track 17.8 -> 0.00 mm, vias 1 -> 0
- net RE_SW: track 15.7 -> 0.00 mm, vias 1 -> 0
- net RE_A: track 12.2 -> 0.00 mm, vias 1 -> 0
- net RE_V: track 8.66 -> 0.00 mm
- removed copper zone on B.Cu, net RE_GND
- removed copper zone on F.Cu, net RE_GND
- removed copper zone on B.Cu, net RE_V
Other:
- board size 100 x 95 mm -> 100 x 75 mm
