File: proj/avr/tx04_s/tx04_s.kicad_sch (KiCad schematic)
At the start: 13 parts, among them J1 USB_C_Receptacle_USB2.0_16P, J2 Conn_02x07_Counter_Clockwise, SW1 SW_Push, U1 ATtiny1604-SS, U2 AP7333

Commit message: -
Parts:
- removed D1: 2BZX84Cxx, Package_TO_SOT_SMD:SOT-23, symbol Diode:2BZX84Cxx
- removed U2: AP7333, Package_TO_SOT_SMD:SOT-23-3, symbol Library:AP7333
- added D1: BZB784-Cxx, Package_TO_SOT_SMD:SOT-323_SC-70, symbol Library:BZB784-Cxx
- R3, R4: value 4k7 -> 1k
Connections:
- net VBUS is gone; now on net VCC: J1.A4 (VBUS), J1.A9 (VBUS), J1.B4 (VBUS), J1.B9 (VBUS)
- net D+: now also D1.2 (K)
- net D-: now also D1.1 (K)
- net GND: now also D1.3 (A)
